File: cellular.sch (KiCad schematic (older format))
At the start: 54 parts, among them Q1 2SC1815, Q2 2SC1815, Q3 2SC1815, Q4 2SC1815, SW1 SW_PUSH, SW2 SW_PUSH, U1 MP2365DN, U2 SIM800, U6 SIM HOLD - PPSS-6P

Commit message: swap TX RX, place component name
Parts:
- renumbered SW1 to PWR1, SW2 to RST1
Changed lines of the file:
@@
 $EndComp
 $Comp
-L GND #PWR01
+L GND #PWR16
 U 1 1 57DA6B65
 P 4750 7450
-F 0 "#PWR01" H 4750 7200 50  0001 C CNN
+F 0 "#PWR16" H 4750 7200 50  0001 C CNN
 F 1 "GND" H 4755 7277 50  0000 C CNN
 F 2 "" H 4750 7450 50  0000 C CNN
@@
 $EndComp
 $Comp
-L GND #PWR02
+L GND #PWR25
 U 1 1 57DA6B68
 P 10450 1900
-F 0 "#PWR02" H 10450 1650 50  0001 C CNN
+F 0 "#PWR25" H 10450 1650 50  0001 C CNN
 F 1 "GND" H 10455 1727 50  0000 C CNN
 F 2 "" H 10450 1900 50  0000 C CNN
@@
 SIM800L_NETLIGHT
 $Comp
-L +5V #PWR03
+L +5V #PWR1
 U 1 1 57DA6B80
 P 800 5700
-F 0 "#PWR03" H 800 5550 50  0001 C CNN
+F 0 "#PWR1" H 800 5550 50  0001 C CNN
 F 1 "+5V" H 815 5873 50  0000 C CNN
 F 2 "" H 800 5700 50  0000 C CNN
@@
 $EndComp
 $Comp
-L GND #PWR04
+L GND #PWR28
 U 1 1 57DA6B94
 P 10450 4750
-F 0 "#PWR04" H 10450 4500 50  0001 C CNN
+F 0 "#PWR28" H 10450 4500 50  0001 C CNN
 F 1 "GND" H 10455 4577 50  0000 C CNN
 F 2 "" H 10450 4750 50  0000 C CNN
@@
 NoConn ~ 1300 6150
 $Comp
-L GND #PWR05
+L GND #PWR5
 U 1 1 57DA6B9E
 P 1100 7450
-F 0 "#PWR05" H 1100 7200 50  0001 C CNN
+F 0 "#PWR5" H 1100 7200 50  0001 C CNN
 F 1 "GND" H 1105 7277 50  0000 C CNN
 F 2 "" H 1100 7450 50  0000 C CNN
@@
 $EndComp
 $Comp
-L VDD #PWR06
+L VDD #PWR10
 U 1 1 57DA6BAA
 P 3750 6090
-F 0 "#PWR06" H 3750 5940 50  0001 C CNN
+F 0 "#PWR10" H 3750 5940 50  0001 C CNN
 F 1 "VDD" H 3767 6263 50  0000 C CNN
 F 2 "" H 3750 6090 50  0000 C CNN
@@
 $EndComp
 $Comp
-L VDD #PWR07
+L VDD #PWR15
 U 1 1 57DA6BAB
 P 4750 7050
-F 0 "#PWR07" H 4750 6900 50  0001 C CNB
+F 0 "#PWR15" H 4750 6900 50  0001 C CNB
 F 1 "VDD" H 4767 7223 50  0000 C CNB
 F 2 "" H 4750 7050 50  0000 C CNN
@@
 $EndComp
 $Comp
-L VDD #PWR08
+L VDD #PWR27
 U 1 1 57DA6BAC
 P 10450 3850
-F 0 "#PWR08" H 10450 3700 50  0001 C CNN
+F 0 "#PWR27" H 10450 3700 50  0001 C CNN
 F 1 "VDD" H 10467 4023 50  0000 C CNB
 F 2 "" H 10450 3850 50  0000 C CNN
@@
 NoConn ~ 7750 5200
 $Comp
-L GND #PWR09
+L GND #PWR22
 U 1 1 57DA6BB4
 P 7900 5050
-F 0 "#PWR09" H 7900 4800 50  0001 C CNN
+F 0 "#PWR22" H 7900 4800 50  0001 C CNN
 F 1 "GND" H 7905 4877 50  0000 C CNN
 F 2 "" H 7900 5050 50  0000 C CNN
@@
 NoConn ~ 7600 5575
 $Comp
-L GND #PWR010
+L GND #PWR21
 U 1 1 57DA6BB5
 P 7400 6225
-F 0 "#PWR010" H 7400 5975 50  0001 C CNN
+F 0 "#PWR21" H 7400 5975 50  0001 C CNN
 F 1 "GND" H 7405 6052 50  0000 C CNN
 F 2 "" H 7400 6225 50  0000 C CNN
@@
 $EndComp
 $Comp
-L GND #PWR011
+L GND #PWR23
 U 1 1 57DA6BB8
 P 8150 5750
-F 0 "#PWR011" H 8150 5500 50  0001 C CNN
+F 0 "#PWR23" H 8150 5500 50  0001 C CNN
 F 1 "GND" H 8155 5577 50  0000 C CNN
 F 2 "" H 8150 5750 50  0000 C CNN
@@
 $EndComp
 $Comp
-L GND #PWR012
+L GND #PWR20
 U 1 1 58A2B6B5
 P 6200 2100
-F 0 "#PWR012" H 6200 1850 50  0001 C CNN
+F 0 "#PWR20" H 6200 1850 50  0001 C CNN
 F 1 "GND" H 6205 1927 50  0000 C CNN
 F 2 "" H 6200 2100 50  0000 C CNN
@@
 $EndComp
 $Comp
-L +5V #PWR013
+L +5V #PWR19
 U 1 1 58A2D721
 P 6200 1850
-F 0 "#PWR013" H 6200 1700 50  0001 C CNN
+F 0 "#PWR19" H 6200 1700 50  0001 C CNN
 F 1 "+5V" H 6215 2023 50  0000 C CNN
 F 2 "" H 6200 1850 50  0000 C CNN
@@
 SIM800L_NETLIGHT
 $Comp
-L VCC #PWR014
+L VCC #PWR4
 U 1 1 58A55439
 P 1000 5700
-F 0 "#PWR014" H 1050 5750 50  0001 C CNN
+F 0 "#PWR4" H 1050 5750 50  0001 C CNN
 F 1 "VCC" H 1017 5873 50  0000 C CNN
 F 2 "" H -3500 -6875 50  0000 C CNN
@@
 $EndComp
 $Comp
-L PWR_FLAG #FLG015
+L PWR_FLAG #FLG1
 U 1 1 58A554C4
 P 1325 5750
-F 0 "#FLG015" H 1375 5800 50  0001 C CNN
+F 0 "#FLG1" H 1375 5800 50  0001 C CNN
 F 1 "PWR_FLAG" H 1325 5974 50  0000 C CNN
 F 2 "" H -2550 -6725 50  0000 C CNN
@@
 $EndComp
 $Comp
-L PWR_FLAG #FLG016
+L PWR_FLAG #FLG2
 U 1 1 58A55AC7
 P 3750 7425
-F 0 "#FLG016" H 3800 7475 50  0001 C CNN
+F 0 "#FLG2" H 3800 7475 50  0001 C CNN
 F 1 "PWR_FLAG" H 3750 7648 50  0000 C CNN
 F 2 "" H -325 -5475 50  0000 C CNN
@@
 Text GLabel 1900 3000 0    60   Input ~ 0
 SIM800L_RXD
+Text GLabel 8300 2875 2    60   Input ~ 0
+SIM800L_TXD
 Text GLabel 8300 2775 2    60   Input ~ 0
-SIM800L_TXD
-Text GLabel 8300 2875 2    60   Input ~ 0
 SIM800L_RXD
 Text GLabel 8300 2375 2    60   Input ~ 12
@@
 $EndComp
 $Comp
-L GND #PWR017
+L GND #PWR30
 U 1 1 58A81DF9
 P 10450 6150
-F 0 "#PWR017" H 10450 5900 50  0001 C CNN
+F 0 "#PWR30" H 10450 5900 50  0001 C CNN
 F 1 "GND" H 10455 5977 50  0000 C CNN
 F 2 "" H 10450 6150 50  0000 C CNN
@@
 $EndComp
 $Comp
-L VDD #PWR018
+L VDD #PWR29
 U 1 1 58A81DFF
 P 10450 5250
-F 0 "#PWR018" H 10450 5100 50  0001 C CNN
+F 0 "#PWR29" H 10450 5100 50  0001 C CNN
 F 1 "VDD" H 10467 5423 50  0000 C CNB
 F 2 "" H 10450 5250 50  0000 C CNN
@@
 $EndComp
 $Comp
-L GND #PWR019
+L GND #PWR26
 U 1 1 58AC7889
 P 10450 3250
-F 0 "#PWR019" H 10450 3000 50  0001 C CNN
+F 0 "#PWR26" H 10450 3000 50  0001 C CNN
 F 1 "GND" H 10455 3077 50  0000 C CNN
 F 2 "" H 10450 3250 50  0000 C CNN
@@
 NoConn ~ 8300 2175
 $Comp
-L GND #PWR020
+L GND #PWR24
 U 1 1 58AD4688
 P 8400 1425
-F 0 "#PWR020" H 8400 1175 50  0001 C CNN
+F 0 "#PWR24" H 8400 1175 50  0001 C CNN
 F 1 "GND" H 8405 1252 50  0000 C CNN
 F 2 "" H 8400 1425 50  0000 C CNN
@@
 $EndComp
 $Comp
-L VDD #PWR021
+L VDD #PWR13
 U 1 1 58B13F89
 P 4200 1400
-F 0 "#PWR021" H 4200 1250 50  0001 C CNN
+F 0 "#PWR13" H 4200 1250 50  0001 C CNN
 F 1 "VDD" H 4217 1573 50  0000 C CNN
 F 2 "" H 4200 1400 50  0000 C CNN
@@
 $EndComp
 $Comp
-L GND #PWR022
+L GND #PWR11
 U 1 1 58B19005
 P 3900 4600
-F 0 "#PWR022" H 3900 4350 50  0001 C CNN
+F 0 "#PWR11" H 3900 4350 50  0001 C CNN
 F 1 "GND" H 3905 4427 50  0000 C CNN
 F 2 "" H 3900 4600 50  0000 C CNN
@@
 	3900 4300 3900 4350
 $Comp
-L GND #PWR023
+L GND #PWR7
 U 1 1 58B19F6A
 P 2200 3700
-F 0 "#PWR023" H 2200 3450 50  0001 C CNN
+F 0 "#PWR7" H 2200 3450 50  0001 C CNN
 F 1 "GND" H 2205 3527 50  0000 C CNN
 F 2 "" H 2200 3700 50  0000 C CNN
@@
 $EndComp
 $Comp
-L GND #PWR024
+L GND #PWR6
 U 1 1 58B1A9F5
 P 2200 2200
-F 0 "#PWR024" H 2200 1950 50  0001 C CNN
+F 0 "#PWR6" H 2200 1950 50  0001 C CNN
 F 1 "GND" H 2205 2027 50  0000 C CNN
 F 2 "" H 2200 2200 50  0000 C CNN
@@
 $EndComp
 $Comp
-L GND #PWR025
+L GND #PWR8
 U 1 1 58B1DF6A
 P 3100 4400
-F 0 "#PWR025" H 3100 4150 50  0001 C CNN
+F 0 "#PWR8" H 3100 4150 50  0001 C CNN
 F 1 "GND" H 3105 4227 50  0000 C CNN
 F 2 "" H 3100 4400 50  0000 C CNN
@@
 $EndComp
 $Comp
-L GND #PWR026
+L GND #PWR18
 U 1 1 58B1E525
 P 5600 3300
-F 0 "#PWR026" H 5600 3050 50  0001 C CNN
+F 0 "#PWR18" H 5600 3050 50  0001 C CNN
 F 1 "GND" H 5605 3127 50  0000 C CNN
 F 2 "" H 5600 3300 50  0000 C CNN
@@
 $EndComp
 $Comp
-L GND #PWR027
+L GND #PWR17
 U 1 1 58B20018
 P 5600 2700
-F 0 "#PWR027" H 5600 2450 50  0001 C CNN
+F 0 "#PWR17" H 5600 2450 50  0001 C CNN
 F 1 "GND" H 5605 2527 50  0000 C CNN
 F 2 "" H 5600 2700 50  0000 C CNN
@@
 $EndComp
 $Comp
-L GND #PWR028
+L GND #PWR14
 U 1 1 58B206EB
 P 4500 1400
-F 0 "#PWR028" H 4500 1150 50  0001 C CNN
+F 0 "#PWR14" H 4500 1150 50  0001 C CNN
 F 1 "GND" H 4505 1227 50  0000 C CNN
 F 2 "" H 4500 1400 50  0000 C CNN
@@
 $EndComp
 $Comp
-L GND #PWR029
+L GND #PWR12
 U 1 1 58B21E26
 P 4000 1400
-F 0 "#PWR029" H 4000 1150 50  0001 C CNN
+F 0 "#PWR12" H 4000 1150 50  0001 C CNN
 F 1 "GND" H 4005 1227 50  0000 C CNN
 F 2 "" H 4000 1400 50  0000 C CNN
@@
 $EndComp
 $Comp
-L GND #PWR030
+L GND #PWR9
 U 1 1 58B22419
 P 3400 1400
-F 0 "#PWR030" H 3400 1150 50  0001 C CNN
+F 0 "#PWR9" H 3400 1150 50  0001 C CNN
 F 1 "GND" H 3405 1227 50  0000 C CNN
 F 2 "" H 3400 1400 50  0000 C CNN
@@
 SIM800L_RESET
 $Comp
-L SW_PUSH SW2
+L SW_PUSH RST1
 U 1 1 58B2A584
 P 1300 3600
-F 0 "SW2" H 1300 3855 50  0000 C CNN
+F 0 "RST1" H 1300 3855 50  0000 C CNN
 F 1 "SW_PUSH" H 1300 3764 50  0000 C CNN
 F 2 "lib:SW_SPST_B3U-1000P-B" H -7300 -4000 50  0001 C CNN
@@
 $EndComp
 $Comp
-L GND #PWR031
+L GND #PWR3
 U 1 1 58B2A58A
 P 950 3650
-F 0 "#PWR031" H 950 3400 50  0001 C CNN
+F 0 "#PWR3" H 950 3400 50  0001 C CNN
 F 1 "GND" H 955 3477 50  0000 C CNN
 F 2 "" H 950 3650 50  0000 C CNN
@@
 SIM800L_PWRKEY
 $Comp
-L SW_PUSH SW1
+L SW_PUSH PWR1
 U 1 1 58B31DFA
 P 1300 2100
-F 0 "SW1" H 1300 2355 50  0000 C CNN
+F 0 "PWR1" H 1300 2355 50  0000 C CNN
 F 1 "SW_PUSH" H 1300 2264 50  0000 C CNN
 F 2 "lib:SW_SPST_B3U-1000P-B" H -7300 -5500 50  0001 C CNN
@@
 $EndComp
 $Comp
-L GND #PWR032
+L GND #PWR2
 U 1 1 58B31E00
 P 950 2150
-F 0 "#PWR032" H 950 1900 50  0001 C CNN
+F 0 "#PWR2" H 950 1900 50  0001 C CNN
 F 1 "GND" H 955 1977 50  0000 C CNN
 F 2 "" H 950 2150 50  0000 C CNN
