File: cellular.sch (KiCad schematic (older format))
At the start: 55 parts, among them P3 Chip anten, Q1 2SC1815, Q2 2SC1815, Q3 2SC1815, Q4 2SC1815, SW1 SW_PUSH, SW2 SW_PUSH, U1 MP2365DN, U2 SIM800H, U6 SIM HOLD - PPSS-6P

Commit message: 3D model diode,inductor,switch
Parts:
- D1: footprint Diodes_SMD:D_SOD-123 -> Diodes_SMD:D_MiniMELF_Standard
Changed lines of the file:
@@
 F 0 "D1" V 8954 14318 50  0000 L CNN
 F 1 "5.1V/500mA" V 9045 14318 50  0000 L CNN
-F 2 "Diodes_SMD:D_SOD-123" V -12950 12550 50  0001 C CNN
+F 2 "Diodes_SMD:D_MiniMELF_Standard" V -12950 12550 50  0001 C CNN
 F 3 "" V -12950 12550 50  0000 C CNN
 	1    9000 14250

Commit message: modifu name compoment & text, fix track pwr
Parts:
- removed P3: Chip anten, lib:point_test, symbol CONN_01X01
- removed SW1, SW2: SW_PUSH, lib:SW_SPST_B3U-1000P-B, symbol SW_PUSH
- removed U2: SIM800H, lib:SIM800H, symbol SIM800H
- added PWR1, RST1: SW_PUSH, lib:SW_SPST_B3U-1000P-B, symbol SW_PUSH
- added U2: SIM800, lib:SIM800, symbol SIM800
Connections:
- wire segments 155 -> 139
- no-connect marks 61 -> 20
Other:
- note added: "DECOUPLING"
- note added: "SIM800"
- note removed: "POWER DECOUPLING"
- note removed: "SIM800L"
- moved on the sheet: ANT1, C10, C12, C13, C2, C28, C29, C31, C32, C33, C34, C4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

Commit message: ra-02 component
Parts:
- added U?: Ra-02, SO-16-W, symbol Ra-02
Changed lines of the file:
@@
 LIBS:sim800
 LIBS:SIM800
+LIBS:ra-02
+LIBS:cellular-cache
 EELAYER 26 0
 EELAYER END
-$Descr A4 11693 8268
+$Descr A3 16535 11693
 encoding utf-8
 Sheet 1 1
 Title "CELLULAR SHIELD"
 Date "2016-07-14"
-Rev ""
+Rev "0.2"
 Comp "NANOCHIP"
 Comment1 ""
@@
 Wire Notes Line
 	4225 7775 4225 5025
+Wire Notes Line
+	11200 500  11200 7775
+Wire Notes Line
+	11200 7775 500  7775
+$Comp
+L Ra-02 U?
+U 1 1 58BA95A8
+P 2500 8550
+F 0 "U?" H 2500 9125 50  0000 C CNN
+F 1 "Ra-02" H 2500 9034 50  0000 C CNN
+F 2 "SO-16-W" H -11300 3225 50  0001 C CIN
+F 3 "" H -10475 4225 50  0001 C CNN
+	1    2500 8550
+	1    0    0    -1
+$EndComp
 $EndSCHEMATC

Commit message: ra-02 footprint
Connections:
- net RA_SCK: now reaches U?.12 (SCK)
- net RA_MISO: now reaches U?.13 (MISO)
- net RA_MOSI: now reaches U?.14 (MOSI)
Changed lines of the file:
@@
 	1    0    0    -1
 $EndComp
+Text GLabel 2900 8400 2    60   Input ~ 0
+RA_MOSI
+Text GLabel 2900 8500 2    60   Input ~ 0
+RA_MISO
+Text GLabel 2900 8600 2    60   Input ~ 0
+RA_SCK
 $EndSCHEMATC

Commit message: 3.3V
Parts:
- added C? (x2): 10uF, lib:C_0603, symbol C_Small
- added U?: LM1117-3.3, symbol LM1117-3.3
Connections:
- net +5V: now also C?.1, U?.3 (VI)
- net GND: now also U?.1 (GND), U?.16 (GND), U?.2 (GND), U?.9 (GND), C?.2, U?.1 (GND/ADJ)
- net RA_CS: now reaches U?.15 (NSS)
- net +3V3: now reaches U?.3 (3.3V)
- net +3V3: now also U?.2 (VO), U?.4 (VO)
- net RA_RESET: now reaches U?.4 (RESET)
Changed lines of the file:
@@
 Text GLabel 2900 8600 2    60   Input ~ 0
 RA_SCK
+Text GLabel 2100 8500 0    60   Input ~ 0
+RA_RESET
+$Comp
+L GND #PWR?
+U 1 1 58BB1771
+P 1950 8200
+F 0 "#PWR?" H 1950 7950 50  0001 C CNN
+F 1 "GND" V 1900 7950 50  0000 C CNN
+F 2 "" H 1950 8200 50  0000 C CNN
+F 3 "" H 1950 8200 50  0000 C CNN
+	1    1950 8200
+	0    1    1    0
+$EndComp
+$Comp
+L GND #PWR?
+U 1 1 58BB20C3
+P 3050 8200
+F 0 "#PWR?" H 3050 7950 50  0001 C CNN
+F 1 "GND" V 3050 8000 50  0000 C CNN
+F 2 "" H 3050 8200 50  0000 C CNN
+F 3 "" H 3050 8200 50  0000 C CNN
+	1    3050 8200
+	0    -1   -1   0
+$EndComp
+$Comp
+L GND #PWR?
+U 1 1 58BB21E1
+P 3050 8900
+F 0 "#PWR?" H 3050 8650 50  0001 C CNN
+F 1 "GND" V 3050 8700 50  0000 C CNN
+F 2 "" H 3050 8900 50  0000 C CNN
+F 3 "" H 3050 8900 50  0000 C CNN
+	1    3050 8900
+	0    -1   -1   0
+$EndComp
+Wire Wire Line
+	1950 8200 2100 8200
+Wire Wire Line
+	2100 8300 2050 8300
+Wire Wire Line
+	2050 8300 2050 8200
+Connection ~ 2050 8200
+Wire Wire Line
+	2900 8200 3050 8200
+Wire Wire Line
+	3050 8900 2900 8900
+$Comp
+L +3V3 #PWR?
+U 1 1 58BB2B76
+P 1950 8400
+F 0 "#PWR?" H 2000 8450 50  0001 C CNN
+F 1 "+3V3" V 1965 8528 50  0000 L CNN
+F 2 "" H -5825 1400 50  0000 C CNN
+F 3 "" H -5825 1400 50  0000 C CNN
+	1    1950 8400
+	0    -1   -1   0
+$EndComp
+Wire Wire Line
+	2100 8400 1950 8400
+Text GLabel 2900 8300 2    60   Input ~ 0
+RA_CS
+$Comp
+L LM1117-3.3 U?
+U 1 1 58BB7D07
+P 4650 8350
+F 0 "U?" H 4650 8717 50  0000 C CNN
+F 1 "LM1117-3.3" H 4650 8626 50  0000 C CNN
+F 2 "" H -525 -250 50  0001 C CNN
+F 3 "" H -525 -250 50  0001 C CNN
+	1    4650 8350
+	1    0    0    -1
+$EndComp
+$Comp
+L +5V #PWR?
+U 1 1 58BB9559
+P 4275 8250
+F 0 "#PWR?" H 4275 8100 50  0001 C CNN
+F 1 "+5V" H 4290 8423 50  0000 C CNN
+F 2 "" H 4275 8250 50  0000 C CNN
+F 3 "" H 4275 8250 50  0000 C CNN
+	1    4275 8250
+	1    0    0    -1
+$EndComp
+$Comp
+L GND #PWR?
+U 1 1 58BB9ED3
+P 4650 8700
+F 0 "#PWR?" H 4650 8450 50  0001 C CNN
+F 1 "GND" H 4655 8527 50  0000 C CNN
+F 2 "" H 4650 8700 50  0000 C CNN
+F 3 "" H 4650 8700 50  0000 C CNN
+	1    4650 8700
+	1    0    0    -1
+$EndComp
+$Comp
+L C_Small C?
+U 1 1 58BBAB8E
+P 1975 8300
+F 0 "C?" H 1625 8375 50  0000 L CNN
+F 1 "10uF" H 1625 8300 50  0000 L CNN
+F 2 "lib:C_0603" H 1975 8300 50  0001 C CNN
+F 3 "" H 1975 8300 50  0000 C CNN
+	1    1975 8300
+	1    0    0    -1
+$EndComp
+$Comp
+L +3V3 #PWR?
+U 1 1 58BBB9EB
+P 5025 8250
+F 0 "#PWR?" H 5075 8300 50  0001 C CNN
+F 1 "+3V3" H 5040 8423 50  0000 C CNN
+F 2 "" H -2750 1250 50  0000 C CNN
+F 3 "" H -2750 1250 50  0000 C CNN
+	1    5025 8250
+	1    0    0    -1
+$EndComp
+$Comp
+L C_Small C?
+U 1 1 58BBCE7C
+P 4275 8500
+F 0 "C?" H 4367 8546 50  0000 L CNN
+F 1 "10uF" H 4367 8455 50  0000 L CNN
+F 2 "lib:C_0603" H 4275 8500 50  0001 C CNN
+F 3 "" H 4275 8500 50  0000 C CNN
+	1    4275 8500
+	1    0    0    -1
+$EndComp
+Wire Wire Line
+	4275 8250 4275 8400
+Wire Wire Line
+	4275 8350 4350 8350
+Connection ~ 4275 8350
+Wire Wire Line
+	4650 8650 4650 8700
+Wire Wire Line
+	4275 8600 4275 8675
+Wire Wire Line
+	4275 8675 4650 8675
+Connection ~ 4650 8675
+Wire Wire Line
+	4950 8350 5025 8350
+Wire Wire Line
+	5025 8350 5025 8250
 $EndSCHEMATC

Commit message: 3.3V ???
Connections:
- net RA_CS: now also SHIELD1.10
- net RA_MISO: now also SHIELD1.12
- net RA_MOSI: now also SHIELD1.11
- net RA_SCK: now also SHIELD1.13
Other:
- note added: "???"
Changed lines of the file:
@@
 L GND #PWR24
 U 1 1 58AD4688
-P 8400 1425
-F 0 "#PWR24" H 8400 1175 50  0001 C CNN
-F 1 "GND" H 8405 1252 50  0000 C CNN
-F 2 "" H 8400 1425 50  0000 C CNN
-F 3 "" H 8400 1425 50  0000 C CNN
-	1    8400 1425
-	1    0    0    -1
+P 8400 1375
+F 0 "#PWR24" H 8400 1125 50  0001 C CNN
+F 1 "GND" H 8405 1202 50  0000 C CNN
+F 2 "" H 8400 1375 50  0000 C CNN
+F 3 "" H 8400 1375 50  0000 C CNN
+	1    8400 1375
+	0    -1   -1   0
 $EndComp
 Connection ~ 3750 6300
 Connection ~ 3250 7400
 Wire Wire Line
-	3750 7100 3750 7425
+	3750 7100 3750 7400
+Wire Wire Line
+	3750 7400 3750 7425
 Connection ~ 2750 7400
 Wire Wire Line
@@
 Connection ~ 1100 7400
 Wire Wire Line
-	1100 7250 1100 7450
+	1100 7250 1100 7400
+Wire Wire Line
+	1100 7400 1100 7450
 Wire Wire Line
 	800  5900 1200 5900
 Connection ~ 6800 3725
 Wire Wire Line
-	6750 3725 6900 3725
+	6750 3725 6800 3725
+Wire Wire Line
+	6800 3725 6900 3725
 Wire Wire Line
 	7100 3725 7150 3725
@@
 	10250 1750 10450 1750
 Wire Wire Line
-	10450 1550 10450 1900
+	10450 1550 10450 1750
+Wire Wire Line
+	10450 1750 10450 1900
 Wire Wire Line
 	10450 950  10450 1150
@@
 	6500 5850 6500 6200
 Wire Wire Line
-	800  5700 800  6300
+	800  5700 800  5800
+Wire Wire Line
+	800  5800 800  5900
+Wire Wire Line
+	800  5900 800  6300
 Connection ~ 800  5900
 Wire Wire Line
 	800  6500 800  7400
 Wire Wire Line
-	2550 5900 2550 6900
-Wire Wire Line
-	2300 6350 2950 6350
+	2550 5900 2550 6350
+Wire Wire Line
+	2550 6350 2550 6900
+Wire Wire Line
+	2300 6350 2550 6350
+Wire Wire Line
+	2550 6350 2950 6350
 Connection ~ 2550 6350
 Wire Wire Line
@@
 Connection ~ 2750 6550
 Wire Wire Line
-	3250 6350 3250 6800
+	3250 6350 3250 6550
+Wire Wire Line
+	3250 6550 3250 6800
 Wire Wire Line
 	1900 6800 1900 6850
 Wire Wire Line
-	3750 6350 3150 6350
-Wire Wire Line
-	3750 6090 3750 6700
+	3750 6350 3250 6350
+Wire Wire Line
+	3250 6350 3150 6350
+Wire Wire Line
+	3750 6090 3750 6300
+Wire Wire Line
+	3750 6300 3750 6350
+Wire Wire Line
+	3750 6350 3750 6700
 Connection ~ 3750 6350
 Wire Wire Line
@@
 Connection ~ 3750 7400
 Wire Wire Line
-	2300 6550 2900 6550
+	2300 6550 2750 6550
+Wire Wire Line
+	2750 6550 2900 6550
 Connection ~ 3250 6350
 Connection ~ 3250 6550
 Wire Wire Line
-	800  7400 3750 7400
-Wire Wire Line
-	4750 7050 4750 7150
-Wire Wire Line
-	4750 7350 4750 7450
-Wire Wire Line
-	4750 7100 6200 7100
+	800  7400 1100 7400
+Wire Wire Line
+	1100 7400 1700 7400
+Wire Wire Line
+	1700 7400 1900 7400
+Wire Wire Line
+	1900 7400 2550 7400
+Wire Wire Line
+	2550 7400 2750 7400
+Wire Wire Line
+	2750 7400 3250 7400
+Wire Wire Line
+	3250 7400 3750 7400
+Wire Wire Line
+	4750 7050 4750 7100
+Wire Wire Line
+	4750 7100 4750 7150
+Wire Wire Line
+	4750 7350 4750 7400
+Wire Wire Line
+	4750 7400 4750 7450
+Wire Wire Line
+	4750 7100 5150 7100
+Wire Wire Line
+	5150 7100 5500 7100
+Wire Wire Line
+	5500 7100 5850 7100
+Wire Wire Line
+	5850 7100 6200 7100
 Wire Wire Line
 	6200 7100 6200 7150
@@
 	6200 7400 6200 7350
 Wire Wire Line
-	4750 7400 6200 7400
+	4750 7400 5150 7400
+Wire Wire Line
+	5150 7400 5500 7400
+Wire Wire Line
+	5500 7400 5850 7400
+Wire Wire Line
+	5850 7400 6200 7400
 Connection ~ 4750 7400
 Wire Wire Line
@@
 Connection ~ 5850 7400
 Wire Wire Line
-	7400 6175 7400 6225
+	7400 6175 7400 6200
+Wire Wire Line
+	7400 6200 7400 6225
 Wire Wire Line
 	6500 6200 7400 6200
 Connection ~ 7400 6200
 Wire Wire Line
-	6200 1975 6200 2100
+	6200 1975 6200 2075
+Wire Wire Line
+	6200 2075 6200 2100
 Wire Wire Line
 	6200 2075 6400 2075
@@
 	1325 5800 1325 5750
 Wire Wire Line
-	800  5800 1325 5800
+	800  5800 1000 5800
+Wire Wire Line
+	1000 5800 1325 5800
 Connection ~ 800  5800
 Wire Wire Line
@@
 	10100 4700 10450 4700
 Wire Wire Line
-	10450 4650 10450 4750
+	10450 4650 10450 4700
+Wire Wire Line
+	10450 4700 10450 4750
 Connection ~ 10450 4700
 Wire Wire Line
-	10050 4450 10150 4450
+	10050 4450 10100 4450
+Wire Wire Line
+	10100 4450 10150 4450
 Wire Wire Line
 	10100 4500 10100 4450
@@
 	10100 6100 10450 6100
 Wire Wire Line
-	10450 6050 10450 6150
+	10450 6050 10450 6100
+Wire Wire Line
+	10450 6100 10450 6150
 Connection ~ 10450 6100
 Wire Wire Line
-	10050 5850 10150 5850
+	10050 5850 10100 5850
+Wire Wire Line
+	10100 5850 10150 5850
 Wire Wire Line
 	10100 5900 10100 5850
@@
 	10250 3100 10450 3100
 Wire Wire Line
-	10450 2900 10450 3250
+	10450 2900 10450 3100
+Wire Wire Line
+	10450 3100 10450 3250
 Wire Wire Line
 	10450 2300 10450 2500
@@
 	8300 1375 8400 1375
 Wire Wire Line
-	8400 1375 8400 1425
-Wire Wire Line
 	7750 5300 7850 5300
 Wire Wire Line
 	7500 5575 7500 5450
 Wire Wire Line
-	8150 5250 8150 5550
+	8150 5250 8150 5300
+Wire Wire Line
+	8150 5300 8150 5450
+Wire Wire Line
+	8150 5450 8150 5550
 Wire Wire Line
 	7500 5450 8150 5450
@@
 $EndComp
 Wire Wire Line
-	3400 1400 3400 1500
-Wire Wire Line
-	3400 1450 3800 1450
+	3400 1400 3400 1450
+Wire Wire Line
+	3400 1450 3400 1500
+Wire Wire Line
+	3400 1450 3500 1450
+Wire Wire Line
+	3500 1450 3600 1450
+Wire Wire Line
+	3600 1450 3700 1450
+Wire Wire Line
+	3700 1450 3800 1450
 Wire Wire Line
 	3800 1450 3800 1500
@@
 Connection ~ 3400 1450
 Wire Wire Line
-	4000 1400 4000 1500
+	4000 1400 4000 1450
+Wire Wire Line
+	4000 1450 4000 1500
 Connection ~ 4000 1450
 Wire Wire Line
 	4100 1450 4100 1500
 Wire Wire Line
-	4500 1400 4500 1500
+	4500 1400 4500 1450
+Wire Wire Line
+	4500 1450 4500 1500
 Connection ~ 4500 1450
 Wire Wire Line
-	4200 1400 4200 1500
-Wire Wire Line
-	4200 1450 4400 1450
+	4200 1400 4200 1450
+Wire Wire Line
+	4200 1450 4200 1500
+Wire Wire Line
+	4200 1450 4300 1450
+Wire Wire Line
+	4300 1450 4400 1450
 Wire Wire Line
 	4300 1450 4300 1500
@@
 	950  3600 1000 3600
 Wire Wire Line
-	1600 3600 1750 3600
+	1600 3600 1700 3600
+Wire Wire Line
+	1700 3600 1750 3600
 Wire Wire Line
 	2050 3600 2300 3600
@@
 	950  2100 1000 2100
 Wire Wire Line
-	1600 2100 2300 2100
+	1600 2100 1700 2100
+Wire Wire Line
+	1700 2100 2300 2100
 Wire Wire Line
 	1650 1750 1700 1750
@@
 	7000 5100 6500 5100
 Wire Wire Line
-	6500 5000 6500 5650
+	6500 5000 6500 5100
+Wire Wire Line
+	6500 5100 6500 5575
+Wire Wire Line
+	6500 5575 6500 5650
 Wire Wire Line
 	6750 5200 6600 5200
 Wire Wire Line
-	6600 5000 6600 5525
+	6600 5000 6600 5200
+Wire Wire Line
+	6600 5200 6600 5525
 Wire Wire Line
 	6700 5300 6750 5300
 Wire Wire Line
-	6700 5000 6700 5475
+	6700 5000 6700 5300
+Wire Wire Line
+	6700 5300 6700 5475
 Connection ~ 6500 5100
 Wire Wire Line
@@
 $EndComp
 Wire Wire Line
-	1950 8200 2100 8200
+	1950 8200 2050 8200
+Wire Wire Line
+	2050 8200 2100 8200
 Wire Wire Line
 	2100 8300 2050 8300
@@
 $EndComp
 Wire Wire Line
-	4275 8250 4275 8400
+	4275 8250 4275 8350
+Wire Wire Line
+	4275 8350 4275 8400
 Wire Wire Line
 	4275 8350 4350 8350
 Connection ~ 4275 8350
 Wire Wire Line
-	4650 8650 4650 8700
+	4650 8650 4650 8675
+Wire Wire Line
+	4650 8675 4650 8700
 Wire Wire Line
 	4275 8600 4275 8675
@@
 Wire Wire Line
 	5025 8350 5025 8250
+Text GLabel 8300 1675 2    60   Input ~ 0
+RA_MOSI
+Text GLabel 8300 1575 2    60   Input ~ 0
+RA_MISO
+Text GLabel 8300 1475 2    60   Input ~ 0
+RA_SCK
+Text GLabel 8300 1775 2    60   Input ~ 0
+RA_CS
+Text Notes 5150 8300 0    118  ~ 24
+???
 $EndSCHEMATC
