File: cellular.kicad_pcb (KiCad board)
At the start: 2 copper layers, 68.6 x 53.3 mm, 55 parts, among them P3 Chip anten, Q1 2SC1815, Q2 2SC1815, Q3 2SC1815, Q4 2SC1815, SW1 SW_PUSH, SW2 SW_PUSH, U1 MP2365DN, U2 SIM800H, U6 SIM HOLD - PPSS-6P

Commit message: replaced components
Parts:
- moved R27 20.9 mm to (141.6, 117.2)
- moved R24 20.9 mm to (139.7, 117.2)
- moved R11 18.8 mm to (141.6, 121.3)
- moved R6 18.8 mm to (139.7, 121.3)
- moved D4 17.9 mm to (141.9, 113.8)
- moved Q1 16.3 mm to (144.8, 117.5), turned to 90 degrees
- moved C31 15.2 mm to (147.1, 129.2), turned to 270 degrees
- moved Q3 13.6 mm to (144.8, 121.3), turned to 90 degrees
- moved C32 11.8 mm to (143.5, 129.9), turned to 270 degrees
- moved D1 11.1 mm to (150.7, 128.9), turned to 270 degrees
- moved R13 9.78 mm to (141.6, 125.2), turned to 270 degrees
- moved C33 9.59 mm to (141.6, 129.9), turned to 270 degrees
- moved R12 9.40 mm to (139.7, 125.2)
- moved C34 7.66 mm to (139.7, 129.9), turned to 270 degrees
- moved D6 7.52 mm to (150.9, 123.6), turned to 270 degrees
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
Commit message: wired power supply
Parts:
- moved C2 0.57 mm to (134.0, 99.8), turned to 270 degrees
Routing:
- net GND: track 0.00 -> 81.8 mm, vias 0 -> 27
- net VDD: track 0.00 -> 39.8 mm, vias 0 -> 2
- net +5V: track 0.00 -> 12.3 mm
- net Net-(C12-Pad1): track 0.00 -> 12.1 mm
- net Net-(C10-Pad1): track 0.00 -> 8.59 mm
- net Net-(R8-Pad1): track 0.00 -> 7.97 mm
- net Net-(D6-Pad1): track 0.00 -> 2.42 mm
- net Net-(C12-Pad2): track 0.00 -> 2.38 mm
- net Net-(C4-Pad1): track 0.00 -> 2.31 mm
- added copper zone on B.Cu, net GND
Other:
- net class Default: clearance 0.2 -> 0.25
- rule trace_clearance: 0.2 -> 0.25
- rule trace_min: 0.2 -> 0.25
- rule via_min_drill: 0.3 -> 0.2
- rule via_min_size: 0.4 -> 0.2
