File: cellular.kicad_pcb (KiCad board)
At the start: 2 copper layers, 68.6 x 53.3 mm, 55 parts, among them P3 Chip anten, Q1 2SC1815, Q2 2SC1815, Q3 2SC1815, Q4 2SC1815, SW1 SW_PUSH, SW2 SW_PUSH, U1 MP2365DN, U2 SIM800H, U6 SIM HOLD - PPSS-6P

Commit message: replace sim800L by sim800
Parts:
- removed P3: Chip anten, lib:point_test
- U2: value SIM800H -> SIM800; footprint lib:SIM800H -> lib:SIM800
- moved D1 48.5 mm to (103.4, 118.4), turned to 180 degrees
- moved D3 47.3 mm to (104.4, 105.9), turned to 180 degrees
- moved R10 46.6 mm to (104.4, 107.8), turned to 0 degrees
- moved C31 45.5 mm to (103.8, 115.3), turned to 180 degrees
- moved C32 42.7 mm to (104.4, 112.9), turned to 180 degrees
- moved C33 41.6 mm to (104.4, 111.3), turned to 180 degrees
- moved U6 41.5 mm to (152.5, 115.4), turned to 90 degrees
- moved C34 40.7 mm to (104.4, 109.6), turned to 180 degrees
- moved ANT1 38.2 mm to (101.6, 123.2), turned to 0 degrees
- moved R26 31.0 mm to (104.9, 123.2), turned to 270 degrees
- moved C29 30.6 mm to (146.7, 115.8), turned to 180 degrees
- moved Q1 30.3 mm to (123.6, 139.1)
- moved R24 30.2 mm to (118.9, 139.1)
- moved R27 30.1 mm to (120.9, 139.1)
- moved D5 28.7 mm to (146.7, 113.2), turned to 90 degrees
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Connections:
- SHIELD1 pad 2: SIM800L_RI -> SIM800L_DTR
- SHIELD1 pad 3: SIM800L_DTR -> SIM800L_RI
- U2 pad 1: VDD -> SIM800L_PWRKEY
- U2 pad 10: (no net) -> Net-(R1-Pad2)
- U2 pad 14: SIM800L_DATA -> (no net)
- U2 pad 15: SIM800L_RST -> (no net)
- U2 pad 16: SIM800L_VDD -> Net-(D4-Pad2)
- U2 pad 17: (no net) -> GND
- U2 pad 18: (no net) -> GND
- U2 pad 26: (no net) -> Net-(C1-Pad1)
- U2 pad 3: (no net) -> Net-(R5-Pad2)
- U2 pad 30: (no net) -> SIM800L_VDD
- U2 pad 31: Net-(R1-Pad2) -> SIM800L_DATA
- U2 pad 32: Net-(R2-Pad2) -> SIM800L_CLK
- U2 pad 33: (no net) -> SIM800L_RST
- U2 pad 35: GND -> (no net)
- U2 pad 37: GND -> (no net)
- U2 pad 38: GND -> (no net)
- U2 pad 4: SIM800L_STATUS -> Net-(R4-Pad2)
- U2 pad 40: GSM_ANT -> (no net)
- U2 pad 41: GND -> (no net)
- U2 pad 42: VDD -> (no net)
- U2 pad 43: GND -> (no net)
- U2 pad 44: GND -> (no net)
- U2 pad 48: SIM800L_PWRKEY -> (no net)
- U2 pad 49: Net-(D4-Pad2) -> (no net)
- U2 pad 5: (no net) -> Net-(R3-Pad2)
- U2 pad 52: (no net) -> SIM800L_NETLIGHT
- U2 pad 54: (no net) -> GND
- U2 pad 55: SIM800L_CLK -> VDD
- U2 pad 56: Net-(C1-Pad1) -> VDD
- U2 pad 57: (no net) -> VDD
- U2 pad 59: (no net) -> GND
- U2 pad 6: GND -> (no net)
- U2 pad 60: (no net) -> GSM_ANT
- U2 pad 61: (no net) -> GND
- U2 pad 62: (no net) -> GND
- U2 pad 63: (no net) -> GND
- U2 pad 64: SIM800L_NETLIGHT -> GND
- U2 pad 65: (no net) -> GND
- U2 pad 66: (no net) -> SIM800L_STATUS
- U2 pad 67: GND -> (no net)
- U2 pad 68: Net-(R4-Pad2) -> (no net)
- U2 pad 8: GND -> (no net)
- U2 pad 9: (no net) -> Net-(R2-Pad2)
Routing:
- net GND: track 125.3 -> 64.3 mm, vias 48 -> 35
- net PWRKEY: track 40.8 -> 4.97 mm, vias 2 -> 0
- net SIM800L_NETLIGHT: track 6.02 -> 41.5 mm, vias 1 -> 2
- net SIM800L_STATUS: track 4.95 -> 30.4 mm, vias 1 -> 0
- net RESET: track 33.9 -> 9.97 mm, vias 2 -> 0
- net SIM800L_RESET: track 45.3 -> 28.4 mm, vias 2 -> 0
- net Net-(R1-Pad2): track 4.61 -> 21.2 mm
- net Net-(R2-Pad2): track 4.40 -> 18.0 mm
- net SIM800L_RI: track 19.5 -> 6.04 mm
- net SIM800L_DCD: track 18.9 -> 5.40 mm
- net SIM800L_TXD: track 19.9 -> 7.30 mm
- net SIM800L_DTR: track 19.2 -> 6.72 mm
- net SIM800L_RXD: track 20.3 -> 8.19 mm
- net SIM800L_PWRKEY: track 47.3 -> 56.7 mm, vias 1 -> 2
- net VDD: track 96.2 -> 87.6 mm
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
Commit message: moved sim socket, added SMA connector hold, added logos
Parts:
- added G***: LOGO, lib:logo-iotmakervn_7.5x5, F.Cu at (146.2, 134.9)
- added G***: LOGO, lib:logo_openhardware_5x5mm, F.Cu at (161.7, 128.3)
- added G***: LOGO, lib:logo_cc-bby-sa_14.1x5mm, F.Cu at (149.5, 128.3)
- moved D2 28.1 mm to (136.9, 101.1)
- moved C28 7.49 mm to (144.3, 120.7)
- moved D5 7.49 mm to (146.7, 120.7)
- moved R18 7.49 mm to (146.7, 118.0)
- moved U6 7.49 mm to (152.5, 122.9)
- moved C29 7.49 mm to (146.7, 123.3)
- moved R19 7.49 mm to (146.7, 114.7)
- moved R20 7.49 mm to (146.7, 116.3)
- moved D3 3.69 mm to (101.6, 108.3), turned to 90 degrees
Routing:
- net SIM800L_VDD: track 25.2 -> 31.0 mm
- net SIM800L_DATA: track 25.8 -> 22.4 mm
- net SIM800L_CLK: track 23.4 -> 20.3 mm
- net VDD: track 87.6 -> 88.3 mm
- net SIM800L_RST: track 21.9 -> 21.2 mm
- net GND: vias 35 -> 36
Other:
- outline, holes or cut-outs redrawn
- board text added: "iotmaker.vn"

Commit message: clear ruler, add 3D model SIM800, sim holder
Parts:
- U6: value SIM HOLD - PPSS-6P -> MICRO SIM
Changed lines of the file:
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@@
     (area 98.374999 92.659999 167.055001 146.100001)
     (thickness 1.6)
-    (drawings 21)
+    (drawings 16)
     (tracks 351)
     (zones 0)
@@
     (pad 67 smd oval (at -7 -12.4) (size 2 0.6) (layers F.Cu F.Paste F.Mask))
     (pad 68 smd oval (at -8 -12.4) (size 2 0.6) (layers F.Cu F.Paste F.Mask))
+    (model ${KIPRJMOD}/lib/SIM800.IGS
+      (at (xyz 0 0 0))
+      (scale (xyz 1 1 1))
+      (rotate (xyz 90 180 180))
+    )
   )
   (module lib:Micro_SIM_6P_PUSH_SKM01 (layer F.Cu)
@@
       (effects (font (size 1.2065 1.2065) (thickness 0.1016)) (justify left bottom))
     )
-    (fp_text value "SIM HOLD - PPSS-6P" (at 18.542 13.97 180) (layer F.SilkS)
+    (fp_text value "MICRO SIM" (at 17.907 -3.429 180) (layer F.SilkS)
       (effects (font (size 1.2065 1.2065) (thickness 0.1016)) (justify left bottom))
     )
@@
     (pad 3 smd rect (at 7.91 -2.45 180) (size 1.5 0.75) (layers F.Cu F.Paste F.Mask)
       (net 44 "Net-(R19-Pad1)"))
+    (model ${KIPRJMOD}/lib/micro-sim-holder.IGS
+      (at (xyz 0.00984251968503937 -0.5590551181102362 0))
+      (scale (xyz 1 1 1))
+      (rotate (xyz -90 0 0))
+    )
   )
   (module lib:logo-iotmakervn_7.5x5 (layer F.Cu)
@@
   (gr_circle (center 107.442 102.235) (end 104.14 102.108) (layer Edge.Cuts) (width 0.1))
   (gr_circle (center 107.442 102.235) (end 107.442 98.985) (layer F.SilkS) (width 0.2))
-  (gr_line (start 113.919 180.467) (end 160.782 180.467) (angle 90) (layer F.SilkS) (width 0.2))
-  (gr_line (start 131.699 130.937) (end 178.562 130.937) (angle 90) (layer F.SilkS) (width 0.2))
-  (gr_line (start 105.41 95.123) (end 105.41 143.383) (angle 90) (layer F.SilkS) (width 0.2))
   (gr_line (start 100.965 92.71) (end 167.005 92.71) (angle 90) (layer Edge.Cuts) (width 0.1))
   (gr_line (start 100.965 95.25) (end 100.965 92.71) (angle 90) (layer Edge.Cuts) (width 0.1))
@@
   (gr_line (start 167.005 146.05) (end 102.235 146.05) (angle 90) (layer Edge.Cuts) (width 0.1))
   (gr_line (start 167.005 92.71) (end 167.005 146.05) (angle 90) (layer Edge.Cuts) (width 0.1))
-  (gr_line (start 138.557 101.346) (end 138.557 149.606) (angle 90) (layer F.SilkS) (width 0.2))
-  (gr_line (start 101.219 104.902) (end 148.082 104.902) (angle 90) (layer F.SilkS) (width 0.2))
   (segment (start 104.902 123.989999) (end 104.852 123.989999) (width 0.4064) (layer F.Cu) (net 1))
   (segment (start 104.852 123.989999) (end 103.619999 125.222) (width 0.4064) (layer F.Cu) (net 1))

Commit message: change design rules, moved via out of footprint, elliptical board egdes
Parts:
- moved Q4 0.28 mm to (137.3, 128.1)
- turned R7 to 270 degrees
Routing:
- net GND: track 64.3 -> 100.4 mm, vias 36 -> 17
- net VDD: track 88.3 -> 97.4 mm
- net Net-(D4-Pad2): track 15.4 -> 19.8 mm
- net SIM800L_DATA: track 22.4 -> 26.4 mm
- net SIM800L_VDD: track 31.0 -> 33.6 mm
- net SIM800L_CLK: track 20.3 -> 21.6 mm
- net SIM800L_PWRKEY: track 56.7 -> 56.1 mm
Other:
- outline, holes or cut-outs redrawn
- net class Default: via_dia 0.8 -> 1.1
- rule via_min_size: 0.2 -> 1.1

Commit message: swap TX RX, place component name
Parts:
- removed G***: LOGO, lib:logo-iotmakervn_7.5x5
- removed G***: LOGO, lib:logo_openhardware_5x5mm
- removed G***: LOGO, lib:logo_cc-bby-sa_14.1x5mm
- removed SW1, SW2: SW_PUSH, lib:SW_SPST_B3U-1000P-B
- added PWR1: SW_PUSH, lib:SW_SPST_B3U-1000P-B, F.Cu at (163.1, 141.4)
- added RST1: SW_PUSH, lib:SW_SPST_B3U-1000P-B, F.Cu at (157.7, 141.4)
- U6: value MICRO SIM -> SIM HOLD - PPSS-6P
- moved R1 1.91 mm to (111.1, 139.1)
- moved R2 1.91 mm to (109.2, 139.1)
Connections:
- C28 pad 1: Net-(C28-Pad1) -> SIM800L_VDD
- D5 pad 6: Net-(C28-Pad1) -> SIM800L_VDD
- SHIELD1 pad 0: SIM800L_RXD -> SIM800L_TXD
- SHIELD1 pad 1: SIM800L_TXD -> SIM800L_RXD
Routing:
- net SIM800L_VDD: track 33.6 -> 40.8 mm
- net Net-(R1-Pad2): track 21.2 -> 19.0 mm, vias 0 -> 2
- net Net-(R2-Pad2): track 18.0 -> 19.9 mm
- net Net-(C28-Pad1): track 1.83 -> 0.00 mm
- net SIM800L_RXD: track 8.19 -> 7.31 mm
- net SIM800L_TXD: track 7.30 -> 8.15 mm

Commit message: pinmap
Parts:
- added G***: LOGO, lib:logo_cc-bby-sa_14.1x5mm, F.Cu at (149.2, 128.3)
- added G***: LOGO, lib:logo-iotmakervn_7.5x5, F.Cu at (145.9, 134.9)
- added VAL**: oshw_logo_500, lib:logo5, F.Cu at (161.9, 128.3)
Other:
- board text added: "-------------"
- board text added: "----------------"
- board text added: "0"
- board text added: "0 1 2 3"
- board text added: "0 1 2 3 4 5 6"
- board text added: "1"
- board text added: "2"
- board text added: "3"
- board text added: "4"
- board text added: "4 5 6"
- board text added: "5"
- board text added: "6"
- board text added: "CS0"
- board text added: "DCD"
- board text added: "DTR"
- board text added: "ESP32"
- board text added: "GPIO00"
- board text added: "GPIO02"
- board text added: "GPIO16"
- board text added: "MISO"
- board text added: "PWR"
- board text added: "RESET"
- board text added: "RI"
- board text added: "RX"
- board text added: "SIM800"
- board text added: "TX"
- board text added: "|"
- board text added: "| ESP32"
- board text added: "| RX | TX | GPIO16 | GPIO00 | GPIO02 | CS0 | MISO"
- board text added: "| SIM800"
- board text added: "| TX | RX | DTR | RI | DCD | PWRKEY | RESET"
- board text added: "| | |"
- board text added: "| | | |"
- board text added: "| | | | | | |"
