File: cellular.kicad_pcb (KiCad board)
At the start: 2 copper layers, 37 parts, among them P3 Chip anten, Q1 2SC1815, Q2 2SC1815, U1 MP2365DN, U2 SIM800H, U6 SIM HOLD - PPSS-6P

Commit message: tets ignore
Parts:
- added SHIELD1: ARDUINO_SHIELD, arduino_shields:ARDUINO_SHIELD_2, F.Cu at (117.6, 79.9)
Changed lines of the file:
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@@
 (kicad_pcb (version 20170123) (host pcbnew no-vcs-found-7647~57~ubuntu14.04.1)
   (general
-    (links 58)
-    (no_connects 58)
+    (links 61)
+    (no_connects 61)
     (area 0 0 0 0)
     (thickness 1.6)
@@
     (tracks 0)
     (zones 0)
-    (modules 37)
+    (modules 38)
     (nets 24)
   )
@@
     (pad Z5 smd rect (at -5.61 -0.225) (size 1.88 0.5) (layers F.Cu F.Paste F.Mask))
   )
+  (module arduino_shields:ARDUINO_SHIELD_2 (layer F.Cu)
+    (at 117.583005 79.85948)
+    (fp_text reference SHIELD1 (at 5.715 -57.15) (layer F.SilkS)
+      (effects (font (thickness 0.3048)))
+    )
+    (fp_text value ARDUINO_SHIELD (at 10.16 -54.61) (layer F.SilkS) hide
+      (effects (font (thickness 0.3048)))
+    )
+    (fp_line (start 0 -44.45) (end 10.16 -44.45) (layer Dwgs.User) (width 0.381))
+    (fp_line (start 10.16 -44.45) (end 10.16 -31.75) (layer Dwgs.User) (width 0.381))
+    (fp_line (start 10.16 -31.75) (end 0 -31.75) (layer Dwgs.User) (width 0.381))
+    (fp_line (start 12.7 -4.318) (end 0 -4.318) (layer Dwgs.User) (width 0.381))
+    (fp_line (start 0 -12.7) (end 12.7 -12.7) (layer Dwgs.User) (width 0.381))
+    (fp_line (start 12.7 -12.7) (end 12.7 -4.572) (layer Dwgs.User) (width 0.381))
+    (fp_circle (center 13.97 -2.54) (end 16.002 -1.524) (layer Dwgs.User) (width 0.381))
+    (fp_circle (center 15.24 -50.8) (end 16.764 -49.276) (layer Dwgs.User) (width 0.381))
+    (fp_circle (center 66.04 -7.62) (end 67.31 -6.096) (layer Dwgs.User) (width 0.381))
+    (fp_circle (center 66.04 -35.56) (end 67.31 -34.036) (layer Dwgs.User) (width 0.381))
+    (fp_line (start 66.04 -40.64) (end 66.04 -52.07) (layer Dwgs.User) (width 0.381))
+    (fp_line (start 66.04 -52.07) (end 64.77 -53.34) (layer Dwgs.User) (width 0.381))
+    (fp_line (start 64.77 -53.34) (end 0 -53.34) (layer Dwgs.User) (width 0.381))
+    (fp_line (start 66.04 0) (end 0 0) (layer Dwgs.User) (width 0.381))
+    (fp_line (start 0 0) (end 0 -53.34) (layer Dwgs.User) (width 0.381))
+    (fp_line (start 66.04 -40.64) (end 68.58 -38.1) (layer Dwgs.User) (width 0.381))
+    (fp_line (start 68.58 -38.1) (end 68.58 -5.08) (layer Dwgs.User) (width 0.381))
+    (fp_line (start 68.58 -5.08) (end 66.04 -2.54) (layer Dwgs.User) (width 0.381))
+    (fp_line (start 66.04 -2.54) (end 66.04 0) (layer Dwgs.User) (width 0.381))
+    (pad AD5 thru_hole oval (at 63.5 -2.54 90) (size 2.54 1.524) (drill 0.8128) (layers *.Cu *.Mask F.SilkS))
+    (pad AD4 thru_hole oval (at 60.96 -2.54 90) (size 2.54 1.524) (drill 0.8128) (layers *.Cu *.Mask F.SilkS))
+    (pad AD3 thru_hole oval (at 58.42 -2.54 90) (size 2.54 1.524) (drill 0.8128) (layers *.Cu *.Mask F.SilkS))
+    (pad AD0 thru_hole oval (at 50.8 -2.54 90) (size 2.54 1.524) (drill 0.8128) (layers *.Cu *.Mask F.SilkS))
+    (pad AD1 thru_hole oval (at 53.34 -2.54 90) (size 2.54 1.524) (drill 0.8128) (layers *.Cu *.Mask F.SilkS))
+    (pad AD2 thru_hole oval (at 55.88 -2.54 90) (size 2.54 1.524) (drill 0.8128) (layers *.Cu *.Mask F.SilkS))
+    (pad V_IN thru_hole oval (at 45.72 -2.54 90) (size 2.54 1.524) (drill 0.8128) (layers *.Cu *.Mask F.SilkS))
+    (pad GND2 thru_hole oval (at 43.18 -2.54 90) (size 2.54 1.524) (drill 0.8128) (layers *.Cu *.Mask F.SilkS)
+      (net 3 GND))
+    (pad GND1 thru_hole oval (at 40.64 -2.54 90) (size 2.54 1.524) (drill 0.8128) (layers *.Cu *.Mask F.SilkS)
+      (net 3 GND))
+    (pad 3V3 thru_hole oval (at 35.56 -2.54 90) (size 2.54 1.524) (drill 0.8128) (layers *.Cu *.Mask F.SilkS))
+    (pad RST thru_hole oval (at 33.02 -2.54 90) (size 2.54 1.524) (drill 0.8128) (layers *.Cu *.Mask F.SilkS))
+    (pad 0 thru_hole oval (at 63.5 -50.8 90) (size 2.54 1.524) (drill 0.8128) (layers *.Cu *.Mask F.SilkS))
+    (pad 1 thru_hole oval (at 60.96 -50.8 90) (size 2.54 1.524) (drill 0.8128) (layers *.Cu *.Mask F.SilkS))
+    (pad 2 thru_hole oval (at 58.42 -50.8 90) (size 2.54 1.524) (drill 0.8128) (layers *.Cu *.Mask F.SilkS))
+    (pad 3 thru_hole oval (at 55.88 -50.8 90) (size 2.54 1.524) (drill 0.8128) (layers *.Cu *.Mask F.SilkS))
+    (pad 4 thru_hole oval (at 53.34 -50.8 90) (size 2.54 1.524) (drill 0.8128) (layers *.Cu *.Mask F.SilkS))
+    (pad 5 thru_hole oval (at 50.8 -50.8 90) (size 2.54 1.524) (drill 0.8128) (layers *.Cu *.Mask F.SilkS))
+    (pad 6 thru_hole oval (at 48.26 -50.8 90) (size 2.54 1.524) (drill 0.8128) (layers *.Cu *.Mask F.SilkS))
+    (pad 7 thru_hole oval (at 45.72 -50.8 90) (size 2.54 1.524) (drill 0.8128) (layers *.Cu *.Mask F.SilkS))
+    (pad 8 thru_hole oval (at 41.656 -50.8 90) (size 2.54 1.524) (drill 0.8128) (layers *.Cu *.Mask F.SilkS))
+    (pad 9 thru_hole oval (at 39.116 -50.8 90) (size 2.54 1.524) (drill 0.8128) (layers *.Cu *.Mask F.SilkS))
+    (pad 10 thru_hole oval (at 36.576 -50.8 90) (size 2.54 1.524) (drill 0.8128) (layers *.Cu *.Mask F.SilkS))
+    (pad 11 thru_hole oval (at 34.036 -50.8 90) (size 2.54 1.524) (drill 0.8128) (layers *.Cu *.Mask F.SilkS))
+    (pad 12 thru_hole oval (at 31.496 -50.8 90) (size 2.54 1.524) (drill 0.8128) (layers *.Cu *.Mask F.SilkS))
+    (pad 13 thru_hole oval (at 28.956 -50.8 90) (size 2.54 1.524) (drill 0.8128) (layers *.Cu *.Mask F.SilkS))
+    (pad GND3 thru_hole oval (at 26.416 -50.8 90) (size 2.54 1.524) (drill 0.8128) (layers *.Cu *.Mask F.SilkS))
+    (pad AREF thru_hole oval (at 23.876 -50.8 90) (size 2.54 1.524) (drill 0.8128) (layers *.Cu *.Mask F.SilkS))
+    (pad 5V thru_hole oval (at 38.1 -2.54 90) (size 2.54 1.524) (drill 0.8128) (layers *.Cu *.Mask F.SilkS)
+      (net 2 +5V))
+  )
 )

Commit message: clean lib
Parts:
- added C1: 10uF, lib:C_0603, F.Cu at (228.8, 23.3)
- added D4: D, lib:do214ac, F.Cu at (214.2, 23.9)
- added D6: Led_SIM, LEDs:LED_0805, F.Cu at (199.8, 37.8)
- added Q3: 2SC1815, lib:SOT-23, F.Cu at (207.6, 23.1)
- added Q4: 2SC1815, lib:SOT-23, F.Cu at (207.6, 29.8)
- added R1: 10R, lib:R_0603, F.Cu at (210.6, 36.1)
- added R11: 4.7k, lib:R_0603, F.Cu at (205.7, 36.4)
- added R12: 4k7, lib:R_0603, F.Cu at (223.8, 23.0)
- added R13: 4k7, lib:R_0603, F.Cu at (217.9, 32.2)
- added R14: 10K, lib:R_0603, F.Cu at (222.8, 27.3)
- added R2: 10R, lib:R_0603, F.Cu at (213.0, 31.9)
- added R3: 1k, lib:R_0603, F.Cu at (217.9, 27.9)
- added R4: 1k, lib:R_0603, F.Cu at (215.5, 36.3)
- added R5: 1k, lib:R_0603, F.Cu at (213.0, 27.9)
- added R6: 4.7k, lib:R_0603, F.Cu at (218.9, 22.7)
- added SW1: SW_PUSH, lib:SW_SPST_B3U-1000P-B, F.Cu at (200.3, 31.8)
- added SW2: SW_PUSH, lib:SW_SPST_B3U-1000P-B, F.Cu at (200.3, 24.8)
Connections:
- net SIM800C_PWRKEY renamed SIM800L_PWRKEY
- R24 pad 2: (no net) -> PWRKEY
- SHIELD1 pad 0: (no net) -> SIM800L_RXD
- SHIELD1 pad 1: (no net) -> SIM800L_TXD
- SHIELD1 pad 2: (no net) -> SIM800L_DTR
- SHIELD1 pad 3: (no net) -> SIM800L_RI
- SHIELD1 pad 4: (no net) -> SIM800L_DCD
- SHIELD1 pad 5: (no net) -> PWRKEY
- SHIELD1 pad 6: (no net) -> RESET
- SHIELD1 pad GND3: (no net) -> GND
- U2 pad 1: (no net) -> VDD
- U2 pad 2: (no net) -> GND
- U2 pad 31: (no net) -> Net-(R1-Pad2)
- U2 pad 32: (no net) -> Net-(R2-Pad2)
- U2 pad 35: (no net) -> GND
- U2 pad 37: (no net) -> GND
- U2 pad 38: (no net) -> GND
- U2 pad 39: (no net) -> GND
- U2 pad 4: (no net) -> SIM800L_STATUS
- U2 pad 41: (no net) -> GND
- U2 pad 42: (no net) -> VDD
- U2 pad 43: (no net) -> GND
- U2 pad 44: (no net) -> GND
- U2 pad 45: (no net) -> GND
- U2 pad 49: (no net) -> Net-(D4-Pad2)
- U2 pad 56: (no net) -> Net-(C1-Pad1)
- U2 pad 58: (no net) -> GND
- U2 pad 6: (no net) -> GND
- U2 pad 67: (no net) -> GND
- U2 pad 68: (no net) -> Net-(R4-Pad2)
- U2 pad 69: (no net) -> Net-(R5-Pad2)
- U2 pad 70: (no net) -> Net-(R3-Pad2)
- U2 pad 71: (no net) -> GND
- U2 pad 72: (no net) -> GND
- U2 pad 73: (no net) -> GND
- U2 pad 76: (no net) -> GND
- U2 pad 77: (no net) -> GND
- U2 pad 78: (no net) -> GND
- U2 pad 79: (no net) -> GND
- U2 pad 8: (no net) -> GND
- U2 pad 80: (no net) -> GND
- U2 pad 81: (no net) -> GND
- U2 pad 82: (no net) -> GND
- U2 pad 83: (no net) -> GND
- U2 pad 84: (no net) -> GND
- U2 pad 85: (no net) -> GND
- U2 pad 86: (no net) -> GND
- U2 pad 87: (no net) -> GND
- U2 pad 88: (no net) -> GND

Commit message: add footprint microsim hold
Parts:
- U6: footprint Wurth_Elektronik_Electromechanic_Input-Output_Connectors_rev16b:693023010811 -> lib:Micro_SIM_6P_PUSH_SKM01
- moved SHIELD1 85.3 mm to (179.1, 138.9)
- moved U6 42.0 mm to (63.2, 64.8)
Connections:
- R18 pad 1: (no net) -> Net-(R18-Pad1)
- R19 pad 1: (no net) -> Net-(R19-Pad1)
- U2 pad 16: (no net) -> SIM800L_VDD
Changed lines of the file:
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@@
 (kicad_pcb (version 20170123) (host pcbnew no-vcs-found-7657~57~ubuntu14.04.1)
   (general
-    (links 125)
-    (no_connects 125)
+    (links 134)
+    (no_connects 134)
     (area 0 0 0 0)
     (thickness 1.6)
@@
     (zones 0)
     (modules 55)
-    (nets 44)
+    (nets 47)
   )
   (page A4)
@@
   (net 42 SIM800L_STATUS)
   (net 43 PWRKEY)
+  (net 44 "Net-(R18-Pad1)")
+  (net 45 "Net-(R19-Pad1)")
+  (net 46 SIM800L_VDD)
   (net_class Default "This is the default net class."
     (clearance 0.2)
@@
     (add_net "Net-(Q4-Pad3)")
     (add_net "Net-(R1-Pad2)")
+    (add_net "Net-(R18-Pad1)")
+    (add_net "Net-(R19-Pad1)")
     (add_net "Net-(R2-Pad2)")
     (add_net "Net-(R3-Pad2)")
@@
     (add_net SIM800L_STATUS)
     (add_net SIM800L_TXD)
+    (add_net SIM800L_VDD)
     (add_net VDD)
   )
@@
     (fp_line (start 1.4605 -0.6985) (end 1.4605 0.6985) (layer F.SilkS) (width 0.1))
     (fp_line (start -1.4605 -0.6985) (end 1.4605 -0.6985) (layer F.SilkS) (width 0.1))
-    (pad 1 smd rect (at -0.799999 0) (size 0.8 0.9) (layers F.Cu F.Paste F.Mask))
+    (pad 1 smd rect (at -0.799999 0) (size 0.8 0.9) (layers F.Cu F.Paste F.Mask)
+      (net 44 "Net-(R18-Pad1)"))
     (pad 2 smd rect (at 0.799999 0) (size 0.8 0.9) (layers F.Cu F.Paste F.Mask)
       (net 21 SIM800L_RST))
@@
     (pad 2 smd rect (at 0.799999 0) (size 0.8 0.9) (layers F.Cu F.Paste F.Mask)
       (net 20 SIM800L_CLK))
-    (pad 1 smd rect (at -0.799999 0) (size 0.8 0.9) (layers F.Cu F.Paste F.Mask))
+    (pad 1 smd rect (at -0.799999 0) (size 0.8 0.9) (layers F.Cu F.Paste F.Mask)
+      (net 45 "Net-(R19-Pad1)"))
     (model Resistors_SMD.3dshapes/R_0603.wrl
       (at (xyz 0 0 0))
@@
     (pad 15 smd rect (at -0.6985 7.0993 90) (size 1.09982 0.89916) (layers F.Cu F.Paste F.Mask)
       (net 21 SIM800L_RST))
-    (pad 16 smd rect (at 0.6985 7.0993 90) (size 1.09982 0.89916) (layers F.Cu F.Paste F.Mask))
+    (pad 16 smd rect (at 0.6985 7.0993 90) (size 1.09982 0.89916) (layers F.Cu F.Paste F.Mask)
+      (net 46 SIM800L_VDD))
     (pad 17 smd rect (at 2.09804 7.0993 90) (size 1.09982 0.89916) (layers F.Cu F.Paste F.Mask))
     (pad 18 smd rect (at 3.49758 7.0993 90) (size 1.09982 0.89916) (layers F.Cu F.Paste F.Mask))
@@
     (pad 1 smd rect (at -0.95 -0.65) (size 0.65 0.4) (layers F.Cu F.Paste F.Mask))
   )
-  (module Wurth_Elektronik_Electromechanic_Input-Output_Connectors_rev16b:693023010811 (layer F.Cu)
-    (at 92.456 34.544)
-    (fp_text reference U6 (at -6.5 -1.75) (layer F.SilkS)
-      (effects (font (size 1.2065 1.2065) (thickness 0.1016)) (justify left bottom))
-    )
-    (fp_text value "SIM HOLD - PPSS-6P" (at -6.25 16.25) (layer F.SilkS)
-      (effects (font (size 1.2065 1.2065) (thickness 0.1016)) (justify left bottom))
-    )
-    (fp_line (start 0 0) (end 0 0) (layer F.SilkS) (width 0.127))
-    (fp_line (start 0 0) (end 0 0) (layer F.SilkS) (width 0.127))
-    (fp_line (start 0 0) (end 0 0) (layer F.SilkS) (width 0.127))
-    (fp_line (start 0 0) (end 0 0) (layer F.SilkS) (width 0.127))
-    (pad C3 smd rect (at -0.47 0 90) (size 0.95 0.67) (layers F.Cu F.Paste F.Mask))
-    (pad C6 smd rect (at 0.63 0 90) (size 0.95 0.67) (layers F.Cu F.Paste F.Mask))
-    (pad C2 smd rect (at 1.73 0 90) (size 0.95 0.67) (layers F.Cu F.Paste F.Mask))
-    (pad SW smd rect (at 2.83 0 90) (size 0.95 0.67) (layers F.Cu F.Paste F.Mask))
-    (pad C5 smd rect (at 3.93 0 90) (size 0.95 0.67) (layers F.Cu F.Paste F.Mask))
-    (pad C1 smd rect (at 5.03 0 90) (size 0.95 0.67) (layers F.Cu F.Paste F.Mask))
-    (pad C7 smd rect (at -1.57 0 90) (size 0.95 0.67) (layers F.Cu F.Paste F.Mask))
-    (pad C4 smd rect (at -2.67 0 90) (size 0.95 0.67) (layers F.Cu F.Paste F.Mask))
-    (pad C8 smd rect (at -3.77 0 90) (size 0.95 0.67) (layers F.Cu F.Paste F.Mask))
-    (pad Z1 smd rect (at -6.175 3.875 90) (size 2 1.35) (layers F.Cu F.Paste F.Mask))
-    (pad Z2 smd rect (at 6.175 3.875 90) (size 2 1.35) (layers F.Cu F.Paste F.Mask))
-    (pad Z3 smd rect (at 6.175 11.525 90) (size 2 1.35) (layers F.Cu F.Paste F.Mask))
-    (pad Z4 smd rect (at -6.175 11.525 90) (size 2 1.35) (layers F.Cu F.Paste F.Mask))
-    (pad Z5 smd rect (at -5.61 -0.225) (size 1.88 0.5) (layers F.Cu F.Paste F.Mask))
-  )
   (module arduino_shields:ARDUINO_SHIELD_2 (layer F.Cu)
-    (at 117.583005 79.85948)
+    (at 179.07 138.938)
     (fp_text reference SHIELD1 (at 5.715 -57.15) (layer F.SilkS)
       (effects (font (thickness 0.3048)))
@@
       (net 3 GND))
   )
+  (module lib:Micro_SIM_6P_PUSH_SKM01 (layer F.Cu)
+    (at 63.246 64.77)
+    (fp_text reference U6 (at 0 -4.064) (layer F.SilkS)
+      (effects (font (size 1.2065 1.2065) (thickness 0.1016)) (justify left bottom))
+    )
+    (fp_text value "SIM HOLD - PPSS-6P" (at 18.542 13.97 90) (layer F.SilkS)
+      (effects (font (size 1.2065 1.2065) (thickness 0.1016)) (justify left bottom))
+    )
+    (fp_line (start 0 -1.3) (end 10.98 -1.3) (layer F.SilkS) (width 0.1))
+    (fp_line (start 10.98 -3.1) (end 10.98 -1.3) (layer F.SilkS) (width 0.1))
+    (fp_line (start 10.98 -3.1) (end 15.8 -3.1) (layer F.SilkS) (width 0.1))
+    (fp_line (start 0 14.3) (end 15.8 14.3) (layer F.SilkS) (width 0.1))
+    (fp_line (start -21.59 -29.21) (end -21.59 -29.21) (layer F.SilkS) (width 0.01))
+    (fp_line (start -21.59 -29.21) (end -21.59 -29.21) (layer F.SilkS) (width 0.01))
+    (fp_line (start -21.59 -29.21) (end -21.59 -29.21) (layer F.SilkS) (width 0.01))
+    (fp_line (start -21.59 -29.21) (end -21.59 -29.21) (layer F.SilkS) (width 0.01))
+    (fp_line (start 0 -1.3) (end 0 14.3) (layer F.SilkS) (width 0.1))
+    (fp_line (start 15.8 -3.1) (end 15.8 14.3) (layer F.SilkS) (width 0.1))
+    (fp_arc (start 6.52 19.5) (end 2.06 14.3) (angle 81.2) (layer F.SilkS) (width 0.1))
+    (fp_line (start 12.52 15.3) (end 12.52 14.3) (layer F.SilkS) (width 0.1))
+    (fp_line (start 1 17.8) (end 10.02 17.8) (layer F.SilkS) (width 0.1))
+    (fp_line (start 0.52 14.3) (end 0.52 17.32) (layer F.SilkS) (width 0.1))
+    (fp_arc (start 1 17.32) (end 1 17.8) (angle 90) (layer F.SilkS) (width 0.1))
+    (fp_line (start 12.52 15.3) (end 10.02 17.8) (layer F.SilkS) (width 0.1))
+    (pad 3 smd rect (at 7.91 -2.45 90) (size 1.5 0.75) (layers F.Cu F.Paste F.Mask)
+      (net 45 "Net-(R19-Pad1)"))
+    (pad 7 smd rect (at 6.64 -2.45 90) (size 1.5 0.75) (layers F.Cu F.Paste F.Mask)
+      (net 18 "Net-(D5-Pad3)"))
+    (pad 2 smd rect (at 5.37 -2.45 90) (size 1.5 0.75) (layers F.Cu F.Paste F.Mask)
+      (net 44 "Net-(R18-Pad1)"))
+    (pad 6 smd rect (at 4.1 -2.45 90) (size 1.5 0.75) (layers F.Cu F.Paste F.Mask))
+    (pad 1 smd rect (at 2.83 -2.45 90) (size 1.5 0.75) (layers F.Cu F.Paste F.Mask)
+      (net 46 SIM800L_VDD))
+    (pad C3 smd rect (at -22.06 -29.21 90) (size 0.95 0.67) (layers F.Cu F.Paste F.Mask))
+    (pad C6 smd rect (at -20.96 -29.21 90) (size 0.95 0.67) (layers F.Cu F.Paste F.Mask))
+    (pad C2 smd rect (at -19.86 -29.21 90) (size 0.95 0.67) (layers F.Cu F.Paste F.Mask))
+    (pad SW smd rect (at -18.76 -29.21 90) (size 0.95 0.67) (layers F.Cu F.Paste F.Mask))
+    (pad C5 smd rect (at -17.66 -29.21 90) (size 0.95 0.67) (layers F.Cu F.Paste F.Mask))
+    (pad C1 smd rect (at -16.56 -29.21 90) (size 0.95 0.67) (layers F.Cu F.Paste F.Mask))
+    (pad C7 smd rect (at -23.16 -29.21 90) (size 0.95 0.67) (layers F.Cu F.Paste F.Mask))
+    (pad C4 smd rect (at -24.26 -29.21 90) (size 0.95 0.67) (layers F.Cu F.Paste F.Mask))
+    (pad 5 smd rect (at 1.56 -2.45 90) (size 1.5 0.75) (layers F.Cu F.Paste F.Mask)
+      (net 3 GND))
+    (pad 5 smd rect (at 0 0 90) (size 2.6 1.55) (layers F.Cu F.Paste F.Mask)
+      (net 3 GND))
+    (pad 5 smd rect (at 15.8 0 90) (size 2.6 1.55) (layers F.Cu F.Paste F.Mask)
+      (net 3 GND))
+    (pad 5 smd rect (at 15.8 12.68 90) (size 2.6 1.55) (layers F.Cu F.Paste F.Mask)
+      (net 3 GND))
+    (pad 5 smd rect (at 0 12.68 90) (size 2.6 1.55) (layers F.Cu F.Paste F.Mask)
+      (net 3 GND))
+    (pad Z5 smd rect (at -27.2 -29.435) (size 1.88 0.5) (layers F.Cu F.Paste F.Mask))
+  )
 )

Commit message: place component
Parts:
- moved R3 139.6 mm to (126.4, 133.3), turned to 90 degrees
- moved R5 137.7 mm to (124.5, 133.3), turned to 90 degrees
- moved C1 137.4 mm to (124.7, 113.0), turned to 180 degrees
- moved R2 137.1 mm to (120.7, 133.3), turned to 90 degrees
- moved R4 134.4 mm to (122.6, 133.3), turned to 90 degrees
- moved R6 134.1 mm to (149.4, 137.4), turned to 270 degrees
- moved R1 133.8 mm to (118.7, 133.3), turned to 90 degrees
- moved Q1 131.4 mm to (146.4, 133.7), turned to 180 degrees
- moved U2 129.2 mm to (127.5, 122.6), turned to 180 degrees
- moved R24 129.0 mm to (145.4, 137.4), turned to 270 degrees
- moved P3 126.9 mm to (130.3, 133.3)
- moved R12 126.5 mm to (149.1, 125.1), turned to 270 degrees
- moved Q3 124.5 mm to (150.4, 133.7), turned to 180 degrees
- moved R27 124.3 mm to (147.4, 137.4), turned to 90 degrees
- moved L1 124.2 mm to (141.0, 104.8), turned to 270 degrees
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Connections:
- D5 pad 3: Net-(D5-Pad3) -> SIM800L_DATA
- R20 pad 2: Net-(D5-Pad3) -> Net-(R20-Pad2)
- SHIELD1 pad 2: SIM800L_DTR -> SIM800L_RI
- SHIELD1 pad 3: SIM800L_RI -> SIM800L_DTR
- U6 pad 7: Net-(D5-Pad3) -> Net-(R20-Pad2)

Commit message: edge.cuts
Other:
- board outline added: 68.6 x 53.3 mm
Changed lines of the file:
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@@
     (links 134)
     (no_connects 134)
-    (area 94.852999 14.1025 218.8395 151.47732)
+    (area 98.374999 92.659999 167.055001 146.100001)
     (thickness 1.6)
-    (drawings 3)
+    (drawings 12)
     (tracks 0)
     (zones 0)
@@
       (net 3 GND))
   )
+  (gr_line (start 100.965 92.71) (end 167.005 92.71) (angle 90) (layer Edge.Cuts) (width 0.1))
+  (gr_line (start 100.965 95.25) (end 100.965 92.71) (angle 90) (layer Edge.Cuts) (width 0.1))
+  (gr_line (start 98.425 97.79) (end 100.965 95.25) (angle 90) (layer Edge.Cuts) (width 0.1))
+  (gr_line (start 98.425 130.81) (end 98.425 97.79) (angle 90) (layer Edge.Cuts) (width 0.1))
+  (gr_line (start 100.965 133.35) (end 98.425 130.81) (angle 90) (layer Edge.Cuts) (width 0.1))
+  (gr_line (start 100.965 144.78) (end 100.965 133.35) (angle 90) (layer Edge.Cuts) (width 0.1))
+  (gr_line (start 102.235 146.05) (end 100.965 144.78) (angle 90) (layer Edge.Cuts) (width 0.1))
+  (gr_line (start 167.005 146.05) (end 102.235 146.05) (angle 90) (layer Edge.Cuts) (width 0.1))
+  (gr_line (start 167.005 92.71) (end 167.005 146.05) (angle 90) (layer Edge.Cuts) (width 0.1))
   (gr_line (start 153.035 143.51) (end 153.162 143.51) (angle 90) (layer F.SilkS) (width 0.2))
   (gr_line (start 153.035 95.25) (end 153.035 143.51) (angle 90) (layer F.SilkS) (width 0.2))
