File: cellular.kicad_pcb (KiCad board)
At the start: 2 copper layers, 68.6 x 53.3 mm, 55 parts, among them P3 Chip anten, Q1 2SC1815, Q2 2SC1815, Q3 2SC1815, Q4 2SC1815, SW1 SW_PUSH, SW2 SW_PUSH, U1 MP2365DN, U2 SIM800H, U6 SIM HOLD - PPSS-6P

Commit message: 3D model diode,inductor,switch
Parts:
- D1: footprint Diodes_SMD:D_SOD-123 -> Diodes_SMD:D_MiniMELF_Standard
- moved D1 0.13 mm to (140.5, 124.7)
Changed lines of the file:
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@@
+      (rotate (xyz 0 0 0))
+    )
+    (model ${KIPRJMOD}/lib/coaxial_u.fl-r-smt-1.wrl
+      (at (xyz 0 0 0))
+      (scale (xyz 1 1 1))
       (rotate (xyz 0 0 0))
     )
@@
       (net 9 VDD))
     (model Capacitors_SMD.3dshapes/C_0603_HandSoldering.wrl
-      (at (xyz 0 0 0))
-      (scale (xyz 1 1 1))
-      (rotate (xyz 0 0 0))
-    )
-  )
-  (module Diodes_SMD:D_SOD-123 (layer F.Cu)
-    (at 140.589 124.714 180)
-    (descr SOD-123)
-    (tags SOD-123)
-    (attr smd)
-    (fp_text reference D1 (at 0 -2 180) (layer F.SilkS)
-      (effects (font (size 1 1) (thickness 0.15)))
-    )
-    (fp_text value 5.1V/500mA (at 0 2.1 180) (layer F.Fab)
-      (effects (font (size 1 1) (thickness 0.15)))
-    )
-    (fp_line (start -2.25 -1) (end 1.65 -1) (layer F.SilkS) (width 0.12))
-    (fp_line (start -2.25 1) (end 1.65 1) (layer F.SilkS) (width 0.12))
-    (fp_line (start -2.35 -1.15) (end -2.35 1.15) (layer F.CrtYd) (width 0.05))
-    (fp_line (start 2.35 1.15) (end -2.35 1.15) (layer F.CrtYd) (width 0.05))
-    (fp_line (start 2.35 -1.15) (end 2.35 1.15) (layer F.CrtYd) (width 0.05))
-    (fp_line (start -2.35 -1.15) (end 2.35 -1.15) (layer F.CrtYd) (width 0.05))
-    (fp_line (start -1.4 -0.9) (end 1.4 -0.9) (layer F.Fab) (width 0.1))
-    (fp_line (start 1.4 -0.9) (end 1.4 0.9) (layer F.Fab) (width 0.1))
-    (fp_line (start 1.4 0.9) (end -1.4 0.9) (layer F.Fab) (width 0.1))
-    (fp_line (start -1.4 0.9) (end -1.4 -0.9) (layer F.Fab) (width 0.1))
-    (fp_line (start -0.75 0) (end -0.35 0) (layer F.Fab) (width 0.1))
-    (fp_line (start -0.35 0) (end -0.35 -0.55) (layer F.Fab) (width 0.1))
-    (fp_line (start -0.35 0) (end -0.35 0.55) (layer F.Fab) (width 0.1))
-    (fp_line (start -0.35 0) (end 0.25 -0.4) (layer F.Fab) (width 0.1))
-    (fp_line (start 0.25 -0.4) (end 0.25 0.4) (layer F.Fab) (width 0.1))
-    (fp_line (start 0.25 0.4) (end -0.35 0) (layer F.Fab) (width 0.1))
-    (fp_line (start 0.25 0) (end 0.75 0) (layer F.Fab) (width 0.1))
-    (fp_line (start -2.25 -1) (end -2.25 1) (layer F.SilkS) (width 0.12))
-    (pad 2 smd rect (at 1.65 0 180) (size 0.9 1.2) (layers F.Cu F.Paste F.Mask)
-      (net 3 GND))
-    (pad 1 smd rect (at -1.65 0 180) (size 0.9 1.2) (layers F.Cu F.Paste F.Mask)
-      (net 9 VDD))
-    (model ${KISYS3DMOD}/Diodes_SMD.3dshapes/D_SOD-123.wrl
       (at (xyz 0 0 0))
       (scale (xyz 1 1 1))
@@
       (rotate (xyz 0 0 0))
     )
+    (model ${KIPRJMOD}/lib/do214ab.wrl
+      (at (xyz 0 0 0))
+      (scale (xyz 1 1 1))
+      (rotate (xyz 0 0 0))
+    )
   )
   (module LEDs:LED_0805 (layer F.Cu)
@@
     (pad 1 smd rect (at -2.75 0 270) (size 1.5 2.4) (layers F.Cu F.Paste F.Mask)
       (net 7 "Net-(C12-Pad1)"))
+    (model ${KIPRJMOD}/lib/SELF-WE-PD-XXL.wrl
+      (at (xyz 0 0 0))
+      (scale (xyz 0.55 0.55 0.55))
+      (rotate (xyz 0 0 0))
+    )
   )
   (module lib:point_test (layer F.Cu)
@@
       (net 18 SIM800L_DATA))
     (pad 1 smd rect (at -0.95 -0.65 270) (size 0.65 0.4) (layers F.Cu F.Paste F.Mask))
+    (model ${KIPRJMOD}/lib/SC-70-6.wrl
+      (at (xyz 0 0 0))
+      (scale (xyz 1 0.9 0.75))
+      (rotate (xyz 0 0 90))
+    )
   )
   (module arduino_shields:ARDUINO_SHIELD_2 (layer F.Cu)
@@
       (rotate (xyz 0 0 0))
     )
+    (model ${KIPRJMOD}/lib/do214ac.wrl
+      (at (xyz 0 0 0))
+      (scale (xyz 1 1 1))
+      (rotate (xyz 0 0 0))
+    )
   )
   (module LEDs:LED_0805 (layer F.Cu)
@@
     (pad 2 smd rect (at 1.8 0 90) (size 1.35 1.7) (layers F.Cu F.Paste F.Mask)
       (net 26 SIM800L_PWRKEY))
+    (model ${KIPRJMOD}/lib/SW_SPST_B3U-1000P-B.wrl
+      (at (xyz 0 0 0))
+      (scale (xyz 0.15 0.15 0.15))
+      (rotate (xyz 0 0 90))
+    )
   )
   (module lib:SW_SPST_B3U-1000P-B (layer F.Cu)
@@
     (pad 1 smd rect (at -1.8 0 90) (size 1.35 1.7) (layers F.Cu F.Paste F.Mask)
       (net 3 GND))
+    (model ${KIPRJMOD}/lib/SW_SPST_B3U-1000P-B.wrl
+      (at (xyz 0 0 0))
+      (scale (xyz 0.15 0.15 0.15))
+      (rotate (xyz 0 0 90))
+    )
   )
   (module lib:Micro_SIM_6P_PUSH_SKM01 (layer F.Cu)
@@
       (net 3 GND))
   )
+  (module Diodes_SMD:D_MiniMELF_Standard (layer F.Cu)
+    (at 140.462 124.714 180)
+    (descr "Diode Mini-MELF Standard")
+    (tags "Diode Mini-MELF Standard")
+    (attr smd)
+    (fp_text reference D1 (at 0 -1.95 180) (layer F.SilkS)
+      (effects (font (size 1 1) (thickness 0.15)))
+    )
+    (fp_text value 5.1V/500mA (at 0 3.81 180) (layer F.Fab)
+      (effects (font (size 1 1) (thickness 0.15)))
+    )
+    (fp_line (start -2.65 1.1) (end -2.65 -1.1) (layer F.CrtYd) (width 0.05))
+    (fp_line (start 2.65 1.1) (end -2.65 1.1) (layer F.CrtYd) (width 0.05))
+    (fp_line (start 2.65 -1.1) (end 2.65 1.1) (layer F.CrtYd) (width 0.05))
+    (fp_line (start -2.65 -1.1) (end 2.65 -1.1) (layer F.CrtYd) (width 0.05))
+    (fp_line (start -0.75 0) (end -0.35 0) (layer F.Fab) (width 0.1))
+    (fp_line (start -0.35 0) (end -0.35 -0.55) (layer F.Fab) (width 0.1))
+    (fp_line (start -0.35 0) (end -0.35 0.55) (layer F.Fab) (width 0.1))
+    (fp_line (start -0.35 0) (end 0.25 -0.4) (layer F.Fab) (width 0.1))
+    (fp_line (start 0.25 -0.4) (end 0.25 0.4) (layer F.Fab) (width 0.1))
+    (fp_line (start 0.25 0.4) (end -0.35 0) (layer F.Fab) (width 0.1))
+    (fp_line (start 0.25 0) (end 0.75 0) (layer F.Fab) (width 0.1))
+    (fp_line (start -1.65 -0.8) (end 1.65 -0.8) (layer F.Fab) (width 0.1))
+    (fp_line (start -1.65 0.8) (end -1.65 -0.8) (layer F.Fab) (width 0.1))
+    (fp_line (start 1.65 0.8) (end -1.65 0.8) (layer F.Fab) (width 0.1))
+    (fp_line (start 1.65 -0.8) (end 1.65 0.8) (layer F.Fab) (width 0.1))
+    (fp_line (start -2.55 1) (end 1.75 1) (layer F.SilkS) (width 0.12))
+    (fp_line (start -2.55 -1) (end -2.55 1) (layer F.SilkS) (width 0.12))
+    (fp_line (start 1.75 -1) (end -2.55 -1) (layer F.SilkS) (width 0.12))
+    (pad 2 smd rect (at 1.75 0 180) (size 1.3 1.7) (layers F.Cu F.Paste F.Mask)
+      (net 3 GND))
+    (pad 1 smd rect (at -1.75 0 180) (size 1.3 1.7) (layers F.Cu F.Paste F.Mask)
+      (net 9 VDD))
+    (model ${KIPRJMOD}/lib/MiniMELF_Standard.wrl
+      (at (xyz 0 0 0))
+      (scale (xyz 0.3937 0.3937 0.3937))
+      (rotate (xyz 0 0 0))
+    )
+  )
   (gr_line (start 100.965 92.71) (end 167.005 92.71) (angle 90) (layer Edge.Cuts) (width 0.1))

Commit message: modifu name compoment & text, fix track pwr
Parts:
- removed P3: Chip anten, lib:point_test
- removed SW1, SW2: SW_PUSH, lib:SW_SPST_B3U-1000P-B
- added G***: LOGO, lib:logo_cc-bby-sa_14.1x5mm, F.Cu at (151.3, 133.0)
- added G***: LOGO, lib:logo-iotmakervn_7.5x5, F.Cu at (145.4, 136.9)
- added PWR1: SW_PUSH, lib:SW_SPST_B3U-1000P-B, F.Cu at (163.1, 141.4)
- added RST1: SW_PUSH, lib:SW_SPST_B3U-1000P-B, F.Cu at (157.7, 141.4)
- added VAL**: oshw_logo_500, lib:logo5, F.Cu at (157.2, 132.6)
- U2: value SIM800H -> SIM800; footprint lib:SIM800H -> lib:SIM800
- moved D3 48.7 mm to (101.6, 108.3), turned to 90 degrees
- moved R10 46.1 mm to (104.4, 107.8), turned to 0 degrees
- moved U6 44.2 mm to (152.5, 122.9), turned to 90 degrees
- moved ANT1 39.9 mm to (101.6, 123.2), turned to 0 degrees
- moved C34 38.2 mm to (104.4, 109.6)
- moved D1 37.6 mm to (103.4, 118.4)
- moved C33 37.2 mm to (104.4, 111.3)
- moved C31 36.7 mm to (103.8, 115.3)
- moved C32 36.5 mm to (104.4, 112.9)
- moved C29 34.4 mm to (146.7, 123.3), turned to 180 degrees
- moved R26 32.1 mm to (104.9, 123.2), turned to 270 degrees
- moved D5 31.5 mm to (146.7, 120.7), turned to 90 degrees
- moved R18 29.4 mm to (146.7, 118.0), turned to 180 degrees
- moved R20 28.4 mm to (146.7, 116.3), turned to 0 degrees
- moved R19 27.9 mm to (146.7, 114.7), turned to 180 degrees
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Connections:
- C28 pad 1: Net-(C28-Pad1) -> SIM800L_VDD
- D5 pad 6: Net-(C28-Pad1) -> SIM800L_VDD
- SHIELD1 pad 0: SIM800L_RXD -> SIM800L_TXD
- SHIELD1 pad 1: SIM800L_TXD -> SIM800L_RXD
- SHIELD1 pad 2: SIM800L_RI -> SIM800L_DTR
- SHIELD1 pad 3: SIM800L_DTR -> SIM800L_RI
- U2 pad 1: VDD -> SIM800L_PWRKEY
- U2 pad 10: (no net) -> Net-(R1-Pad2)
- U2 pad 14: SIM800L_DATA -> (no net)
- U2 pad 15: SIM800L_RST -> (no net)
- U2 pad 16: SIM800L_VDD -> Net-(D4-Pad2)
- U2 pad 17: (no net) -> GND
- U2 pad 18: (no net) -> GND
- U2 pad 26: (no net) -> Net-(C1-Pad1)
- U2 pad 3: (no net) -> Net-(R5-Pad2)
- U2 pad 30: (no net) -> SIM800L_VDD
- U2 pad 31: Net-(R1-Pad2) -> SIM800L_DATA
- U2 pad 32: Net-(R2-Pad2) -> SIM800L_CLK
- U2 pad 33: (no net) -> SIM800L_RST
- U2 pad 35: GND -> (no net)
- U2 pad 37: GND -> (no net)
- U2 pad 38: GND -> (no net)
- U2 pad 4: SIM800L_STATUS -> Net-(R4-Pad2)
- U2 pad 40: GSM_ANT -> (no net)
- U2 pad 41: GND -> (no net)
- U2 pad 42: VDD -> (no net)
- U2 pad 43: GND -> (no net)
- U2 pad 44: GND -> (no net)
- U2 pad 48: SIM800L_PWRKEY -> (no net)
- U2 pad 49: Net-(D4-Pad2) -> (no net)
- U2 pad 5: (no net) -> Net-(R3-Pad2)
- U2 pad 52: (no net) -> SIM800L_NETLIGHT
- U2 pad 54: (no net) -> GND
- U2 pad 55: SIM800L_CLK -> VDD
- U2 pad 56: Net-(C1-Pad1) -> VDD
- U2 pad 57: (no net) -> VDD
- U2 pad 59: (no net) -> GND
- U2 pad 6: GND -> (no net)
- U2 pad 60: (no net) -> GSM_ANT
- U2 pad 61: (no net) -> GND
- U2 pad 62: (no net) -> GND
- U2 pad 63: (no net) -> GND
- U2 pad 64: SIM800L_NETLIGHT -> GND
- U2 pad 65: (no net) -> GND
- U2 pad 66: (no net) -> SIM800L_STATUS
- U2 pad 67: GND -> (no net)
- U2 pad 68: Net-(R4-Pad2) -> (no net)
- U2 pad 8: GND -> (no net)
- U2 pad 9: (no net) -> Net-(R2-Pad2)
Routing:
- net GND: track 0.00 -> 357.8 mm, vias 0 -> 19
- net VDD: track 0.00 -> 97.4 mm, vias 0 -> 4
- net SIM800L_PWRKEY: track 0.00 -> 56.1 mm, vias 0 -> 2
- net SIM800L_NETLIGHT: track 0.00 -> 41.2 mm, vias 0 -> 2
- net SIM800L_VDD: track 0.00 -> 40.8 mm, vias 0 -> 2
- net SIM800L_STATUS: track 0.00 -> 30.4 mm
- net SIM800L_RESET: track 0.00 -> 28.4 mm
- net SIM800L_DATA: track 0.00 -> 26.4 mm, vias 0 -> 2
- net Net-(C12-Pad1): track 0.00 -> 25.9 mm
- net SIM800L_CLK: track 0.00 -> 21.6 mm, vias 0 -> 2
- net SIM800L_RST: track 0.00 -> 20.8 mm, vias 0 -> 2
- net Net-(R2-Pad2): track 0.00 -> 19.9 mm
- net Net-(D4-Pad2): track 0.00 -> 19.8 mm, vias 0 -> 2
- net Net-(R1-Pad2): track 0.00 -> 19.0 mm, vias 0 -> 2
- net +5V: track 0.00 -> 13.9 mm
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- added copper zone on B.Cu, net GND
- added copper zone on F.Cu, net GND
Other:
- outline, holes or cut-outs redrawn
- net class Default: clearance 0.2 -> 0.254; trace_width 0.25 -> 0.3; via_dia 0.8 -> 1.1; via_drill 0.4 -> 0.6
- rule trace_clearance: 0.2 -> 0.254
- rule trace_min: 0.2 -> 0.254
- rule via_min_drill: 0.3 -> 0.2
- rule via_min_size: 0.4 -> 1.1
- board text added: "-------------"
- board text added: "0"
- board text added: "0 1 2 3"
- board text added: "1"
- board text added: "2"
- board text added: "3"
- board text added: "4"
- board text added: "4 5 6"
- board text added: "5"
- board text added: "6"
- board text added: "DCD"
- board text added: "DTR"
- board text added: "ESP32"
- board text added: "GPIO00"
- board text added: "GPIO02"
- board text added: "GPIO04"
- board text added: "GPIO25"
- board text added: "GPIO26"
- board text added: "Maker"
- board text added: "NETLIGHT"
- board text added: "PWR"
- board text added: "PWRKEY"
- board text added: "RESET"
- board text added: "RI"
- board text added: "RST"
- board text added: "RX"
- board text added: "SIM800"
- board text added: "STATUS"
- board text added: "TX"
- board text added: "|"
- board text added: "| | |"
- board text added: "| | | |"
