File: esp32-cellular-shield.kicad_pcb (KiCad board)
At the start: 2 copper layers, 68.6 x 53.3 mm, 57 parts, among them Q1 2SC1815, Q2 2SC1815, Q3 2SC1815, Q4 2SC1815, U1 MP2365DN, U2 SIM800, U6 SIM HOLD - PPSS-6P

Commit message: modify esp-uno.lib & add footprint esp-uno-shield
Parts:
- removed ANT1: ANTENNA, lib:coaxial_u.fl-r-smt-1
- removed C1, C32: 10uF, lib:C_0603
- removed C10: 4.7nF, lib:C_0603
- removed C12: 10nF, lib:C_0603
- removed C13: 47uF, lib:C_0603
- removed C2: 10uF/35V, Capacitors_SMD:C_1210
- removed C28: 100nF, lib:C_0603
- removed C29: 22pF, lib:C_0603
- removed C31: 100uF, Capacitors_SMD:C_1210
- removed C33: 33pF, lib:C_0603
- removed C34: 10pF, lib:C_0603
- removed C4: 0.1uF, lib:C_0603
- removed D1: 5.1V/500mA, Diodes_SMD:D_MiniMELF_Standard
- removed D2: MBRS340, lib:do214ab
- removed D3: Led_pwr, LEDs:LED_0805
- removed D4: D, lib:do214ac
- removed D5: SMF05C, TO_SOT_Packages_SMD:SOT-363_SC-70-6
- removed D6, D7: Led_SIM, LEDs:LED_0805
- removed G***: LOGO, lib:logo_cc-bby-sa_14.1x5mm
- removed G***: LOGO, lib:logo-iotmakervn_7.5x5
- removed L1: 4.7uH-2.2A, Choke_SMD:Choke_SMD_6.3x6.3_H3
- removed PWR1, RST1: SW_PUSH, lib:SW_SPST_B3U-1000P-B
- removed Q1, Q2, Q3, Q4: 2SC1815, lib:SOT-23
- removed R1, R2: 10R, lib:R_0603
- removed R10: 10k, lib:R_0603
- removed R11, R24, R27, R6: 4.7k, lib:R_0603
- removed R12, R13, R25, R28: 4k7, lib:R_0603
- removed R14, R29: 10K, lib:R_0603
- removed R18, R19, R20: 22R, lib:R_0603
- removed R26: 0R, lib:R_0603
- removed R3, R4, R5: 1k, lib:R_0603
- removed R7: 20k, lib:R_0603
- removed R8: 10k-1%, lib:R_0603
- removed R9: 33,6k-1%, lib:R_0603
- removed SHIELD1: ARDUINO_SHIELD, arduino_shields:ARDUINO_SHIELD_2
- removed U1: MP2365DN, SMD_Packages:SOIC-8-N
- removed U2: SIM800, lib:SIM800
- removed VAL**: oshw_logo_500, lib:logo5
- added S1: ESP-UNO, lib:ESP-UNO-SH, F.Cu at (139.7, 76.2)
- moved U6 46.7 mm to (127.0, 83.8), turned to 270 degrees
Other:
- board size 68.6 x 53.3 mm -> 68.5 x 53.3 mm
- board text removed: "-------------"
- board text removed: "0"
- board text removed: "0 1 2 3"
- board text removed: "1"
- board text removed: "2"
- board text removed: "3"
- board text removed: "4"
- board text removed: "4 5 6"
- board text removed: "5"
- board text removed: "6"
- board text removed: "DCD"
- board text removed: "DTR"
- board text removed: "ESP32"
- board text removed: "GPIO00"
- board text removed: "GPIO02"
- board text removed: "GPIO04"
- board text removed: "GPIO25"
- board text removed: "GPIO26"
- board text removed: "Maker"
- board text removed: "NETLIGHT"
- board text removed: "PWR"
- board text removed: "PWRKEY"
- board text removed: "RESET"
- board text removed: "RI"
- board text removed: "RST"
- board text removed: "RX"
- board text removed: "SIM800"
- board text removed: "STATUS"
- board text removed: "TX"
- board text removed: "|"
- board text removed: "| | |"
- board text removed: "| | | |"

Commit message: read .net file in pcb
Parts:
- added ANT1: ANTENNA, lib:coaxial_u.fl-r-smt-1, F.Cu at (253.4, 109.1)
- added C1: 4.7uF, lib:C_0603, F.Cu at (287.6, 76.8)
- added C10: 4.7nF, lib:C_0603, F.Cu at (281.1, 89.8)
- added C12: 10nF, lib:C_0603, F.Cu at (287.6, 80.8)
- added C13: 47uF, lib:C_0603, F.Cu at (287.6, 84.8)
- added C2: 10uF/35V, Capacitors_SMD:C_1210, F.Cu at (282.8, 71.1)
- added C28: 100nF, lib:C_0603, F.Cu at (262.4, 109.8)
- added C29: 22pF, lib:C_0603, F.Cu at (257.9, 112.6)
- added C3: 10uF, lib:C_0603, F.Cu at (234.1, 130.9)
- added C31: 100uF, Capacitors_SMD:C_1210, F.Cu at (195.7, 127.9)
- added C32: 10uF, lib:C_0603, F.Cu at (224.1, 130.9)
- added C33: 33pF, lib:C_0603, F.Cu at (244.1, 126.7)
- added C34: 10pF, lib:C_0603, F.Cu at (262.4, 105.7)
- added C4: 0.1uF, lib:C_0603, F.Cu at (213.3, 130.9)
- added C5: 10uF, lib:C_0603, F.Cu at (276.1, 94.6)
- added D1: 5.1V/500mA, Diodes_SMD:D_MiniMELF_Standard, F.Cu at (179.5, 127.6)
- added D2: MBRS340, lib:do214ab, F.Cu at (255.8, 103.0)
- added D3: Led_pwr, LEDs:LED_0805, F.Cu at (272.5, 81.3)
- added D5: SMF05C, TO_SOT_Packages_SMD:SOT-363_SC-70-6, F.Cu at (208.2, 127.7)
- added D6: Led_SIM, LEDs:LED_0805, F.Cu at (201.7, 127.1)
- added D7: Led_SIM, LEDs:LED_0805, F.Cu at (266.0, 90.2)
- added L1: 4.7uH-2.2A, Choke_SMD:Choke_SMD_6.3x6.3_H3, F.Cu at (274.0, 73.3)
- added R1: 10R, lib:R_0603, F.Cu at (224.0, 126.1)
- added R10: 10k, lib:R_0603, F.Cu at (282.6, 80.6)
- added R11: 4.7k, lib:R_0603, F.Cu at (271.0, 89.8)
- added R12: 4k7, lib:R_0603, F.Cu at (252.9, 114.2)
- added R13: 4k7, lib:R_0603, F.Cu at (276.0, 89.8)
- added R14: 10K, lib:R_0603, F.Cu at (271.0, 94.3)
- added R18: 22R, lib:R_0603, F.Cu at (239.1, 126.4)
- added R19: 22R, lib:R_0603, F.Cu at (277.6, 80.5)
- added R2: 10R, lib:R_0603, F.Cu at (264.5, 94.3)
- added R20: 22R, lib:R_0603, F.Cu at (267.2, 103.2)
- added R24: 4.7k, lib:R_0603, F.Cu at (272.2, 98.7)
- added R25: 4k7, lib:R_0603, F.Cu at (252.9, 118.7)
- added R26: 0R, lib:R_0603, F.Cu at (282.6, 85.0)
- added R27: 4.7k, lib:R_0603, F.Cu at (229.0, 126.4)
- added R28: 4k7, lib:R_0603, F.Cu at (267.2, 98.7)
- added R29: 10K, lib:R_0603, F.Cu at (219.0, 126.4)
- added R3: 1k, lib:R_0603, F.Cu at (257.4, 107.8)
- added R4: 1k, lib:R_0603, F.Cu at (262.2, 100.9)
- added R5: 1k, lib:R_0603, F.Cu at (234.0, 126.1)
- added R6: 4.7k, lib:R_0603, F.Cu at (282.6, 76.1)
- added R7: 20k, lib:R_0603, F.Cu at (277.6, 84.7)
- added R8: 10k-1%, lib:R_0603, F.Cu at (271.4, 85.4)
- added R9: 33,6k-1%, lib:R_0603, F.Cu at (214.0, 126.1)
- added U1: MP2365DN, SMD_Packages:SOIC-8-N, F.Cu at (188.8, 128.7)
- added U2: SIM800C, lib:SIM800C, F.Cu at (260.2, 77.8)
- added U3: Ra-02, SO-16-W, F.Cu at (256.9, 93.6)

Commit message: add PWR 3.3V with IC tc1264-33VAB, swap IC PWR to MCP16311-MNY with Vdd=4.2V
Parts:
- moved U2 136.9 mm to (123.8, 89.5), turned to 180 degrees
- moved U6 38.5 mm to (94.1, 103.8)
Other:
- outline, holes or cut-outs redrawn
Changed lines of the file:
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@@
     (area 108.967475 50.785954 177.602094 104.185956)
     (thickness 1.6)
-    (drawings 753)
+    (drawings 754)
     (tracks 0)
     (zones 0)
@@
   )
   (module lib:Micro_SIM_6P_PUSH_SKM01 (layer F.Cu)
-    (at 127 83.84 270)
+    (at 94.07 103.85 270)
     (fp_text reference U6 (at 0 -4.064 270) (layer F.SilkS)
       (effects (font (size 1.2065 1.2065) (thickness 0.1016)) (justify left bottom))
@@
   )
   (module lib:SIM800C (layer F.Cu)
-    (at 260.23962 77.752596)
-    (fp_text reference U2 (at 0 0.5) (layer F.SilkS)
-      (effects (font (size 1 1) (thickness 0.15)))
-    )
-    (fp_text value SIM800C (at 0 -0.5) (layer F.Fab)
+    (at 123.825 89.535 180)
+    (fp_text reference U2 (at 0 0.5 180) (layer F.SilkS)
+      (effects (font (size 1 1) (thickness 0.15)))
+    )
+    (fp_text value SIM800C (at 0 -0.5 180) (layer F.Fab)
       (effects (font (size 1 1) (thickness 0.15)))
     )
@@
     (fp_line (start -6.9 -7.6) (end -7.85 -6.55) (layer F.SilkS) (width 0.15))
     (fp_line (start -7.85 -6.55) (end -8.8 -7.6) (layer F.SilkS) (width 0.15))
-    (pad 1 smd oval (at -7.85 -6.05) (size 1.8 0.6) (layers F.Cu F.Paste F.Mask)
+    (pad 1 smd oval (at -7.85 -6.05 180) (size 1.8 0.6) (layers F.Cu F.Paste F.Mask)
       (net 22 "Net-(R2-Pad2)"))
-    (pad 2 smd oval (at -7.85 -4.95) (size 1.8 0.6) (layers F.Cu F.Paste F.Mask)
+    (pad 2 smd oval (at -7.85 -4.95 180) (size 1.8 0.6) (layers F.Cu F.Paste F.Mask)
       (net 21 "Net-(R1-Pad2)"))
-    (pad 3 smd oval (at -7.85 -3.85) (size 1.8 0.6) (layers F.Cu F.Paste F.Mask))
-    (pad 4 smd oval (at -7.85 -2.75) (size 1.8 0.6) (layers F.Cu F.Paste F.Mask))
-    (pad 5 smd oval (at -7.85 -1.65) (size 1.8 0.6) (layers F.Cu F.Paste F.Mask)
+    (pad 3 smd oval (at -7.85 -3.85 180) (size 1.8 0.6) (layers F.Cu F.Paste F.Mask))
+    (pad 4 smd oval (at -7.85 -2.75 180) (size 1.8 0.6) (layers F.Cu F.Paste F.Mask))
+    (pad 5 smd oval (at -7.85 -1.65 180) (size 1.8 0.6) (layers F.Cu F.Paste F.Mask)
       (net 23 "Net-(R3-Pad2)"))
-    (pad 6 smd oval (at -7.85 -0.55) (size 1.8 0.6) (layers F.Cu F.Paste F.Mask)
+    (pad 6 smd oval (at -7.85 -0.55 180) (size 1.8 0.6) (layers F.Cu F.Paste F.Mask)
       (net 25 "Net-(R5-Pad2)"))
-    (pad 7 smd oval (at -7.85 0.55) (size 1.8 0.6) (layers F.Cu F.Paste F.Mask)
+    (pad 7 smd oval (at -7.85 0.55 180) (size 1.8 0.6) (layers F.Cu F.Paste F.Mask)
       (net 24 "Net-(R4-Pad2)"))
-    (pad 8 smd oval (at -7.85 1.65) (size 1.8 0.6) (layers F.Cu F.Paste F.Mask)
-      (net 1 GND))
-    (pad 9 smd oval (at -7.85 2.75) (size 1.8 0.6) (layers F.Cu F.Paste F.Mask))
-    (pad 10 smd oval (at -7.85 3.85) (size 1.8 0.6) (layers F.Cu F.Paste F.Mask))
-    (pad 11 smd oval (at -7.85 4.95) (size 1.8 0.6) (layers F.Cu F.Paste F.Mask))
-    (pad 12 smd oval (at -7.85 6.05) (size 1.8 0.6) (layers F.Cu F.Paste F.Mask))
-    (pad 22 smd oval (at 7.85 6.05) (size 1.8 0.6) (layers F.Cu F.Paste F.Mask))
-    (pad 23 smd oval (at 7.85 4.95) (size 1.8 0.6) (layers F.Cu F.Paste F.Mask))
-    (pad 24 smd oval (at 7.85 3.85) (size 1.8 0.6) (layers F.Cu F.Paste F.Mask))
-    (pad 25 smd oval (at 7.85 2.75) (size 1.8 0.6) (layers F.Cu F.Paste F.Mask))
-    (pad 26 smd oval (at 7.85 1.65) (size 1.8 0.6) (layers F.Cu F.Paste F.Mask))
-    (pad 27 smd oval (at 7.85 0.55) (size 1.8 0.6) (layers F.Cu F.Paste F.Mask)
-      (net 1 GND))
-    (pad 28 smd oval (at 7.85 -0.55) (size 1.8 0.6) (layers F.Cu F.Paste F.Mask)
+    (pad 8 smd oval (at -7.85 1.65 180) (size 1.8 0.6) (layers F.Cu F.Paste F.Mask)
+      (net 1 GND))
+    (pad 9 smd oval (at -7.85 2.75 180) (size 1.8 0.6) (layers F.Cu F.Paste F.Mask))
+    (pad 10 smd oval (at -7.85 3.85 180) (size 1.8 0.6) (layers F.Cu F.Paste F.Mask))
+    (pad 11 smd oval (at -7.85 4.95 180) (size 1.8 0.6) (layers F.Cu F.Paste F.Mask))
+    (pad 12 smd oval (at -7.85 6.05 180) (size 1.8 0.6) (layers F.Cu F.Paste F.Mask))
+    (pad 22 smd oval (at 7.85 6.05 180) (size 1.8 0.6) (layers F.Cu F.Paste F.Mask))
+    (pad 23 smd oval (at 7.85 4.95 180) (size 1.8 0.6) (layers F.Cu F.Paste F.Mask))
+    (pad 24 smd oval (at 7.85 3.85 180) (size 1.8 0.6) (layers F.Cu F.Paste F.Mask))
+    (pad 25 smd oval (at 7.85 2.75 180) (size 1.8 0.6) (layers F.Cu F.Paste F.Mask))
+    (pad 26 smd oval (at 7.85 1.65 180) (size 1.8 0.6) (layers F.Cu F.Paste F.Mask))
+    (pad 27 smd oval (at 7.85 0.55 180) (size 1.8 0.6) (layers F.Cu F.Paste F.Mask)
+      (net 1 GND))
+    (pad 28 smd oval (at 7.85 -0.55 180) (size 1.8 0.6) (layers F.Cu F.Paste F.Mask)
       (net 7 "Net-(C1-Pad1)"))
-    (pad 29 smd oval (at 7.85 -1.65) (size 1.8 0.6) (layers F.Cu F.Paste F.Mask))
-    (pad 30 smd oval (at 7.85 -2.75) (size 1.8 0.6) (layers F.Cu F.Paste F.Mask)
-      (net 1 GND))
-    (pad 31 smd oval (at 7.85 -3.85) (size 1.8 0.6) (layers F.Cu F.Paste F.Mask)
-      (net 1 GND))
-    (pad 32 smd oval (at 7.85 -4.95) (size 1.8 0.6) (layers F.Cu F.Paste F.Mask)
+    (pad 29 smd oval (at 7.85 -1.65 180) (size 1.8 0.6) (layers F.Cu F.Paste F.Mask))
+    (pad 30 smd oval (at 7.85 -2.75 180) (size 1.8 0.6) (layers F.Cu F.Paste F.Mask)
+      (net 1 GND))
+    (pad 31 smd oval (at 7.85 -3.85 180) (size 1.8 0.6) (layers F.Cu F.Paste F.Mask)
+      (net 1 GND))
+    (pad 32 smd oval (at 7.85 -4.95 180) (size 1.8 0.6) (layers F.Cu F.Paste F.Mask)
       (net 33 GSM_ANT))
-    (pad 33 smd oval (at 7.85 -6.05) (size 1.8 0.6) (layers F.Cu F.Paste F.Mask)
-      (net 1 GND))
-    (pad 42 smd oval (at -4.4 -8.8 90) (size 1.8 0.6) (layers F.Cu F.Paste F.Mask)
+    (pad 33 smd oval (at 7.85 -6.05 180) (size 1.8 0.6) (layers F.Cu F.Paste F.Mask)
+      (net 1 GND))
+    (pad 42 smd oval (at -4.4 -8.8 270) (size 1.8 0.6) (layers F.Cu F.Paste F.Mask)
       (net 29 SIM800L_STATUS))
-    (pad 41 smd oval (at -3.3 -8.8 90) (size 1.8 0.6) (layers F.Cu F.Paste F.Mask)
+    (pad 41 smd oval (at -3.3 -8.8 270) (size 1.8 0.6) (layers F.Cu F.Paste F.Mask)
       (net 31 SIM800L_NETLIGHT))
-    (pad 40 smd oval (at -2.2 -8.8 90) (size 1.8 0.6) (layers F.Cu F.Paste F.Mask))
-    (pad 39 smd oval (at -1.1 -8.8 90) (size 1.8 0.6) (layers F.Cu F.Paste F.Mask))
-    (pad 38 smd oval (at 0 -8.8 90) (size 1.8 0.6) (layers F.Cu F.Paste F.Mask))
-    (pad 37 smd oval (at 1.1 -8.8 90) (size 1.8 0.6) (layers F.Cu F.Paste F.Mask)
-      (net 1 GND))
-    (pad 36 smd oval (at 2.2 -8.8 90) (size 1.8 0.6) (layers F.Cu F.Paste F.Mask)
-      (net 1 GND))
-    (pad 35 smd oval (at 3.3 -8.8 90) (size 1.8 0.6) (layers F.Cu F.Paste F.Mask))
-    (pad 34 smd oval (at 4.4 -8.8 90) (size 1.8 0.6) (layers F.Cu F.Paste F.Mask))
-    (pad 17 smd oval (at 0 8.8 90) (size 1.8 0.6) (layers F.Cu F.Paste F.Mask)
+    (pad 40 smd oval (at -2.2 -8.8 270) (size 1.8 0.6) (layers F.Cu F.Paste F.Mask))
+    (pad 39 smd oval (at -1.1 -8.8 270) (size 1.8 0.6) (layers F.Cu F.Paste F.Mask))
+    (pad 38 smd oval (at 0 -8.8 270) (size 1.8 0.6) (layers F.Cu F.Paste F.Mask))
+    (pad 37 smd oval (at 1.1 -8.8 270) (size 1.8 0.6) (layers F.Cu F.Paste F.Mask)
+      (net 1 GND))
+    (pad 36 smd oval (at 2.2 -8.8 270) (size 1.8 0.6) (layers F.Cu F.Paste F.Mask)
+      (net 1 GND))
+    (pad 35 smd oval (at 3.3 -8.8 270) (size 1.8 0.6) (layers F.Cu F.Paste F.Mask))
+    (pad 34 smd oval (at 4.4 -8.8 270) (size 1.8 0.6) (layers F.Cu F.Paste F.Mask))
+    (pad 17 smd oval (at 0 8.8 270) (size 1.8 0.6) (layers F.Cu F.Paste F.Mask)
       (net 18 SIM800L_RST))
-    (pad 18 smd oval (at 1.1 8.8 90) (size 1.8 0.6) (layers F.Cu F.Paste F.Mask)
+    (pad 18 smd oval (at 1.1 8.8 270) (size 1.8 0.6) (layers F.Cu F.Paste F.Mask)
       (net 2 SIM800L_VDD))
-    (pad 19 smd oval (at 2.2 8.8 90) (size 1.8 0.6) (layers F.Cu F.Paste F.Mask)
-      (net 1 GND))
-    (pad 20 smd oval (at 3.3 8.8 90) (size 1.8 0.6) (layers F.Cu F.Paste F.Mask))
-    (pad 21 smd oval (at 4.4 8.8 90) (size 1.8 0.6) (layers F.Cu F.Paste F.Mask)
-      (net 1 GND))
-    (pad 16 smd oval (at -1.1 8.8 90) (size 1.8 0.6) (layers F.Cu F.Paste F.Mask)
+    (pad 19 smd oval (at 2.2 8.8 270) (size 1.8 0.6) (layers F.Cu F.Paste F.Mask)
+      (net 1 GND))
+    (pad 20 smd oval (at 3.3 8.8 270) (size 1.8 0.6) (layers F.Cu F.Paste F.Mask))
+    (pad 21 smd oval (at 4.4 8.8 270) (size 1.8 0.6) (layers F.Cu F.Paste F.Mask)
+      (net 1 GND))
+    (pad 16 smd oval (at -1.1 8.8 270) (size 1.8 0.6) (layers F.Cu F.Paste F.Mask)
       (net 17 SIM800L_CLK))
-    (pad 13 smd oval (at -4.4 8.8 90) (size 1.8 0.6) (layers F.Cu F.Paste F.Mask)
-      (net 1 GND))
-    (pad 14 smd oval (at -3.3 8.8 90) (size 1.8 0.6) (layers F.Cu F.Paste F.Mask))
-    (pad 15 smd oval (at -2.2 8.8 90) (size 1.8 0.6) (layers F.Cu F.Paste F.Mask)
+    (pad 13 smd oval (at -4.4 8.8 270) (size 1.8 0.6) (layers F.Cu F.Paste F.Mask)
+      (net 1 GND))
+    (pad 14 smd oval (at -3.3 8.8 270) (size 1.8 0.6) (layers F.Cu F.Paste F.Mask))
+    (pad 15 smd oval (at -2.2 8.8 270) (size 1.8 0.6) (layers F.Cu F.Paste F.Mask)
       (net 15 SIM800L_DATA))
-    (model ${KIPRJMOD}/3dshapes/SIM800C.wrl
+    (model ${KIPRJMOD}/lib/SIM800C.wrl
       (at (xyz 0 0 0))
       (scale (xyz 1 1 1))
@@
     )
   )
+  (gr_circle (center 113 100) (end 116 100) (layer Edge.Cuts) (width 0.2))
   (gr_line (start 175.006 101.5746) (end 175.006 101.5746) (layer Edge.Cuts) (width 0.1))
   (gr_line (start 173.736 53.4035) (end 173.736 53.4035) (layer Edge.Cuts) (width 0.1))

Commit message: add PCB
Parts:
- removed C28: 100nF, lib:C_0603
- removed C29: 22pF, lib:C_0603
- removed C31: 100uF, Capacitors_SMD:C_1210
- removed C32: 10uF, lib:C_0603
- removed C33: 33pF, lib:C_0603
- removed C34: 10pF, lib:C_0603
- removed D6, D7: Led_SIM, LEDs:LED_0805
- removed R24, R27: 4.7k, lib:R_0603
- removed R25, R28: 4k7, lib:R_0603
- removed R26: 0R, lib:R_0603
- removed R29: 10K, lib:R_0603
- added C11: 100nF, lib:C_0603, F.Cu at (145.7, 92.1)
- added C14: 10uF/25V, Capacitors_SMD:C_1210, F.Cu at (140.2, 87.5)
- added C15: 10uF/25V, Capacitors_SMD:C_1210, F.Cu at (143.5, 87.5)
- added C16: 1uF/25V, lib:C_0603, F.Cu at (140.0, 83.2)
- added C17: 1uF, lib:C_0603, F.Cu at (149.9, 95.2)
- added C6: 33pF, lib:C_0603, F.Cu at (139.0, 44.0)
- added C7: 100nF, lib:C_0603, F.Cu at (139.0, 45.5)
- added C8: 33pF, lib:C_0603, F.Cu at (139.0, 47.0)
- added C9: 4.7uF, lib:C_0603, F.Cu at (130.4, 48.0)
- added D4: Led_SIM, LEDs:LED_0603, F.Cu at (195.9, 55.0)
- added PWR1: PWRKEY, lib:Tact_switch-4pin, F.Cu at (111.5, 65.0)
- added Q1: Q_NPN_BEC, TO_SOT_Packages_SMD:SOT-23, F.Cu at (189.6, 50.9)
- added Q2: Q_NPN_BEC, TO_SOT_Packages_SMD:SOT-23, F.Cu at (202.7, 63.7)
- added Q3: Q_NPN_BEC, TO_SOT_Packages_SMD:SOT-23, F.Cu at (195.4, 65.5)
- added R15: 10K, lib:R_0603, F.Cu at (195.9, 61.0)
- added R16: 4k7, lib:R_0603, F.Cu at (195.9, 59.0)
- added R17: 4k7, lib:R_0603, F.Cu at (195.9, 57.0)
- added R21: 47k/1%, lib:R_0603, F.Cu at (152.4, 96.1)
- added U4: MCP601OT, TO_SOT_Packages_SMD:SOT-23-5, F.Cu at (155.4, 87.5)
- added U5: IRLM6402, TO_SOT_Packages_SMD:SOT-23_Handsoldering, F.Cu at (155.4, 82.9)
- added U7: TC1264-3.3VAB, lib:TO-220, F.Cu at (146.3, 81.2)
- C1: value 4.7uF -> 100uF/16v; footprint lib:C_0603 -> Capacitors_SMD:C_1210
- C10: value 4.7nF -> 100nF
- C12: value 10nF -> 10uF/50V; footprint lib:C_0603 -> Capacitors_SMD:C_1210
- C13: value 47uF -> 10uF/50V; footprint lib:C_0603 -> Capacitors_SMD:C_1210
- C2: value 10uF/35V -> 10uF/16v; footprint Capacitors_SMD:C_1210 -> lib:C_0603
- C3: value 10uF -> 33pF/16v
- C4: value 0.1uF -> 10pF/16v
- C5: value 10uF -> 22pF
- D2: value MBRS340 -> SMF05C; footprint lib:do214ab -> TO_SOT_Packages_SMD:SOT-363_SC-70-6
- D3: value Led_pwr -> Led_SIM; footprint LEDs:LED_0805 -> LEDs:LED_0603
- D5: value SMF05C -> SS34; footprint TO_SOT_Packages_SMD:SOT-363_SC-70-6 -> lib:do214ac
- L1: value 4.7uH-2.2A -> 22uH; footprint Choke_SMD:Choke_SMD_6.3x6.3_H3 -> Choke_SMD:Choke_SMD_Wuerth-WE-PD2-Typ-MS
- R1: value 10R -> 0R
- R10: value 10k -> 1K
- R11: value 4.7k -> 1K
- R12: value 4k7 -> 10K
- R14: value 10K -> 4k7
- R18, R19: value 22R -> 10k
- R2: value 10R -> 4.7k
- R20: value 22R -> 200k/1%
- R3, R4, R5: value 1k -> 22R
- R7: value 20k -> 1K
- R8: value 10k-1% -> 1K
- R9: value 33,6k-1% -> 1K
- U1: value MP2365DN -> SIM HOLD - PPSS-6P; footprint SMD_Packages:SOIC-8-N -> lib:sim_socket_PP
- U3: footprint SO-16-W -> lib:Lora-RA02
- U6: value SIM HOLD - PPSS-6P -> MCP16311-MNY; footprint lib:Micro_SIM_6P_PUSH_SKM01 -> Housings_SSOP:MSOP-8_3x3mm_Pitch0.65mm
- moved C1 162.5 mm to (125.2, 78.0), turned to 270 degrees
- moved C2 160.1 mm to (122.8, 78.0), turned to 270 degrees
- moved R10 157.0 mm to (130.4, 41.9)
- moved R7 152.0 mm to (130.4, 46.5)
- moved R11 149.0 mm to (130.4, 40.4)
- moved C5 146.7 mm to (139.0, 42.5)
- moved R8 146.7 mm to (130.4, 45.0)
- moved ANT1 144.4 mm to (120.4, 52.7)
- moved C12 141.0 mm to (146.8, 87.5), turned to 90 degrees
- moved C13 137.6 mm to (150.1, 87.5), turned to 90 degrees
- moved L1 134.0 mm to (141.5, 93.7), turned to 270 degrees
- moved U3 129.3 mm to (127.6, 90.0), turned to 90 degrees
- moved C10 128.6 mm to (152.7, 83.2), turned to 270 degrees
- moved R4 128.0 mm to (147.0, 45.0)
- moved R3 126.0 mm to (147.0, 47.0)
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Connections:
- C1 pad 1: Net-(C1-Pad1) -> VDD
- C10 pad 1: Net-(C10-Pad1) -> +5VD
- C10 pad 2: Net-(C10-Pad2) -> GND
- C12 pad 2: Net-(C12-Pad2) -> GND
- C13 pad 1: VDD -> Net-(C12-Pad1)
- C2 pad 1: +5V -> VDD
- C3 pad 1: (no net) -> VDD
- C3 pad 2: (no net) -> GND
- C4 pad 1: Net-(C4-Pad1) -> VDD
- C5 pad 1: +5V -> SIM800C_DATA
- D2 pad 1: Net-(C12-Pad1) -> (no net)
- D3 pad 1: GND -> Net-(D3-Pad1)
- D3 pad 2: Net-(D3-Pad2) -> VDD
- D5 pad 1: (no net) -> Net-(C12-Pad1)
- D5 pad 2: GND -> Vin
- L1 pad 1: Net-(C12-Pad1) -> Net-(C11-Pad2)
- R1 pad 1: (no net) -> GSM_ANT
- R1 pad 2: Net-(R1-Pad2) -> Net-(ANT1-Pad1)
- R10 pad 1: Net-(D3-Pad2) -> SIM800C_DTR
- R10 pad 2: VDD -> Net-(R10-Pad2)
- R11 pad 1: GND -> SIM800C_RI
- R11 pad 2: Net-(Q2-Pad1) -> Net-(R11-Pad2)
- R12 pad 1: Net-(Q4-Pad1) -> Net-(D3-Pad1)
- R12 pad 2: SIM800L_STATUS -> Net-(Q2-Pad3)
- R13 pad 1: Net-(Q4-Pad1) -> Net-(Q2-Pad1)
- R13 pad 2: GND -> SIM800C_NETLIGHT
- R14 pad 1: Net-(D6-Pad1) -> Net-(Q2-Pad1)
- R14 pad 2: (no net) -> GND
- R18 pad 2: SIM800L_RST -> Vin
- R19 pad 1: Net-(R19-Pad1) -> GND
- R19 pad 2: SIM800L_CLK -> Net-(R18-Pad1)
- R2 pad 1: (no net) -> Net-(Q1-Pad1)
- R2 pad 2: Net-(R2-Pad2) -> PWRKEY
- R20 pad 1: SIM800L_DATA -> VDD
- R3 pad 1: (no net) -> Net-(R3-Pad1)
- R3 pad 2: Net-(R3-Pad2) -> SIM800C_RST
- R4 pad 1: (no net) -> Net-(R4-Pad1)
- R4 pad 2: Net-(R4-Pad2) -> SIM800C_CLK
- R5 pad 1: (no net) -> SIM800C_DATA
- R6 pad 1: Net-(Q2-Pad1) -> GND
- R6 pad 2: (no net) -> Net-(Q1-Pad1)
- R7 pad 1: Net-(C10-Pad2) -> SIM800C_TXD
- R7 pad 2: GND -> Net-(R7-Pad2)
- R8 pad 1: Net-(R8-Pad1) -> SIM800C_RXD
- R8 pad 2: GND -> Net-(R8-Pad2)
- R9 pad 1: VDD -> SIM800C_DCD
- R9 pad 2: Net-(R8-Pad1) -> Net-(R9-Pad2)
- S1 pad 1: (no net) -> RA_RESET
- S1 pad 15: (no net) -> SIM800C_TXD
- S1 pad 16: (no net) -> SIM800C_RXD
- S1 pad 17: (no net) -> SIM800C_DTR
- S1 pad 18: (no net) -> SIM800C_RI
- S1 pad 19: (no net) -> SIM800C_DCD
- S1 pad 2: (no net) -> RA_SCK
- S1 pad 20: (no net) -> PWRKEY
- S1 pad 28: (no net) -> RA_MOSI/SPID
- S1 pad 29: (no net) -> RA_MISO/SPIQ
- S1 pad 5: (no net) -> +5VD
- S1 pad 6: (no net) -> GND
- S1 pad 7: (no net) -> GND
- S1 pad 8: (no net) -> Vin
- U1 pad 1: Net-(C12-Pad2) -> SIM800C_VDD
- U1 pad 2: +5V -> Net-(R3-Pad1)
- U1 pad 3: Net-(C12-Pad1) -> Net-(R4-Pad1)
- U1 pad 5: Net-(R8-Pad1) -> GND
- U1 pad 6: Net-(C10-Pad1) -> (no net)
- U1 pad 7: (no net) -> Net-(R5-Pad2)
- U1 pad 8: Net-(C4-Pad1) -> (no net)
- U2 pad 1: Net-(R2-Pad2) -> Net-(R7-Pad2)
- U2 pad 15: SIM800L_DATA -> SIM800C_DATA
- U2 pad 16: SIM800L_CLK -> SIM800C_CLK
- U2 pad 17: SIM800L_RST -> SIM800C_RST
- U2 pad 18: SIM800L_VDD -> SIM800C_VDD
- U2 pad 2: Net-(R1-Pad2) -> Net-(R8-Pad2)
- U2 pad 28: Net-(C1-Pad1) -> Net-(C9-Pad1)
- U2 pad 34: (no net) -> VDD
- U2 pad 35: (no net) -> VDD
- U2 pad 39: (no net) -> SIM800C_PWRKEY
- U2 pad 41: SIM800L_NETLIGHT -> SIM800C_NETLIGHT
- U2 pad 42: SIM800L_STATUS -> SIM800C_STATUS
- U2 pad 5: Net-(R3-Pad2) -> Net-(R9-Pad2)
- U2 pad 6: Net-(R5-Pad2) -> Net-(R10-Pad2)
- U2 pad 7: Net-(R4-Pad2) -> Net-(R11-Pad2)
- U3 pad 12: (no net) -> RA_SCK
- U3 pad 13: (no net) -> RA_MISO/SPIQ
- U3 pad 14: (no net) -> RA_MOSI/SPID
- U3 pad 3: (no net) -> +3V3
- U3 pad 4: (no net) -> RA_RESET
- U6 pad 1: SIM800L_VDD -> Net-(R20-Pad2)
- U6 pad 2: Net-(R18-Pad1) -> Net-(C17-Pad1)
- U6 pad 3: Net-(R19-Pad1) -> Net-(C12-Pad1)
- U6 pad 6: (no net) -> Net-(C11-Pad2)
- U6 pad 7: Net-(R20-Pad2) -> Net-(C11-Pad1)
Other:
- outline, holes or cut-outs redrawn
- net class Default: clearance 0.254 -> 0.1
- rule trace_clearance: 0.254 -> 0.1
- board text added: "Vin"

Commit message: add header NEO GPS
Parts:
- moved D3 66.2 mm to (139.5, 73.8), turned to 180 degrees
- moved R12 65.1 mm to (139.5, 72.1), turned to 180 degrees
- moved R13 63.5 mm to (139.5, 66.9), turned to 180 degrees
- moved Q2 63.4 mm to (139.5, 69.5), turned to 180 degrees
- moved R14 61.4 mm to (142.3, 69.3), turned to 90 degrees
- moved R16 56.7 mm to (139.5, 64.9), turned to 180 degrees
- moved D4 56.4 mm to (139.5, 58.1), turned to 180 degrees
- moved R15 56.4 mm to (139.5, 59.9), turned to 180 degrees
- moved Q3 55.9 mm to (139.5, 62.4), turned to 180 degrees
- moved R17 53.8 mm to (142.3, 62.7), turned to 90 degrees
- moved R6 53.4 mm to (145.4, 75.6), turned to 180 degrees
- moved R2 53.2 mm to (145.4, 77.2)
- moved Q1 49.3 mm to (145.4, 72.9), turned to 180 degrees
- moved R11 37.6 mm to (137.5, 77.4), turned to 90 degrees
- moved R10 35.8 mm to (135.7, 77.4), turned to 90 degrees
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Connections:
- D5 pad 2: Vin -> +5VD
Other:
- outline, holes or cut-outs redrawn
- net class Default: trace_width 0.3 -> 2
