File: esp32-cellular-shield.kicad_pcb (KiCad board)
At the start: 2 copper layers, 68.5 x 53.3 mm, 57 parts, among them Q1 Q_NPN_BEC, Q2 Q_NPN_BEC, Q3 Q_NPN_BEC, U1 SIM HOLD - PPSS-6P, U2 SIM800C, U3 Ra-02, U4 MCP601OT, U5 IRLM6402, U6 MCP16311-MNY, U7 TC1264-3.3VAB

Commit message: add ignore .dcm in .gitignore & final connect PCB
Parts:
- added J1: CONN_01X04, Pin_Headers:Pin_Header_Straight_1x04_Pitch2.54mm, F.Cu at (148.6, 87.8)
- added J2: CONN_01X05, Pin_Headers:Pin_Header_Straight_1x05_Pitch2.54mm, F.Cu at (145.3, 80.2)
- moved C14 32.5 mm to (172.6, 89.1)
- moved C15 26.1 mm to (169.6, 89.1)
- moved L1 25.1 mm to (166.7, 94.7), turned to 0 degrees
- moved C11 21.7 mm to (167.1, 89.1), turned to 270 degrees
- moved R20 18.8 mm to (163.0, 85.7)
- moved C17 18.1 mm to (165.3, 85.7), turned to 90 degrees
- moved U6 13.5 mm to (163.0, 89.2), turned to 0 degrees
- moved R21 13.4 mm to (160.8, 85.7), turned to 90 degrees
- moved C12 13.0 mm to (157.6, 94.7), turned to 270 degrees
- moved C13 12.9 mm to (160.8, 94.7), turned to 270 degrees
- moved C16 12.2 mm to (138.4, 83.9), turned to 0 degrees
- moved C10 10.0 mm to (150.3, 92.4)
- moved U7 9.25 mm to (139.0, 90.4), turned to 90 degrees
- moved R19 7.77 mm to (153.3, 95.2), turned to 0 degrees
- moved R18 7.68 mm to (153.3, 97.4)
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Connections:
- ANT1 pad 2: (no net) -> GND
- D5 pad 2: +5VD -> +5V
- S1 pad 28: RA_MOSI/SPID -> (no net)
- S1 pad 29: RA_MISO/SPIQ -> RA_MOSI/SPID
- S1 pad 30: (no net) -> RA_MISO/SPIQ
- S1 pad 35: (no net) -> GND
- S1 pad 36: (no net) -> +3V3
- U5 pad 2: +5VD -> +5V
Routing:
- net GND: track 0.00 -> 397.0 mm, vias 0 -> 10
- net VDD: track 0.00 -> 176.7 mm, vias 0 -> 6
- net +3V3: track 0.00 -> 70.5 mm, vias 0 -> 2
- net SIM800C_TXD: track 0.00 -> 60.4 mm, vias 0 -> 2
- net SIM800C_PWRKEY: track 0.00 -> 59.6 mm, vias 0 -> 2
- net SIM800C_RXD: track 0.00 -> 51.3 mm, vias 0 -> 2
- net RA_MISO/SPIQ: track 0.00 -> 49.0 mm, vias 0 -> 1
- net SIM800C_RI: track 0.00 -> 48.7 mm, vias 0 -> 2
- net SIM800C_DTR: track 0.00 -> 46.7 mm, vias 0 -> 1
- net RA_MOSI/SPID: track 0.00 -> 44.9 mm, vias 0 -> 1
- net SIM800C_DCD: track 0.00 -> 41.2 mm, vias 0 -> 1
- net +5VD: track 0.00 -> 34.0 mm
- net SIM800C_DATA: track 0.00 -> 32.3 mm, vias 0 -> 3
- net PWRKEY: track 0.00 -> 31.7 mm
- net SIM800C_VDD: track 0.00 -> 29.9 mm, vias 0 -> 2
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Other:
- net class Default: clearance 0.1 -> 0.254; trace_width 2 -> 1.5
- rule trace_clearance: 0.1 -> 0.254

Commit message: completed PCB
Parts:
- removed J1: CONN_01X04, Pin_Headers:Pin_Header_Straight_1x04_Pitch2.54mm
- added G***: LOGO, lib:logo-iotmakervn_7.5x5, F.Cu at (113.3, 92.2)
- added R24: 100R, lib:R_0603, F.Cu at (146.3, 86.9)
- added R25: 100R, lib:R_0603, F.Cu at (146.3, 89.4)
- moved C16 13.0 mm to (137.5, 96.8)
- moved J2 12.3 mm to (141.8, 91.9), turned to 180 degrees
- moved U7 2.39 mm to (136.7, 90.4), turned to 270 degrees
- moved R1 1.18 mm to (120.0, 55.9)
- moved U3 0.50 mm to (126.1, 90.5)
Connections:
- ANT1 pad 2: GND -> (no net)
- J2 pad 2: GPS_RX -> Net-(J2-Pad2)
- J2 pad 3: GPS_TX -> Net-(J2-Pad3)
- J2 pad 5: +5VD -> VDD
- R7 pad 1: SIM800C_TXD -> GPS_TX
- R8 pad 1: SIM800C_RXD -> GPS_RX
- S1 pad 15: SIM800C_TXD -> GPS_TX
- S1 pad 16: SIM800C_RXD -> GPS_RX
- U1 pad 8: (no net) -> GND
Routing:
- net GPS_TX: track 3.30 -> 90.0 mm, vias 0 -> 2
- net GPS_RX: track 3.30 -> 88.0 mm, vias 0 -> 2
- net SIM800C_TXD: track 60.4 -> 0.00 mm, vias 2 -> 0
- net SIM800C_RXD: track 51.3 -> 0.00 mm, vias 2 -> 0
- net VDD: track 176.7 -> 155.0 mm, vias 6 -> 5
- net +5VD: track 34.0 -> 18.1 mm
- net GND: track 397.0 -> 406.1 mm, vias 10 -> 12
- net +3V3: track 70.5 -> 61.7 mm
- net Net-(J2-Pad3): track 0.00 -> 3.75 mm
- net Net-(J2-Pad2): track 0.00 -> 3.75 mm
- net SIM800C_VDD: track 29.9 -> 27.7 mm
- net RA_MISO/SPIQ: track 49.0 -> 51.2 mm
- net SIM800C_RI: track 48.7 -> 50.6 mm
- net SIM800C_DTR: track 46.7 -> 48.1 mm
- net RA_SCK: track 28.6 -> 27.2 mm
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- added copper zone on B.Cu, net GND
Other:
- outline, holes or cut-outs redrawn
- net class Default: trace_width 1.5 -> 1
- board text added: "0"
- board text added: "02"
- board text added: "04"
- board text added: "05"
- board text added: "06"
- board text added: "07"
- board text added: "08"
- board text added: "09"
- board text added: "10"
- board text added: "11"
- board text added: "12"
- board text added: "13"
- board text added: "14"
- board text added: "15"
- board text added: "18"
- board text added: "19"
- board text added: "21"
- board text added: "22"
- board text added: "23"
- board text added: "25"
- board text added: "26"
- board text added: "27"
- board text added: "3.3V"
- board text added: "34"
- board text added: "35"
- board text added: "36"
- board text added: "39"
- board text added: "5V"
- board text added: "EN"
- board text added: "GND"
- board text added: "Maker"
- board text added: "PSS"
- board text added: "RX"
- board text added: "SCL 22"
- board text added: "SDA 21"
- board text added: "TX"

Commit message: add table connect & name pin
Routing:
- added copper zone on F.Cu, net GND
Other:
- board text added: "4.2V"
- board text added: "DCD"
- board text added: "DTR"
- board text added: "ESP32"
- board text added: "GPIO0"
- board text added: "GPIO02"
- board text added: "GPIO04"
- board text added: "GPIO05"
- board text added: "GPIO06"
- board text added: "GPIO07"
- board text added: "GPIO08"
- board text added: "GPIO09"
- board text added: "GPIO10"
- board text added: "GPIO11"
- board text added: "GPIO12"
- board text added: "GPIO13"
- board text added: "GPIO14"
- board text added: "GPIO15"
- board text added: "GPIO18"
- board text added: "GPIO19"
- board text added: "GPIO21"
- board text added: "GPIO22"
- board text added: "GPIO23"
- board text added: "GPIO25"
- board text added: "GPIO26"
- board text added: "GPIO27"
- board text added: "GPIO34"
- board text added: "GPIO35"
- board text added: "GPIO36"
- board text added: "GPIO39"
- board text added: "HEADER NEO-6M"
- board text added: "LORA-02"
- board text added: "MISO"
- board text added: "MOSI"
- board text added: "NEO-6M"
- board text added: "NETLIGHT"
- board text added: "OLED"
- board text added: "PWRKEY"
- board text added: "RESET"
- board text added: "RI"
- board text added: "RXD"
- board text added: "SCK"
- board text added: "SIM800C"
- board text added: "STATUS"
- board text added: "TXD"
