File: esp32-cellular-shield.kicad_pcb (KiCad board)
At the start: 2 copper layers, 68.5 x 53.3 mm, 61 parts, among them J2 CONN_01X05, Q1 Q_NPN_BEC, Q2 Q_NPN_BEC, Q3 Q_NPN_BEC, U1 SIM HOLD - PPSS-6P, U2 SIM800C, U3 Ra-02, U4 MCP601OT, U5 IRLM6402, U6 MCP16311-MNY, U7 TC1264-3.3VAB

Commit message: compledted modify PCB - TC1264 change TO-220 to SOT223, Connec SCL, SDA to 21, 22 on PCB
Parts:
- removed PWR1: PWRKEY, lib:Tact_switch-4pin
- removed U5: IRLM6402, TO_SOT_Packages_SMD:SOT-23_Handsoldering
- added Q4: Q_PMOS_GSD, lib:SOT-23, F.Cu at (153.3, 88.2)
- added REF**: SolderWirePad_single_1mmDrill, Wire_Pads:SolderWirePad_single_1mmDrill, F.Cu at (139.4, 55.6)
- added REF**: SolderWirePad_single_1mmDrill, Wire_Pads:SolderWirePad_single_1mmDrill, F.Cu at (153.0, 56.3)
- added SW1: SW_Push, lib:Tact_switch-4pin, F.Cu at (111.4, 64.5)
- U1: value SIM HOLD - PPSS-6P -> SIM_HOLDER
- U7: footprint lib:TO-220 -> TO_SOT_Packages_SMD:SOT-223-3Lead_TabPin2
- moved C16 11.4 mm to (135.3, 85.6)
- moved U3 1.90 mm to (124.2, 90.7)
- moved U7 1.27 mm to (136.4, 91.7)
- moved G*** 1.05 mm to (112.3, 92.5)
Connections:
- S1 pad 23: (no net) -> SCL
- S1 pad 24: (no net) -> SDA
- S1 pad 33: (no net) -> SDA
- S1 pad 34: (no net) -> SCL
- U1 pad 8: GND -> (no net)
Routing:
- net SCL: track 0.00 -> 83.9 mm, vias 0 -> 2
- net SDA: track 0.00 -> 83.0 mm, vias 0 -> 2
- net VDD: track 155.0 -> 169.4 mm
- net GND: track 406.1 -> 416.5 mm
- net +3V3: track 61.7 -> 70.1 mm, vias 2 -> 3
- net SIM800C_DATA: track 33.5 -> 38.7 mm
- net RA_SCK: track 27.2 -> 31.8 mm
- net +5VD: track 18.1 -> 21.8 mm
- net RA_RESET: track 13.8 -> 16.9 mm
- net Net-(Q4-Pad1): track 7.82 -> 5.17 mm
- net SIM800C_VDD: track 27.7 -> 29.3 mm
- net +5V: track 2.93 -> 4.44 mm
- net SIM800C_PWRKEY: track 59.4 -> 60.6 mm
- net RA_MOSI/SPID: track 43.8 -> 44.9 mm
- net RA_MISO/SPIQ: track 51.2 -> 50.1 mm
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Other:
- outline, holes or cut-outs redrawn
- net class Default: clearance 0.254 -> 0.1; trace_width 1 -> 0.4
- rule trace_clearance: 0.254 -> 0.1

Commit message: change MOSFET irlml6402 to AO3401 30v, 4A & add gerber
Other:
- board text added: "21 SDA"
- board text added: "22 SCL"
- board text added: "9"
- board text removed: "SCL 22"
- board text removed: "SDA 21"

Commit message: modifypinout sample esp32-uno
Parts:
- removed the REF** at (139.4, 55.6)
- removed the REF** at (153.0, 56.3)
- added REF**: SolderWirePad_single_1mmDrill, Wire_Pads:SolderWirePad_single_1mmDrill, F.Cu at (152.8, 56.9)
- added REF**: SolderWirePad_single_1mmDrill, Wire_Pads:SolderWirePad_single_1mmDrill, F.Cu at (165.6, 59.6)
- Q4: value Q_PMOS_GSD -> AO3401_PMOS_GSD
- moved G*** 0.11 mm to (112.3, 92.4)
Connections:
- S1 pad 1: RA_RESET -> (no net)
- S1 pad 2: RA_SCK -> (no net)
- S1 pad 25: (no net) -> RA_RESET
- S1 pad 26: (no net) -> RA_MOSI/SPID
- S1 pad 27: (no net) -> RA_MISO/SPIQ
- S1 pad 28: (no net) -> RA_SCK
- S1 pad 29: RA_MOSI/SPID -> (no net)
- S1 pad 30: RA_MISO/SPIQ -> (no net)
Routing:
- net RA_RESET: track 16.9 -> 86.6 mm, vias 0 -> 4
- net RA_SCK: track 31.8 -> 56.9 mm
- net RA_MOSI/SPID: track 44.9 -> 50.5 mm
- net RA_MISO/SPIQ: track 50.1 -> 53.7 mm
- net SIM800C_PWRKEY: track 60.6 -> 58.2 mm
- net PWRKEY: track 32.7 -> 34.8 mm
- net +3V3: track 70.1 -> 71.8 mm
- net GND: track 416.5 -> 414.9 mm
- net VDD: track 169.4 -> 167.8 mm
- net GPS_TX: track 90.3 -> 91.2 mm
- net SDA: track 83.0 -> 83.9 mm
- net SCL: track 83.9 -> 84.7 mm
Other:
- net class Default: clearance 0.1 -> 0.254
- rule trace_clearance: 0.1 -> 0.254
- board text added: "16"
- board text added: "17"
- board text added: "GPIO16"
- board text added: "GPIO17"
- board text removed: "06"
- board text removed: "07"
- board text removed: "08"
- board text removed: "09"
- board text removed: "10"
- board text removed: "11"
- board text removed: "9"
- board text removed: "GPIO07"
- board text removed: "GPIO08"
- board text removed: "GPIO09"
- board text removed: "GPIO10"
- board text removed: "OLED"

Commit message: update gerber file
Other:
- board text added: "x"
Changed lines of the file:
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@@
-(kicad_pcb (version 20170123) (host pcbnew no-vcs-found-23a23d3~58~ubuntu16.04.1)
+(kicad_pcb (version 20170123) (host pcbnew no-vcs-found-4011ed4~58~ubuntu16.04.1)
   (general
-    (links 0)
+    (links 141)
     (no_connects 0)
     (area 108.595999 50.785954 177.602094 104.185956)
     (thickness 1.6)
-    (drawings 1138)
+    (drawings 1148)
     (tracks 745)
     (zones 0)
@@
     (pad 3 thru_hole circle (at 3.675 -2 270) (size 2.2 2.2) (drill 1.5) (layers *.Cu *.Mask))
   )
+  (gr_text x (at 138.303 61.087 270) (layer B.SilkS)
+    (effects (font (size 1 1) (thickness 0.25)) (justify mirror))
+  )
+  (gr_text x (at 140.843 61.087 270) (layer B.SilkS)
+    (effects (font (size 1 1) (thickness 0.25)) (justify mirror))
+  )
+  (gr_text x (at 143.383 61.087 270) (layer B.SilkS)
+    (effects (font (size 1 1) (thickness 0.25)) (justify mirror))
+  )
+  (gr_text x (at 145.796 61.087 270) (layer B.SilkS)
+    (effects (font (size 1 1) (thickness 0.25)) (justify mirror))
+  )
+  (gr_text x (at 159.893 61.087 270) (layer B.SilkS)
+    (effects (font (size 1 1) (thickness 0.25)) (justify mirror))
+  )
+  (gr_text x (at 167.513 61.087 270) (layer B.SilkS)
+    (effects (font (size 1 1) (thickness 0.25)) (justify mirror))
+  )
+  (gr_text x (at 162.433 61.087 270) (layer B.SilkS)
+    (effects (font (size 1 1) (thickness 0.25)) (justify mirror))
+  )
+  (gr_text x (at 164.973 61.087 270) (layer B.SilkS)
+    (effects (font (size 1 1) (thickness 0.25)) (justify mirror))
+  )
+  (gr_text x (at 170.053 61.087 270) (layer B.SilkS)
+    (effects (font (size 1 1) (thickness 0.25)) (justify mirror))
+  )
+  (gr_text x (at 172.593 61.087 270) (layer B.SilkS)
+    (effects (font (size 1 1) (thickness 0.25)) (justify mirror))
+  )
   (gr_text 16 (at 145.4912 85.4456 90) (layer F.SilkS)

Commit message: fix mistake TX, RX GPS to GPIO26 - TX_GPS, GPIO27 - RX_GPS
Changed lines of the file:
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@@
-(kicad_pcb (version 20170123) (host pcbnew no-vcs-found-4011ed4~58~ubuntu16.04.1)
+(kicad_pcb (version 20170123) (host pcbnew no-vcs-found-bf21640~58~ubuntu16.10.1)
   (general
     (links 141)
@@
     (effects (font (size 0.7 0.7) (thickness 0.175)))
   )
-  (gr_text GPIO16 (at 155.194 81.534) (layer F.SilkS)
+  (gr_text GPIO16 (at 155.2575 80.01) (layer F.SilkS)
     (effects (font (size 0.7 0.7) (thickness 0.175)))
   )
-  (gr_text GPIO17 (at 155.194 80.01) (layer F.SilkS)
+  (gr_text GPIO17 (at 155.194 81.534) (layer F.SilkS)
     (effects (font (size 0.7 0.7) (thickness 0.175)))
   )

Commit message: drop IC PWR 3.3V & swap pin connect to the module
Parts:
- removed ANT1: ANTENNA, lib:coaxial_u.fl-r-smt-1
- removed C10: 100nF, lib:C_0603
- removed C16: 1uF/25V, lib:C_0603
- removed G***: LOGO, lib:logo-iotmakervn_7.5x5
- removed Q4: AO3401_PMOS_GSD, lib:SOT-23
- removed R19: 10k, lib:R_0603
- removed REF** (x2): SolderWirePad_single_1mmDrill, Wire_Pads:SolderWirePad_single_1mmDrill
- removed SW1: SW_Push, lib:Tact_switch-4pin
- removed U4: MCP601OT, TO_SOT_Packages_SMD:SOT-23-5
- removed U7: TC1264-3.3VAB, TO_SOT_Packages_SMD:SOT-223-3Lead_TabPin2
- added AE1: Antenna_Shield, lib:sma_90_r300.124.403, F.Cu at (109.4, 99.1)
- added AE2: Antenna_Shield, lib:sma_90_r300.124.403, F.Cu at (109.4, 55.9)
- added D6: Led_PWR, LEDs:LED_0603, F.Cu at (163.3, 95.8)
- added R22: 470R, lib:R_0603, F.Cu at (163.3, 92.1)
- J2: footprint Pin_Headers:Pin_Header_Straight_1x05_Pitch2.54mm -> lib:Pin_Header_NEO6M_GPS_R2_1x05_Pitch2.54mm
- R18: value 10k -> 0R
- R20: value 200k/1% -> 52.5k/1%
- R21: value 47k/1% -> 12k/1%
- U1: footprint lib:sim_socket_PP -> lib:MicroSim-Socket-6P
- moved J2 40.3 mm to (164.8, 58.9), turned to 270 degrees
- moved R18 33.9 mm to (119.4, 99.1)
- moved R25 30.9 mm to (163.1, 63.5)
- moved R24 26.6 mm to (159.0, 63.5), turned to 180 degrees
- moved C17 18.1 mm to (147.4, 88.9), turned to 270 degrees
- moved U1 17.4 mm to (161.3, 81.8), turned to 90 degrees
- moved D5 12.8 mm to (146.1, 94.0), turned to 90 degrees
- moved U6 11.3 mm to (151.8, 88.9)
- moved C11 10.9 mm to (156.2, 88.8)
- moved C15 10.9 mm to (158.8, 87.6), turned to 270 degrees
- moved R21 10.8 mm to (150.0, 85.9), turned to 180 degrees
- moved C14 10.2 mm to (162.6, 87.6), turned to 270 degrees
- moved R20 9.43 mm to (153.5, 85.9), turned to 180 degrees
- moved L1 7.95 mm to (158.8, 94.0), turned to 270 degrees
- moved C12 7.81 mm to (149.9, 94.0)
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Connections:
- D2 pad 1: (no net) -> Net-(D2-Pad1)
- D5 pad 2: +5V -> +5VD
- J2 pad 1: (no net) -> Net-(J2-Pad1)
- J2 pad 5: VDD -> +3V3
- R1 pad 1: GSM_ANT -> Net-(AE2-Pad1)
- R1 pad 2: Net-(ANT1-Pad1) -> Net-(R1-Pad2)
- R18 pad 2: Vin -> Net-(R18-Pad2)
- R7 pad 1: GPS_TX -> SIM800C_TXD
- R8 pad 1: GPS_RX -> SIM800C_RXD
- S1 pad 1: (no net) -> Net-(S1-Pad1)
- S1 pad 10: (no net) -> RA_CS
- S1 pad 11: (no net) -> RA_SCK
- S1 pad 12: (no net) -> RA_MISO/SPIQ
- S1 pad 13: (no net) -> RA_MOSI/SPID
- S1 pad 14: (no net) -> RA_RESET
- S1 pad 15: GPS_TX -> Net-(S1-Pad15)
- S1 pad 16: GPS_RX -> Net-(S1-Pad16)
- S1 pad 17: SIM800C_DTR -> Net-(S1-Pad17)
- S1 pad 18: SIM800C_RI -> Net-(S1-Pad18)
- S1 pad 19: SIM800C_DCD -> Net-(S1-Pad19)
- S1 pad 2: (no net) -> Net-(S1-Pad2)
- S1 pad 20: PWRKEY -> Net-(S1-Pad20)
- S1 pad 21: (no net) -> GPS_TX
- S1 pad 22: (no net) -> GPS_RX
- S1 pad 25: RA_RESET -> SIM800C_DTR
- S1 pad 26: RA_MOSI/SPID -> SIM800C_RI
- S1 pad 27: RA_MISO/SPIQ -> SIM800C_DCD
- S1 pad 28: RA_SCK -> PWRKEY
- S1 pad 29: (no net) -> SIM800C_RXD
- S1 pad 3: (no net) -> Net-(S1-Pad3)
- S1 pad 30: (no net) -> SIM800C_TXD
- S1 pad 31: (no net) -> Net-(S1-Pad31)
- S1 pad 32: (no net) -> Net-(S1-Pad32)
- S1 pad 4: (no net) -> +3V3
- S1 pad 9: (no net) -> Net-(S1-Pad9)
- U1 pad 6: (no net) -> Net-(U1-Pad6)
- U2 pad 10: (no net) -> Net-(U2-Pad10)
- U2 pad 11: (no net) -> Net-(U2-Pad11)
- U2 pad 12: (no net) -> Net-(U2-Pad12)
- U2 pad 14: (no net) -> Net-(U2-Pad14)
- U2 pad 20: (no net) -> Net-(U2-Pad20)
- U2 pad 22: (no net) -> UART2_T
- U2 pad 23: (no net) -> UART2_R
- U2 pad 24: (no net) -> USB_VBUS
- U2 pad 25: (no net) -> USB_DP
- U2 pad 26: (no net) -> Net-(U2-Pad26)
- U2 pad 29: (no net) -> Net-(U2-Pad29)
- U2 pad 3: (no net) -> Net-(U2-Pad3)
- U2 pad 32: GSM_ANT -> Net-(R1-Pad2)
- U2 pad 38: (no net) -> ADC
- U2 pad 4: (no net) -> Net-(U2-Pad4)
- U2 pad 40: (no net) -> Net-(U2-Pad40)
- U2 pad 9: (no net) -> Net-(U2-Pad9)
- U3 pad 1: GND -> Net-(R18-Pad2)
- U3 pad 10: (no net) -> Net-(U3-Pad10)
- U3 pad 11: (no net) -> Net-(U3-Pad11)
- U3 pad 15: (no net) -> RA_CS
- U3 pad 5: (no net) -> Net-(U3-Pad5)
- U3 pad 6: (no net) -> Net-(U3-Pad6)
- U3 pad 7: (no net) -> Net-(U3-Pad7)
- U3 pad 8: (no net) -> Net-(U3-Pad8)
Routing:
- net GND: track 414.9 -> 184.6 mm, vias 12 -> 2
- net VDD: track 167.8 -> 48.7 mm, vias 5 -> 3
- net RA_RESET: track 86.6 -> 0.00 mm, vias 4 -> 0
- net GPS_RX: track 87.3 -> 15.5 mm, vias 2 -> 0
- net GPS_TX: track 91.2 -> 20.5 mm, vias 2 -> 0
- net SIM800C_PWRKEY: track 58.2 -> 0.00 mm, vias 2 -> 0
- net RA_SCK: track 56.9 -> 0.00 mm, vias 1 -> 0
- net RA_MISO/SPIQ: track 53.7 -> 0.00 mm, vias 1 -> 0
- net SIM800C_RI: track 50.6 -> 0.00 mm, vias 2 -> 0
- net RA_MOSI/SPID: track 50.5 -> 0.00 mm, vias 1 -> 0
- net SIM800C_DTR: track 47.9 -> 0.00 mm, vias 1 -> 0
- net SIM800C_DCD: track 41.0 -> 0.00 mm, vias 1 -> 0
- net SDA: track 83.9 -> 44.3 mm, vias 2 -> 0
- net SIM800C_DATA: track 38.7 -> 0.00 mm, vias 3 -> 0
- net SCL: track 84.7 -> 48.2 mm, vias 2 -> 0
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- removed copper zone on B.Cu, net GND
- removed copper zone on F.Cu, net GND
Other:
- outline, holes or cut-outs redrawn
- net class Default: clearance 0.254 -> 0.1
- rule trace_clearance: 0.254 -> 0.1

Commit message: compledted connect pcb
Parts:
- moved D2 0.05 mm to (145.3, 58.4)
Connections:
- U1 pad 10: (no net) -> GND
- U1 pad 11: (no net) -> GND
- U1 pad 8: (no net) -> GND
- U1 pad 9: (no net) -> GND
Routing:
- net GND: track 184.6 -> 444.2 mm, vias 2 -> 12
- net VDD: track 48.7 -> 133.1 mm, vias 3 -> 7
- net RA_RESET: track 0.00 -> 81.2 mm, vias 0 -> 1
- net RA_CS: track 0.00 -> 73.0 mm, vias 0 -> 1
- net RA_MOSI/SPID: track 0.00 -> 71.8 mm, vias 0 -> 2
- net RA_SCK: track 0.00 -> 69.2 mm, vias 0 -> 2
- net RA_MISO/SPIQ: track 0.00 -> 68.0 mm, vias 0 -> 1
- net +3V3: track 49.1 -> 114.4 mm
- net SIM800C_RI: track 0.00 -> 50.8 mm, vias 0 -> 2
- net SIM800C_VDD: track 0.00 -> 44.2 mm, vias 0 -> 2
- net SIM800C_DTR: track 0.00 -> 44.0 mm, vias 0 -> 1
- net SIM800C_DATA: track 0.00 -> 43.9 mm, vias 0 -> 3
- net SIM800C_DCD: track 0.00 -> 43.8 mm, vias 0 -> 1
- net SIM800C_RXD: track 0.00 -> 43.5 mm, vias 0 -> 1
- net SIM800C_TXD: track 0.00 -> 40.4 mm, vias 0 -> 1
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Other:
- outline, holes or cut-outs redrawn
- net class Default: clearance 0.1 -> 0.254
- rule trace_clearance: 0.1 -> 0.254
- board text added: "CS"
- board text added: "LORA"
- board text removed: "LORA-02"

Commit message: add header battery
Parts:
- added J1: CONN_01X02, Pin_Headers:Pin_Header_Straight_1x02_Pitch2.00mm, F.Cu at (112.7, 66.6)
Routing:
- net VDD: track 133.1 -> 135.5 mm
