File: esp32-cellular-shield.kicad_pcb (KiCad board)
At the start: 2 copper layers, 68.5 x 53.3 mm, 57 parts, among them J1 CONN_01X02, J2 CONN_01X05, Q1 Q_NPN_BEC, Q2 Q_NPN_BEC, Q3 Q_NPN_BEC, U1 SIM_HOLDER, U2 SIM800C, U3 Ra-02, U6 MCP16311-MNY

Commit message: final PCB
Parts:
- added G***: LOGO, lib:logo_cc-bby-sa_14.1x5mm, F.Cu at (167.8, 89.7)
- added G***: LOGO, lib:logo-iotmakervn_7.5x5, F.Cu at (113.5, 91.4)
- added VAL**: oshw_logo_500, lib:logo5, F.Cu at (118.9, 88.4)
- J2: footprint lib:Pin_Header_NEO6M_GPS_R2_1x05_Pitch2.54mm -> Pin_Header_NEO6M_GPS_R2_1x05_Pitch2.54mm
- moved S1 0.25 mm to (139.4, 76.2)
Routing:
- net RA_CS: track 73.0 -> 76.9 mm
- net SIM800C_DATA: track 43.9 -> 40.3 mm
- net GND: track 444.3 -> 447.7 mm
- net VDD: track 135.5 -> 138.0 mm
- net +3V3: track 114.4 -> 116.6 mm
- net RA_MOSI/SPID: track 71.8 -> 73.9 mm
- net SIM800C_VDD: track 44.2 -> 46.0 mm
- net SIM800C_DCD: track 43.8 -> 42.4 mm
- net RA_MISO/SPIQ: track 68.0 -> 69.1 mm
- net RA_RESET: track 81.2 -> 82.3 mm
- net SIM800C_PWRKEY: track 31.8 -> 32.7 mm
- net RA_SCK: track 69.2 -> 70.1 mm
- net GPS_TX: track 20.5 -> 21.2 mm
- net SIM800C_NETLIGHT: track 27.2 -> 27.9 mm
- net SIM800C_RXD: track 43.5 -> 43.0 mm
- added copper zone on B.Cu, net GND
- added copper zone on F.Cu, net GND
Other:
- board text added: "+"
- board text added: "-"
- board text added: "BAT"
- board text added: "IO0"
- board text added: "IO02"
- board text added: "IO04"
- board text added: "IO05"
- board text added: "IO12"
- board text added: "IO13"
- board text added: "IO14"
- board text added: "IO15"
- board text added: "IO16"
- board text added: "IO17"
- board text added: "IO18"
- board text added: "IO19"
- board text added: "IO21"
- board text added: "IO22"
- board text added: "IO23"
- board text added: "IO25"
- board text added: "IO26"
- board text added: "IO27"
- board text added: "IO34"
- board text added: "IO35"
- board text added: "IO36"
- board text added: "IO39"
- board text added: "https://esp32.vn"
- board text removed: "4.2V"
- board text removed: "GPIO0"
- board text removed: "GPIO02"
- board text removed: "GPIO04"
- board text removed: "GPIO06"
- board text removed: "GPIO11"
- board text removed: "GPIO21"
- board text removed: "GPIO22"
- board text removed: "GPIO25"
- board text removed: "GPIO34"
- board text removed: "GPIO35"
- board text removed: "GPIO36"
- board text removed: "HEADER NEO-6M"
