File: esp32-cellular-shield.sch (KiCad schematic (older format))
At the start: 57 parts, among them Q1 Q_NPN_BEC, Q2 Q_NPN_BEC, Q3 Q_NPN_BEC, Q4 Q_NPN_BEC, U1 MP2365DN, U2 SIM800C, U3 Ra-02, U4 LM1117-3.3, U6 SIM HOLD - PPSS-6P

Commit message: deleted RESET, SIM800C_RESET
Parts:
- removed D?: D_TVS_ALT, symbol D_TVS_ALT
- removed Q2: Q_NPN_BEC, symbol Q_NPN_BEC
- removed R11, R6: 4.7k, lib:R_0603, symbol R_Small
- D2: value MBRS340 -> SS34
Connections:
- net labels added: UART2_R, UART2_T
- net labels removed: SIM800C_RESET, USB_DN
- wire segments 208 -> 152
- no-connect marks 12 -> 19

Commit message: completed connect sim800C & lora-ra02
Parts:
- removed C3: 10uF, lib:C_0603, symbol C_Small
- added C? (x2): 33pF, lib:C_0603, symbol C_Small
- added C?: 22nF, lib:C_0603, symbol C_Small
- added C? (x2): 1uF, lib:C_0603, symbol C_Small
- added D?: SS34, lib:do214ab, symbol D_Schottky_Small
- Q1, Q3, Q4: footprint (none) -> TO_SOT_Packages_SMD:SOT-23
Connections:
- net labels added: RA_MISO/SPIQ, RA_MOSI/SPID
- net labels removed: RA_MISO, RA_MOSI, RESET, VCC
- wire segments 152 -> 176
- no-connect marks 19 -> 48
Other:
- note added: "Cần làm nguồn 3.3V ?\nhay lấy thẳng từ 3.3V của board esp32-uno ???"
- note added: "GPIO02\n"
- note added: "GPIO04\n"
- note added: "GPIO06\n"
- note added: "GPIO07\n"
- note added: "GPIO08\n"
- note added: "GPIO09\n"
- note added: "GPIO0\n"
- note added: "GPIO10\n"
- note added: "GPIO11\n"
- note added: "GPIO25\n"
- note removed: "???"
- note removed: "ANTENNA"
- note removed: "DECOUPLING"
- moved on the sheet: ANT1, C1, C10, C12, C13, C2, C28, C29, C31, C32, C33, C34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

Commit message: add PWR 3.3V with IC tc1264-33VAB, swap IC PWR to MCP16311-MNY with Vdd=4.2V
Parts:
- removed C2: 10uF/35V, Capacitors_SMD:C_1210, symbol C_Small
- removed C4: 0.1uF, lib:C_0603, symbol C_Small
- removed C5: 10uF, lib:C_0603, symbol C_Small
- removed C?: 22nF, lib:C_0603, symbol C_Small
- removed C? (x2): 1uF, lib:C_0603, symbol C_Small
- removed D2, D?: SS34, lib:do214ab, symbol D_Schottky_Small
- removed D3: Led_pwr, LEDs:LED_0805, symbol LED_Small
- removed R10: 10k, lib:R_0603, symbol R_Small
- removed R7: 20k, lib:R_0603, symbol R_Small
- removed R8: 20k-1%, lib:R_0603, symbol R_Small
- removed R9: 68k-1%, lib:R_0603, symbol R_Small
- removed U1: MP2365DN, SMD_Packages:SOIC-8-N, symbol MP2365DN
- removed U4: LM1117-3.3, symbol LM1117-3.3
- added C11: 100nF, footprint:C_0603, symbol C_Small
- added C14, C15: 10uF/25V, footprint:C_1210, symbol C_Small
- added C16: 1uF/25V, footprint:C_1210, symbol C_Small
- added C17: 1uF, footprint:C_0603, symbol C_Small
- added D5: SS34, footprint:do214aa-g, symbol D_Schottky_Small
- added R18, R19: 10k, footprint:R_0603, symbol R_Small
- added R20: 200k/1%, footprint:R_0603, symbol R_Small
- added R21: 47k/1%, footprint:R_0603, symbol R_Small
- added U4: MCP601OT, TO_SOT_Packages_SMD:SOT-23-5, symbol MCP601OT
- added U5: IRLM6402, TO_SOT_Packages_SMD:SOT-23_Handsoldering, symbol MOSFET-P
- added U6: MCP16311-MNY, Housings_SSOP:MSOP-8_3x3mm_Pitch0.65mm, symbol MCP16311-MNY
- added U7: TC1264-3.3VAB, symbol TC1264-3.3VAB
- C10: value 4.7nF -> 100nF; footprint lib:C_0603 -> footprint:C_0603
- C12: value 10nF -> 10uF/50V; footprint lib:C_0603 -> footprint:C_1210
- C13: value 47uF -> 10uF/50V; footprint lib:C_0603 -> footprint:C_1210
- L1: value 4.7uH-2.2A -> 22uH; footprint Choke_SMD:Choke_SMD_6.3x6.3_H3 -> Choke_SMD:Choke_SMD_Wuerth-WE-PD2-Typ-MS
- gave numbers to parts that had none: 2
- renumbered C31 to C1, C32 to C2, C33 to C3, C34 to C4, C29 to C5, C28 to C7, C1 to C9, D5 to D2, D7 to D3, D6 to D4, Q3 to Q2, Q4 to Q3, R26 to R1, R5 to R10, R4 to R11, R29 to R12, R25 to R13, R28 to R14, R14 to R15, R12 to R16, R13 to R17, R24 to R2, R18 to R3, R19 to R4, R20 to R5, R27 to R6, R2 to R7, R1 to R8, R3 to R9, U6 to U1
Connections:
- net labels added: +3.3V, +5VD, VCC, Vin
- net labels removed: +5V
- wire segments 176 -> 198
- no-connect marks 48 -> 46
Other:
- note added: "5V mạch ESP32"
- note added: "ESP_UNO CASE"
- note added: "POWER"
- note added: "SIM800C"
- note added: "VDD=4.2V"
- note added: "Vin ESP32"
- note removed: "ARDUINO CASE"
- note removed: "Cần làm nguồn 3.3V ?\nhay lấy thẳng từ 3.3V của board esp32-uno ???"
- note removed: "SIM800"

Commit message: add PCB
Parts:
- C10, C11, C17: footprint footprint:C_0603 -> lib:C_0603
- C12, C13, C14, C15: footprint footprint:C_1210 -> Capacitors_SMD:C_1210
- C16: footprint footprint:C_1210 -> lib:C_0603
- D3, D4: footprint LEDs:LED_0805 -> LEDs:LED_0603
- D5: footprint footprint:do214aa-g -> lib:do214ac
- PWR1: footprint lib:SW_SPST_B3U-1000P-B -> lib:Tact_switch-4pin
- R18, R19, R20, R21: footprint footprint:R_0603 -> lib:R_0603
- U1: footprint lib:Micro_SIM_6P_PUSH_SKM01 -> lib:sim_socket_PP
- U3: footprint (none) -> lib:Lora-RA02
- U7: footprint (none) -> lib:TO-220
Connections:
- net labels removed: VCC
Other:
- moved on the sheet: C16, U7

Commit message: add header NEO GPS
Parts:
- added J?: CONN_01X04, Pin_Headers:Pin_Header_Straight_1x04_Pitch2.54mm, symbol CONN_01X04
- added J?: CONN_01X05, Pin_Headers:Pin_Header_Straight_1x05_Pitch2.54mm, symbol CONN_01X05
Connections:
- net labels added: +5V, GPS_RX, GPS_TX
- wire segments 198 -> 210
Other:
- note added: "5V OUT"
- note added: "Vin = Vin esp32\nVcc = 5V esp32"

Commit message: add ignore .dcm in .gitignore & final connect PCB
Parts:
- removed S1: ESP-UNO, lib:ESP-UNO-SH, symbol ESP-UNO-RESCUE-esp32-cellular-shield
- added S1: ESP-UNO, lib:ESP-UNO-SH, symbol ESP-UNO
- gave numbers to parts that had none: 2
Connections:
- net labels added: SCL, SDA
- wire segments 210 -> 216
- no-connect marks 46 -> 42

Commit message: completed PCB
Parts:
- removed J1: CONN_01X04, Pin_Headers:Pin_Header_Straight_1x04_Pitch2.54mm, symbol CONN_01X04
- added R24, R25: 100R, lib:R_0603, symbol R_Small
Connections:
- wire segments 216 -> 214
- no-connect marks 42 -> 43
Other:
- moved on the sheet: J2
Changed lines of the file:
@@
 EESchema Schematic File Version 2
+LIBS:esp32-cellular-shield-rescue
 LIBS:power
 LIBS:device
@@
 $EndComp
 $Comp
-L GND #PWR38
+L GND #PWR37
 U 1 1 58C464DF
 P 15150 2400
-F 0 "#PWR38" H 15150 2150 50  0001 C CNN
+F 0 "#PWR37" H 15150 2150 50  0001 C CNN
 F 1 "GND" H 15155 2227 50  0000 C CNN
 F 2 "" H 15150 2400 50  0000 C CNN
@@
 	0    -1   -1   0
 $EndComp
-Entry Wire Line
-	19800 -1000 19900 -900
 Text GLabel 14800 2100 1    60   Input ~ 0
 Vin
@@
 $EndComp
 $Comp
-L +5VD #PWR37
+L +5VD #PWR36
 U 1 1 58C3EE4E
 P 15000 2200
-F 0 "#PWR37" H 15050 2250 50  0001 C CNN
+F 0 "#PWR36" H 15050 2250 50  0001 C CNN
 F 1 "+5VD" H 15015 2373 50  0000 C CNN
 F 2 "" H -375 175 50  0001 C CNN
@@
 Vin = Vin esp32\nVcc = 5V esp32
 $Comp
-L CONN_01X04 J1
-U 1 1 58C904B8
-P 12050 5900
-F 0 "J1" H 11969 5525 50  0000 C CNN
-F 1 "CONN_01X04" H 11969 5616 50  0000 C CNN
-F 2 "Pin_Headers:Pin_Header_Straight_1x04_Pitch2.54mm" H 300 350 50  0001 C CNN
-F 3 "" H 300 350 50  0001 C CNN
-	1    12050 5900
-	-1   0    0    1
-$EndComp
-$Comp
 L CONN_01X05 J2
 U 1 1 58C90694
-P 13000 5950
-F 0 "J2" H 12919 5525 50  0000 C CNN
-F 1 "CONN_01X05" H 12919 5616 50  0000 C CNN
-F 2 "Pin_Headers:Pin_Header_Straight_1x05_Pitch2.54mm" H -550 -300 50  0001 C CNN
-F 3 "" H -550 -300 50  0001 C CNN
-	1    13000 5950
+P 13950 5950
+F 0 "J2" H 13869 5525 50  0000 C CNN
+F 1 "CONN_01X05" H 13869 5616 50  0000 C CNN
+F 2 "Pin_Headers:Pin_Header_Straight_1x05_Pitch2.54mm" H 400 -300 50  0001 C CNN
+F 3 "" H 400 -300 50  0001 C CNN
+	1    13950 5950
 	-1   0    0    1
-$EndComp
-$Comp
-L +5VD #PWR31
-U 1 1 58C90950
-P 12400 5450
-F 0 "#PWR31" H 12450 5500 50  0001 C CNN
-F 1 "+5VD" H 12415 5623 50  0000 C CNN
-F 2 "" H -2975 3425 50  0001 C CNN
-F 3 "" H -2975 3425 50  0001 C CNN
-	1    12400 5450
-	1    0    0    -1
-$EndComp
-$Comp
-L GND #PWR32
-U 1 1 58C909D1
-P 12700 6350
-F 0 "#PWR32" H 12700 6100 50  0001 C CNN
-F 1 "GND" H 12705 6177 50  0000 C CNN
-F 2 "" H 12700 6350 50  0000 C CNN
-F 3 "" H 12700 6350 50  0000 C CNN
-	1    12700 6350
-	1    0    0    -1
-$EndComp
-$Comp
-L +5VD #PWR34
-U 1 1 58C90E93
-P 13800 5700
-F 0 "#PWR34" H 13850 5750 50  0001 C CNN
-F 1 "+5VD" H 13815 5873 50  0000 C CNN
-F 2 "" H -1575 3675 50  0001 C CNN
-F 3 "" H -1575 3675 50  0001 C CNN
-	1    13800 5700
-	1    0    0    -1
 $EndComp
 Connection ~ 10450 2050
@@
 Connection ~ 8200 10150
 Wire Wire Line
-	13800 5700 13800 5750
-Wire Wire Line
-	13800 5750 13200 5750
-Wire Wire Line
-	12400 5450 12400 5750
-Wire Wire Line
-	12400 5750 12250 5750
-$Comp
-L GND #PWR35
+	14750 5700 14750 5750
+Wire Wire Line
+	14750 5750 14150 5750
+$Comp
+L GND #PWR38
 U 1 1 58C9149B
-P 13800 6250
-F 0 "#PWR35" H 13800 6000 50  0001 C CNN
-F 1 "GND" H 13805 6077 50  0000 C CNN
-F 2 "" H 13800 6250 50  0000 C CNN
-F 3 "" H 13800 6250 50  0000 C CNN
-	1    13800 6250
-	1    0    0    -1
-$EndComp
-Wire Wire Line
-	13200 5850 13800 5850
-Wire Wire Line
-	13800 5850 13800 6250
-Wire Wire Line
-	12250 6050 12700 6050
-Wire Wire Line
-	12700 6050 12700 6350
-Text GLabel 12350 5950 2    60   Input ~ 0
+P 15250 6250
+F 0 "#PWR38" H 15250 6000 50  0001 C CNN
+F 1 "GND" H 15255 6077 50  0000 C CNN
+F 2 "" H 15250 6250 50  0000 C CNN
+F 3 "" H 15250 6250 50  0000 C CNN
+	1    15250 6250
+	1    0    0    -1
+$EndComp
+Wire Wire Line
+	14150 5850 15250 5850
+Wire Wire Line
+	15250 5850 15250 6250
+Text GLabel 14700 5950 2    60   Input ~ 0
+GPS_RX
+Text GLabel 14700 6050 2    60   Input ~ 0
 GPS_TX
-Text GLabel 12350 5850 2    60   Input ~ 0
-GPS_RX
-Wire Wire Line
-	12350 5850 12250 5850
-Wire Wire Line
-	12350 5950 12250 5950
-Text GLabel 13300 6050 2    60   Input ~ 0
-GPS_RX
-Text GLabel 13300 5950 2    60   Input ~ 0
-GPS_TX
-Wire Wire Line
-	13300 5950 13200 5950
-Wire Wire Line
-	13300 6050 13200 6050
+Wire Wire Line
+	14150 5950 14350 5950
+Wire Wire Line
+	14150 6050 14350 6050
 Text Notes 1850 7850 0    60   ~ 0
 5V mạch ESP32
@@
 	13800 3600 13800 3750
 $Comp
-L +3.3V #PWR36
+L +3.3V #PWR34
 U 1 1 58C9B32D
 P 14225 3750
-F 0 "#PWR36" H 14275 3800 50  0001 C CNN
+F 0 "#PWR34" H 14275 3800 50  0001 C CNN
 F 1 "+3.3V" H 14240 3923 50  0000 C CNN
 F 2 "" H 5975 -5850 50  0001 C CNN
@@
 $Comp
 L ESP-UNO S1
-U 1 1 58C9C3C7
+U 1 1 58C9FD5D
 P 13750 2200
 F 0 "S1" H 13725 913 60  0000 C CNN
 F 1 "ESP-UNO" H 13725 1019 60  0000 C CNN
-F 2 "lib:ESP-UNO-SH" H -1425 925 60  0001 C CNN
-F 3 "" H -1425 925 60  0001 C CNN
+F 2 "lib:ESP-UNO-SH" H 800 -1200 60  0001 C CNN
+F 3 "" H 800 -1200 60  0001 C CNN
 	1    13750 2200
 	-1   0    0    1
 $EndComp
+Text GLabel 12550 1200 1    60   Input ~ 0
+GPS_TX
+Text GLabel 12400 1200 1    60   Input ~ 0
+GPS_RX
+Wire Wire Line
+	12550 1200 12550 1300
+Connection ~ 12550 1300
+Wire Wire Line
+	12400 1200 12400 1400
+Connection ~ 12400 1400
+$Comp
+L R_Small R24
+U 1 1 58CA211F
+P 14450 5950
+F 0 "R24" V 14550 5950 50  0000 L CNN
+F 1 "100R" V 14450 5800 50  0000 L CNN
+F 2 "lib:R_0603" H 14450 5950 50  0001 C CNN
+F 3 "" H 14450 5950 50  0000 C CNN
+	1    14450 5950
+	0    -1   -1   0
+$EndComp
+$Comp
+L R_Small R25
+U 1 1 58CA3493
+P 14450 6050
+F 0 "R25" V 14550 6050 50  0000 L CNN
+F 1 "100R" V 14450 5900 50  0000 L CNN
+F 2 "lib:R_0603" H 14450 6050 50  0001 C CNN
+F 3 "" H 14450 6050 50  0000 C CNN
+	1    14450 6050
+	0    -1   -1   0
+$EndComp
+Wire Wire Line
+	14550 5950 14700 5950
+Wire Wire Line
+	14550 6050 14700 6050
+NoConn ~ 14150 6150
+$Comp
+L VDD #PWR?
+U 1 1 58CA7D0A
+P 14750 5700
+F 0 "#PWR?" H 14800 5750 50  0001 C CNN
+F 1 "VDD" H 14767 5873 50  0000 C CNN
+F 2 "" H 8400 -3875 50  0001 C CNN
+F 3 "" H 8400 -3875 50  0001 C CNN
+	1    14750 5700
+	1    0    0    -1
+$EndComp
+Text Notes 14550 5500 0    60   ~ 0
+VDD=4.2V
 $EndSCHEMATC
