File: esp32-cellular-shield.sch (KiCad schematic (older format))
At the start: 60 parts, among them J2 CONN_01X05, Q1 Q_NPN_BEC, Q2 Q_NPN_BEC, Q3 Q_NPN_BEC, U1 SIM HOLD - PPSS-6P, U2 SIM800C, U3 Ra-02, U4 MCP601OT, U5 IRLM6402, U6 MCP16311-MNY, U7 TC1264-3.3VAB

Commit message: compledted modify PCB - TC1264 change TO-220 to SOT223, Connec SCL, SDA to 21, 22 on PCB
Parts:
- removed PWR1: PWRKEY, lib:Tact_switch-4pin, symbol SW_PUSH
- removed U1: SIM HOLD - PPSS-6P, lib:sim_socket_PP, symbol C707_10M006_049_2
- removed U5: IRLM6402, TO_SOT_Packages_SMD:SOT-23_Handsoldering, symbol MOSFET-P
- added Q4: Q_PMOS_GSD, lib:SOT-23, symbol Q_PMOS_GSD
- added SW1: SW_Push, lib:Tact_switch-4pin, symbol SW_Push
- added U1: SIM_HOLDER, lib:sim_socket_PP, symbol SIM_HOLDER
- U7: footprint lib:TO-220 -> TO_SOT_Packages_SMD:SOT-223-3Lead_TabPin2
Connections:
- wire segments 214 -> 216
- no-connect marks 43 -> 42
Other:
- note added: "Right or Wrong ?"
- note added: "cấp cho IC \nMCP16311-MNY"
- moved on the sheet: C5, R5
Changed lines of the file:
@@
 LIBS:sim800c
 LIBS:tc1264-33VAB
+LIBS:dc-dc
+LIBS:microsd_spi_cd
+LIBS:switches
 LIBS:esp32-cellular-shield-cache
 EELAYER 26 0
@@
 	1    0    0    -1
 $EndComp
-Text GLabel 8600 1725 1    60   Input ~ 0
+Text GLabel 8650 1725 1    60   Input ~ 0
 SIM800C_DATA
 Text GLabel 6925 1500 1    60   Input ~ 0
@@
 Text GLabel 6225 1500 1    60   Input ~ 0
 SIM800C_VDD
-NoConn ~ 8100 1700
+NoConn ~ 8150 1700
 $Comp
 L GND #PWR05
 U 1 1 57DA6BB4
-P 8275 1525
-F 0 "#PWR05" H 8275 1275 50  0001 C CNN
-F 1 "GND" H 8280 1352 50  0000 C CNN
-F 2 "" H 8275 1525 50  0000 C CNN
-F 3 "" H 8275 1525 50  0000 C CNN
-	1    8275 1525
+P 8325 1525
+F 0 "#PWR05" H 8325 1275 50  0001 C CNN
+F 1 "GND" H 8330 1352 50  0000 C CNN
+F 2 "" H 8325 1525 50  0000 C CNN
+F 3 "" H 8325 1525 50  0000 C CNN
+	1    8325 1525
 	-1   0    0    1
 $EndComp
@@
 L C_Small C5
 U 1 1 57DA6BB7
-P 8600 2175
-F 0 "C5" H 8692 2221 50  0000 L CNN
-F 1 "22pF" H 8692 2130 50  0000 L CNN
-F 2 "lib:C_0603" H 8600 2175 50  0001 C CNN
-F 3 "" H 8600 2175 50  0000 C CNN
-	1    8600 2175
+P 8650 2175
+F 0 "C5" H 8742 2221 50  0000 L CNN
+F 1 "22pF" H 8742 2130 50  0000 L CNN
+F 2 "lib:C_0603" H 8650 2175 50  0001 C CNN
+F 3 "" H 8650 2175 50  0000 C CNN
+	1    8650 2175
 	1    0    0    -1
 $EndComp
@@
 L GND #PWR07
 U 1 1 57DA6BB8
-P 8600 2275
-F 0 "#PWR07" H 8600 2025 50  0001 C CNN
-F 1 "GND" H 8605 2102 50  0000 C CNN
-F 2 "" H 8600 2275 50  0000 C CNN
-F 3 "" H 8600 2275 50  0000 C CNN
-	1    8600 2275
+P 8650 2275
+F 0 "#PWR07" H 8650 2025 50  0001 C CNN
+F 1 "GND" H 8655 2102 50  0000 C CNN
+F 2 "" H 8650 2275 50  0000 C CNN
+F 3 "" H 8650 2275 50  0000 C CNN
+	1    8650 2275
 	1    0    0    -1
 $EndComp
@@
 L R_Small R5
 U 1 1 57DA6BBA
-P 8325 1800
-F 0 "R5" V 8255 1800 50  0000 C CNN
-F 1 "22R" V 8325 1810 50  0000 C CNN
-F 2 "lib:R_0603" H 8325 1800 50  0001 C CNN
-F 3 "" H 8325 1800 50  0000 C CNN
-	1    8325 1800
+P 8375 1800
+F 0 "R5" V 8305 1800 50  0000 C CNN
+F 1 "22R" V 8375 1810 50  0000 C CNN
+F 2 "lib:R_0603" H 8375 1800 50  0001 C CNN
+F 3 "" H 8375 1800 50  0000 C CNN
+	1    8375 1800
 	0    1    -1   0
 $EndComp
@@
 Text GLabel 1900 2525 1    60   Input ~ 0
 SIM800C_PWRKEY
-$Comp
-L SW_PUSH PWR1
-U 1 1 58B31DFA
-P 1500 2600
-F 0 "PWR1" H 1500 2855 50  0000 C CNN
-F 1 "PWRKEY" H 1500 2764 50  0000 C CNN
-F 2 "lib:Tact_switch-4pin" H -7100 -5000 50  0001 C CNN
-F 3 "" H -7100 -5000 50  0000 C CNN
-	1    1500 2600
-	1    0    0    -1
-$EndComp
 $Comp
 L GND #PWR012
@@
 	1    6925 2375
 	1    0    0    -1
-$EndComp
-$Comp
-L C707_10M006_049_2 U1
-U 1 1 57DA6BAF
-P 7500 1700
-F 0 "U1" V 7135 1925 50  0000 C CNN
-F 1 "SIM HOLD - PPSS-6P" V 7226 1925 50  0000 C CNN
-F 2 "lib:sim_socket_PP" H 7500 1700 60  0001 C CNN
-F 3 "" H 7500 1700 60  0000 C CNN
-	1    7500 1700
-	0    1    1    0
 $EndComp
 $Comp
@@
 NoConn ~ 12850 2500
 NoConn ~ 12850 2400
-NoConn ~ 12850 2300
 NoConn ~ 12850 3000
 NoConn ~ 12850 3100
@@
 $EndComp
 $Comp
-L MOSFET-P U5
-U 1 1 58C3E074
-P 3300 8550
-F 0 "U5" H 3393 8520 30  0000 L CNN
-F 1 "IRLM6402" H 3393 8580 30  0000 L CNN
-F 2 "TO_SOT_Packages_SMD:SOT-23_Handsoldering" H 3300 8500 60  0001 C CNN
-F 3 "" H 3300 8500 60  0000 C CNN
-	1    3300 8550
-	1    0    0    1
-$EndComp
-$Comp
 L R_Small R18
 U 1 1 58C3E075
@@
 L +5VD #PWR024
 U 1 1 58C3F322
-P 3775 8700
-F 0 "#PWR024" H 3825 8750 50  0001 C CNN
-F 1 "+5VD" H 3790 8873 50  0000 C CNN
-F 2 "" H -11600 6675 50  0001 C CNN
-F 3 "" H -11600 6675 50  0001 C CNN
-	1    3775 8700
-	1    0    0    -1
-$EndComp
-Text Notes 3475 8450 0    60   ~ 0
+P 3800 8950
+F 0 "#PWR024" H 3850 9000 50  0001 C CNN
+F 1 "+5VD" H 3815 9123 50  0000 C CNN
+F 2 "" H -11575 6925 50  0001 C CNN
+F 3 "" H -11575 6925 50  0001 C CNN
+	1    3800 8950
+	1    0    0    -1
+$EndComp
+Text Notes 3500 8750 0    60   ~ 0
 5V mạch ESP32
 Text Notes 5100 9700 0    60   ~ 0
@@
 F 0 "U7" H 7150 10737 60  0000 C CNN
 F 1 "TC1264-3.3VAB" H 7150 10631 60  0000 C CNN
-F 2 "lib:TO-220" H -2400 800 60  0001 C CNN
+F 2 "TO_SOT_Packages_SMD:SOT-223-3Lead_TabPin2" H -2400 800 60  0001 C CNN
 F 3 "" H -2400 800 60  0001 C CNN
 	1    7150 10250
@@
 	9475 5575 9475 5875
 Wire Wire Line
-	8100 1800 8225 1800
+	8150 1800 8275 1800
 Wire Wire Line
 	7825 2100 7825 1950
 Wire Wire Line
-	8600 1725 8600 2075
-Wire Wire Line
-	7825 1950 8600 1950
-Connection ~ 8600 1950
+	8650 1725 8650 2075
+Wire Wire Line
+	7825 1950 8650 1950
+Connection ~ 8650 1950
 Wire Wire Line
 	4400 4450 4400 4650
@@
 	1150 2650 1150 2600
 Wire Wire Line
-	1150 2600 1200 2600
-Wire Wire Line
-	1800 2600 2500 2600
+	1150 2600 1300 2600
+Wire Wire Line
+	1700 2600 2500 2600
 Connection ~ 1900 2600
 Wire Wire Line
-	8425 1800 8600 1800
-Connection ~ 8600 1800
+	8475 1800 8650 1800
+Connection ~ 8650 1800
 Wire Wire Line
 	7350 1600 6225 1600
@@
 Connection ~ 6925 2700
 Wire Wire Line
-	8275 1525 8275 1600
-Wire Wire Line
-	8275 1600 8100 1600
+	8325 1525 8325 1600
+Wire Wire Line
+	8325 1600 8150 1600
 Wire Wire Line
 	12125 1600 12850 1600
@@
 	2850 9900 2700 9900
 Wire Wire Line
-	2700 9900 2700 9800
+	2700 9800 2700 9900
 Connection ~ 2700 9800
 Wire Wire Line
@@
 	2550 8550 3100 8550
 Wire Wire Line
-	3300 8900 3300 8750
-Wire Wire Line
-	3775 8900 3300 8900
-Wire Wire Line
-	3300 8250 3300 8350
+	3400 8250 3400 8350
 Wire Wire Line
 	2150 8100 2150 8250
@@
 Wire Wire Line
 	2000 10600 5350 10600
-Wire Wire Line
-	3775 8700 3775 8900
 Wire Wire Line
 	7750 10350 7900 10350
@@
 Text Notes 1850 7850 0    60   ~ 0
 5V mạch ESP32
-Text Notes 3150 8050 0    60   ~ 0
+Text Notes 3250 8050 0    60   ~ 0
 5V OUT
 $Comp
 L +5V #PWR030
 U 1 1 58C94A58
-P 3300 8250
-F 0 "#PWR030" H 3350 8300 50  0001 C CNN
-F 1 "+5V" H 3315 8423 50  0000 C CNN
-F 2 "" H 0   100 50  0001 C CNN
-F 3 "" H 0   100 50  0001 C CNN
-	1    3300 8250
+P 3400 8250
+F 0 "#PWR030" H 3450 8300 50  0001 C CNN
+F 1 "+5V" H 3415 8423 50  0000 C CNN
+F 2 "" H 100 100 50  0001 C CNN
+F 3 "" H 100 100 50  0001 C CNN
+	1    3400 8250
 	1    0    0    -1
 $EndComp
@@
 Text Notes 14550 5500 0    60   ~ 0
 VDD=4.2V
+$Comp
+L SIM_HOLDER U1
+U 1 1 58CB5237
+P 7750 1750
+F 0 "U1" H 7750 2162 60  0000 C CNN
+F 1 "SIM_HOLDER" H 7750 2056 60  0000 C CNN
+F 2 "lib:sim_socket_PP" H -375 -275 60  0001 C CNN
+F 3 "" H -375 -275 60  0000 C CNN
+	1    7750 1750
+	1    0    0    -1
+$EndComp
+$Comp
+L Q_PMOS_GSD Q4
+U 1 1 58CB5C4D
+P 3300 8550
+F 0 "Q4" H 3506 8504 50  0000 L CNN
+F 1 "Q_PMOS_GSD" H 3506 8595 50  0000 L CNN
+F 2 "lib:SOT-23" H 200 0   50  0001 C CNN
+F 3 "" H 0   -100 50  0001 C CNN
+	1    3300 8550
+	1    0    0    1
+$EndComp
+Wire Wire Line
+	3400 8750 3400 9000
+Wire Wire Line
+	3400 9000 3800 9000
+Wire Wire Line
+	3800 9000 3800 8950
+Text GLabel 12750 2300 0    60   Input ~ 0
+SDA
+Text GLabel 12750 2200 0    60   Input ~ 0
+SCL
+Wire Wire Line
+	12850 2300 12750 2300
+Wire Wire Line
+	12850 2200 12750 2200
+$Comp
+L SW_Push SW1
+U 1 1 58CB69CF
+P 1500 2600
+F 0 "SW1" H 1500 2885 50  0000 C CNN
+F 1 "SW_Push" H 1500 2794 50  0000 C CNN
+F 2 "lib:Tact_switch-4pin" H -1000 400 50  0001 C CNN
+F 3 "" H -1000 400 50  0001 C CNN
+	1    1500 2600
+	1    0    0    -1
+$EndComp
+Wire Notes Line
+	3600 8000 4350 8000
+Text Notes 4500 8050 0    118  ~ 24
+Right or Wrong ?
+Text Notes 3700 8100 0    60   ~ 0
+cấp cho IC \nMCP16311-MNY
 $EndSCHEMATC

Commit message: change MOSFET irlml6402 to AO3401 30v, 4A & add gerber
Parts:
- Q4: value Q_PMOS_GSD -> AO3401_PMOS_GSD
Other:
- note added: "Header GPS NEO"
- note removed: "Right or Wrong ?"
- note removed: "cấp cho IC \nMCP16311-MNY"
- moved on the sheet: J2, R24, R25
Changed lines of the file:
@@
 Text GLabel 4500 2400 1    60   Input ~ 0
 SIM800C_NETLIGHT
-Text Notes 5050 9150 0    157  ~ 31
+Text Notes 5050 8350 0    157  ~ 31
 POWER SUPPLY
 Text Notes 12850 800  0    157  ~ 31
@@
 	1    0    0    -1
 $EndComp
-Text Notes 3000 7550 0    118  ~ 24
+Text Notes 5200 8850 0    118  ~ 24
 Vin = Vin esp32\nVcc = 5V esp32
 $Comp
 L CONN_01X05 J2
 U 1 1 58C90694
-P 13950 5950
-F 0 "J2" H 13869 5525 50  0000 C CNN
-F 1 "CONN_01X05" H 13869 5616 50  0000 C CNN
-F 2 "Pin_Headers:Pin_Header_Straight_1x05_Pitch2.54mm" H 400 -300 50  0001 C CNN
-F 3 "" H 400 -300 50  0001 C CNN
-	1    13950 5950
+P 13350 6000
+F 0 "J2" H 13269 5575 50  0000 C CNN
+F 1 "CONN_01X05" H 13269 5666 50  0000 C CNN
+F 2 "Pin_Headers:Pin_Header_Straight_1x05_Pitch2.54mm" H -200 -250 50  0001 C CNN
+F 3 "" H -200 -250 50  0001 C CNN
+	1    13350 6000
 	-1   0    0    1
 $EndComp
@@
 	6000 5025 6000 6800
 Wire Notes Line
-	400  6800 11200 6800
+	400  6800 16100 6800
 Wire Notes Line
 	11200 4700 16100 4700
@@
 	2850 9900 2700 9900
 Wire Wire Line
-	2700 9800 2700 9900
+	2700 9900 2700 9800
 Connection ~ 2700 9800
 Wire Wire Line
@@
 Connection ~ 8200 10150
 Wire Wire Line
-	14750 5700 14750 5750
-Wire Wire Line
-	14750 5750 14150 5750
+	14150 5750 14150 5800
+Wire Wire Line
+	14150 5800 13550 5800
 $Comp
 L GND #PWR029
 U 1 1 58C9149B
-P 15250 6250
-F 0 "#PWR029" H 15250 6000 50  0001 C CNN
-F 1 "GND" H 15255 6077 50  0000 C CNN
-F 2 "" H 15250 6250 50  0000 C CNN
-F 3 "" H 15250 6250 50  0000 C CNN
-	1    15250 6250
-	1    0    0    -1
-$EndComp
-Wire Wire Line
-	14150 5850 15250 5850
-Wire Wire Line
-	15250 5850 15250 6250
-Text GLabel 14700 5950 2    60   Input ~ 0
+P 14650 6300
+F 0 "#PWR029" H 14650 6050 50  0001 C CNN
+F 1 "GND" H 14655 6127 50  0000 C CNN
+F 2 "" H 14650 6300 50  0000 C CNN
+F 3 "" H 14650 6300 50  0000 C CNN
+	1    14650 6300
+	1    0    0    -1
+$EndComp
+Wire Wire Line
+	13550 5900 14650 5900
+Wire Wire Line
+	14650 5900 14650 6300
+Text GLabel 14100 6000 2    60   Input ~ 0
 GPS_RX
-Text GLabel 14700 6050 2    60   Input ~ 0
+Text GLabel 14100 6100 2    60   Input ~ 0
 GPS_TX
 Wire Wire Line
-	14150 5950 14350 5950
-Wire Wire Line
-	14150 6050 14350 6050
+	13550 6000 13750 6000
+Wire Wire Line
+	13550 6100 13750 6100
 Text Notes 1850 7850 0    60   ~ 0
 5V mạch ESP32
@@
 L R_Small R24
 U 1 1 58CA211F
-P 14450 5950
-F 0 "R24" V 14550 5950 50  0000 L CNN
-F 1 "100R" V 14450 5800 50  0000 L CNN
-F 2 "lib:R_0603" H 14450 5950 50  0001 C CNN
-F 3 "" H 14450 5950 50  0000 C CNN
-	1    14450 5950
+P 13850 6000
+F 0 "R24" V 13950 6000 50  0000 L CNN
+F 1 "100R" V 13850 5850 50  0000 L CNN
+F 2 "lib:R_0603" H 13850 6000 50  0001 C CNN
+F 3 "" H 13850 6000 50  0000 C CNN
+	1    13850 6000
 	0    -1   -1   0
 $EndComp
@@
 L R_Small R25
 U 1 1 58CA3493
-P 14450 6050
-F 0 "R25" V 14550 6050 50  0000 L CNN
-F 1 "100R" V 14450 5900 50  0000 L CNN
-F 2 "lib:R_0603" H 14450 6050 50  0001 C CNN
-F 3 "" H 14450 6050 50  0000 C CNN
-	1    14450 6050
+P 13850 6100
+F 0 "R25" V 13950 6100 50  0000 L CNN
+F 1 "100R" V 13850 5950 50  0000 L CNN
+F 2 "lib:R_0603" H 13850 6100 50  0001 C CNN
+F 3 "" H 13850 6100 50  0000 C CNN
+	1    13850 6100
 	0    -1   -1   0
 $EndComp
 Wire Wire Line
-	14550 5950 14700 5950
-Wire Wire Line
-	14550 6050 14700 6050
-NoConn ~ 14150 6150
+	13950 6000 14100 6000
+Wire Wire Line
+	13950 6100 14100 6100
+NoConn ~ 13550 6200
 $Comp
 L VDD #PWR036
 U 1 1 58CA7D0A
-P 14750 5700
-F 0 "#PWR036" H 14800 5750 50  0001 C CNN
-F 1 "VDD" H 14767 5873 50  0000 C CNN
-F 2 "" H 8400 -3875 50  0001 C CNN
-F 3 "" H 8400 -3875 50  0001 C CNN
-	1    14750 5700
-	1    0    0    -1
-$EndComp
-Text Notes 14550 5500 0    60   ~ 0
+P 14150 5750
+F 0 "#PWR036" H 14200 5800 50  0001 C CNN
+F 1 "VDD" H 14167 5923 50  0000 C CNN
+F 2 "" H 7800 -3825 50  0001 C CNN
+F 3 "" H 7800 -3825 50  0001 C CNN
+	1    14150 5750
+	1    0    0    -1
+$EndComp
+Text Notes 13950 5550 0    60   ~ 0
 VDD=4.2V
 $Comp
@@
 P 3300 8550
 F 0 "Q4" H 3506 8504 50  0000 L CNN
-F 1 "Q_PMOS_GSD" H 3506 8595 50  0000 L CNN
+F 1 "AO3401_PMOS_GSD" H 3506 8595 50  0000 L CNN
 F 2 "lib:SOT-23" H 200 0   50  0001 C CNN
 F 3 "" H 0   -100 50  0001 C CNN
@@
 	1    0    0    -1
 $EndComp
-Wire Notes Line
-	3600 8000 4350 8000
-Text Notes 4500 8050 0    118  ~ 24
-Right or Wrong ?
-Text Notes 3700 8100 0    60   ~ 0
-cấp cho IC \nMCP16311-MNY
+Text Notes 13200 5200 0    118  ~ 24
+Header GPS NEO
 $EndSCHEMATC
